File: PCB/FSAE-BaseBoard/FSAE-BaseBoard-1.kicad_sch (KiCad schematic)
At the start: 6 parts, among them J1 Hat_ESP, U6 ESP32 C3, U7 ESP32 S3

Commit message: Actualizacion de la placa de desarollo - v.2
Parts:
- removed J1: Hat_ESP, symbol Connector:Conn_01x11_Socket
- removed TP1: TestPoint, symbol Connector:TestPoint
- added BZ1: Buzzer, symbol Device:Buzzer
- added J1: Conn_01x14_Socket, symbol Connector:Conn_01x14_Socket
- added R2: R, symbol Device:R
- added R3, R4, R5, R6: 10k, symbol Device:R
- added SW1, SW2, SW3, SW4: SW_Push, symbol Switch:SW_Push
- renumbered U6 to U4, U7 to U5
Connections:
- net GPIO21 is gone; now on net INT_LORA: U5.27 (GPIO21/RTC)
- net GPIO47 is gone; now on net RST_LORA: U5.28 (GPIO47/SPICLK_P)
- net GPIO48 is gone; now on net CS_LORA: U5.29 (GPIO48/SPICLK_N)
- net MISO_LORA is gone; now on net ENC_B: U5.18 (GPIO12/RTC/TOUCH12/ADC2_1)
- net MOSI_LORA is gone; now on net ENC_A: U5.17 (GPIO11/RTC/TOUCH11/ADC2_0)
- net SCK_LORA is gone; now on net RX: U5.19 (GPIO13/RTC/TOUCH13/ADC2_2)
- net +5V: now also J1.1 (Pin_1)
- net A0_MODE: now also U5.15 (GPIO9/RTC/TOUCH9/ADC1_8); no longer U5.11 (GPIO18/RTC/U1RXD/ADC2_7/CLK_OUT3)
- net A1_MODE: now also U5.16 (GPIO10/RTC/TOUCH10/ADC1_9); no longer U5.12 (GPIO8/RTC/TOUCH8/ADC1_7)
- net CS_LORA: no longer U5.20 (GPIO14/RTC/TOUCH14/ADC2_3)
- net CS_RES: now also U5.12 (GPIO8/RTC/TOUCH8/ADC1_7); no longer U5.38 (GPIO41/MTDI/CLK_OUT1)
- net CTRL_RELE: now also U5.4 (GPIO4/RTC/TOUCH4/ADC1_3); no longer U4.3 (GPIO7/CS), U5.7 (GPIO7/RTC/TOUCH7/ADC1_6)
- net ENC_A: no longer U5.37 (GPIO40/MTDO/CLK_OUT2)
- net ENC_B: no longer U5.36 (GPIO39/MTCK/CLK_OUT3)
- net GND: now also BZ1.2 (-), J1.13 (Pin_13), J1.14 (Pin_14), SW1.2, SW2.2, SW3.2, SW4.2
- net INT_LORA: no longer U5.9 (GPIO16/RTC/U0CTS/ADC2_5)
- net INT_MPU: no longer U5.15 (GPIO9/RTC/TOUCH9/ADC1_8)
- net RST_LORA: no longer U5.8 (GPIO15/RTC/U0RTS/ADC2_4)
- net RX: no longer U5.5 (GPIO5/RTC/TOUCH5/ADC1_4)
- net SAMPLE: now also U5.36 (GPIO39/MTCK/CLK_OUT3); no longer U5.10 (GPIO17/RTC/U1TXD/ADC2_6)
- net SCL_MPU: now also J1.4 (Pin_4); no longer U5.16 (GPIO10/RTC/TOUCH10/ADC1_9)
- net SDA_MPU: now also J1.3 (Pin_3); no longer U5.4 (GPIO4/RTC/TOUCH4/ADC1_3)
- net TX: now also U5.20 (GPIO14/RTC/TOUCH14/ADC2_3); no longer U5.6 (GPIO6/RTC/TOUCH6/ADC1_5)
- net GPIO3: now reaches U5.13 (GPIO3/RTC/TOUCH3/ADC1_2/JTAG)
- net GPIO3: now also J1.12 (Pin_12)
- net 3V3_ESP renamed +3.3V
- net +3.3V: now also J1.2 (Pin_2), R3.1, R4.1, R5.1, R6.1
- net MISO_RES renamed CTRL_BUZZER
- net CTRL_BUZZER: now also R2.1
- net MOSI_RES renamed BTN_1
- net BTN_1: now also U4.3 (GPIO7/CS), R3.2, SW1.1
- net SCK_RES renamed BTN_2
- net BTN_2: now also R4.2, SW2.1
- new net: BZ1.1 (+), R2.2
- new net ADC1_4: J1.10 (Pin_10), U5.5 (GPIO5/RTC/TOUCH5/ADC1_4)
- new net ADC1_5: J1.11 (Pin_11), U5.6 (GPIO6/RTC/TOUCH6/ADC1_5)
- new net BTN_3: R5.2, SW3.1, U5.38 (GPIO41/MTDI/CLK_OUT1)
- new net BTN_4: R6.2, SW4.1, U5.37 (GPIO40/MTDO/CLK_OUT2)
- new net MISO: J1.6 (Pin_6), U5.7 (GPIO7/RTC/TOUCH7/ADC1_6)
- new net MOSI: J1.5 (Pin_5), U5.8 (GPIO15/RTC/U0RTS/ADC2_4)
- new net SCK: J1.7 (Pin_7), U5.9 (GPIO16/RTC/U0CTS/ADC2_5)
- new net UART1_RX: J1.9 (Pin_9), U5.11 (GPIO18/RTC/U1RXD/ADC2_7/CLK_OUT3)
- new net UART1_TX: J1.8 (Pin_8), U5.10 (GPIO17/RTC/U1TXD/ADC2_6)
- no-connect marks 17 -> 16

Commit message: Actualizacion diseño BaseBoard
Parts:
- BZ1: footprint (none) -> Buzzer_Beeper:Buzzer_12x9.5RM7.6
- D1: footprint (none) -> LED_SMD:LED_0805_2012Metric_Pad1.15x1.40mm_HandSolder
- J1: footprint (none) -> Connector_PinSocket_2.54mm:PinSocket_1x14_P2.54mm_Vertical
- R1, R3, R4, R5, R6: footprint (none) -> Resistor_SMD:R_0805_2012Metric_Pad1.20x1.40mm_HandSolder
- R2: value R -> 100; footprint (none) -> Resistor_SMD:R_0805_2012Metric_Pad1.20x1.40mm_HandSolder
- SW1, SW2, SW3, SW4: footprint (none) -> Button_Switch_THT:SW_PUSH_6mm_H5mm
- U1: renamed from U4; footprint (none) -> FSAE_Kicad_Footprints:ESP32 C3 SM
- renumbered U5 to U2
Connections:
- net A0_MODE: now also U2.37 (GPIO40/MTDO/CLK_OUT2); no longer U2.15 (GPIO9/RTC/TOUCH9/ADC1_8)
- net A1_MODE: now also U2.38 (GPIO41/MTDI/CLK_OUT1); no longer U2.16 (GPIO10/RTC/TOUCH10/ADC1_9)
- net BTN_1: now also U1.2 (GPIO6/MOSI), U2.18 (GPIO12/RTC/TOUCH12/ADC2_1); no longer U1.3 (GPIO7/CS), U2.40 (GPIO2/RTC/TOUCH2/ADC1_1)
- net BTN_2: now also U2.17 (GPIO11/RTC/TOUCH11/ADC2_0); no longer U2.39 (GPIO42/MTMS)
- net BTN_3: now also U2.16 (GPIO10/RTC/TOUCH10/ADC1_9); no longer U2.38 (GPIO41/MTDI/CLK_OUT1)
- net BTN_4: now also U2.19 (GPIO13/RTC/TOUCH13/ADC2_2); no longer U2.37 (GPIO40/MTDO/CLK_OUT2)
- net CS_LORA: now also U2.40 (GPIO2/RTC/TOUCH2/ADC1_1); no longer U2.29 (GPIO48/SPICLK_N)
- net CS_RES: now also U2.39 (GPIO42/MTMS); no longer U2.12 (GPIO8/RTC/TOUCH8/ADC1_7)
- net CTRL_BUZZER: now also U2.7 (GPIO7/RTC/TOUCH7/ADC1_6); no longer U2.41 (GPIO1/RTC/TOUCH1/ADC1_0)
- net CTRL_RELE: now also U2.41 (GPIO1/RTC/TOUCH1/ADC1_0); no longer U2.4 (GPIO4/RTC/TOUCH4/ADC1_3)
- net ENC_A: now also U2.28 (GPIO47/SPICLK_P); no longer U2.17 (GPIO11/RTC/TOUCH11/ADC2_0)
- net ENC_B: now also U2.27 (GPIO21/RTC); no longer U2.18 (GPIO12/RTC/TOUCH12/ADC2_1)
- net GPIO3: now also U2.15 (GPIO9/RTC/TOUCH9/ADC1_8); no longer U2.13 (GPIO3/RTC/TOUCH3/ADC1_2/JTAG)
- net INT_LORA: now also U2.35 (GPIO38/RGB_LED); no longer U2.27 (GPIO21/RTC)
- net INT_MPU: now also U1.16 (GPIO0/A0); no longer U1.15 (GPIO1/A1)
- net LED_ESTADO: now also U1.1 (GPIO5/A5/MISO), U2.20 (GPIO14/RTC/TOUCH14/ADC2_3); no longer U1.16 (GPIO0/A0), U2.35 (GPIO38/RGB_LED)
- net MISO: now also J1.5 (Pin_5), U2.4 (GPIO4/RTC/TOUCH4/ADC1_3); no longer J1.6 (Pin_6), U2.7 (GPIO7/RTC/TOUCH7/ADC1_6)
- net MOSI: now also J1.6 (Pin_6), U2.5 (GPIO5/RTC/TOUCH5/ADC1_4); no longer J1.5 (Pin_5), U2.8 (GPIO15/RTC/U0RTS/ADC2_4)
- net RST_LORA: now also U2.29 (GPIO48/SPICLK_N); no longer U2.28 (GPIO47/SPICLK_P)
- net RX: now also U1.6 (GPIO10), U2.8 (GPIO15/RTC/U0RTS/ADC2_4); no longer U1.1 (GPIO5/A5/MISO), U2.19 (GPIO13/RTC/TOUCH13/ADC2_2)
- net SCK: now also U2.6 (GPIO6/RTC/TOUCH6/ADC1_5); no longer U2.9 (GPIO16/RTC/U0CTS/ADC2_5)
- net SCL_MPU: now also J1.3 (Pin_3), U1.13 (GPIO3/A3); no longer J1.4 (Pin_4), U1.6 (GPIO10)
- net SDA_MPU: now also J1.4 (Pin_4), U1.15 (GPIO1/A1); no longer J1.3 (Pin_3), U1.12 (GPIO4/A4/SCK)
- net SENSOR_RPM: now also U1.12 (GPIO4/A4/SCK); no longer U1.13 (GPIO3/A3)
- net TX: now also U1.3 (GPIO7/CS), U2.9 (GPIO16/RTC/U0CTS/ADC2_5); no longer U1.2 (GPIO6/MOSI), U2.20 (GPIO14/RTC/TOUCH14/ADC2_3)
- net ADC1_4 renamed ADC2_0
- net ADC2_0: now also U2.12 (GPIO8/RTC/TOUCH8/ADC1_7); no longer U2.5 (GPIO5/RTC/TOUCH5/ADC1_4)
- net ADC1_5 renamed ADC2_1
- net ADC2_1: now also U2.13 (GPIO3/RTC/TOUCH3/ADC1_2/JTAG); no longer U2.6 (GPIO6/RTC/TOUCH6/ADC1_5)
Other:
- moved on the sheet: J1, U1, U2
