File: PCB/FSAE-BaseBoard/FSAE-BaseBoard-3.kicad_sch (KiCad schematic)
At the start: 23 parts, among them J8 Conn_01x02, J9 Conn_01x02, U10 LM2596S-ADJ, U11 AMS1117-3.3

Commit message: Actualizacion de la placa de desarollo - v.2
Parts:
- removed TP_3V3_ESP1, TP_3V3_ESP_GND1, TP_3V3_GND1, TP_5V1, TP_5V_GND1, TP_BAT1, TP_BAT_GND1: TestPoint, symbol Connector:TestPoint
- added J7: Conn_01x02, symbol Connector_Generic:Conn_01x02
- added TP_5V_MAIN1, TP_5V_PER1, TP_GND1: TestPoint, symbol Connector:TestPoint
- renumbered D4 to D2, D2 to D3, D3 to D4, J8 to J6, J9 to J8, R4 to R8, R5 to R9, U10 to U7, U11 to U8
Connections:
- net 3V3_ESP is gone; now on net +3.3V: J8.2 (Pin_2)
- net +5V: now also J7.2 (Pin_2), TP_5V_PER1.1; no longer C6.1, D3.1 (K), D4.1 (K), U8.3 (VI)
- net GND: now also TP_GND1.1
- new net: C6.1, D3.1 (K), D4.1 (K), J7.1 (Pin_1), TP_5V_MAIN1.1, U8.3 (VI)
Other:
- moved on the sheet: C6, C7, D3, D4, J8, U8

Commit message: Actualizacion diseño BaseBoard
Parts:
- C3, C4, C5, C6, C7: footprint (none) -> Capacitor_SMD:C_0805_2012Metric_Pad1.18x1.45mm_HandSolder
- J7: renamed from J6; footprint (none) -> Connector_PinHeader_2.54mm:PinHeader_1x02_P2.54mm_Vertical
- J8: renamed from J7; footprint (none) -> Connector_PinHeader_2.54mm:PinHeader_1x02_P2.54mm_Vertical
- J9: renamed from J8; footprint (none) -> Connector_PinHeader_2.54mm:PinHeader_1x02_P2.54mm_Vertical
- L1: footprint (none) -> Inductor_SMD:L_Wuerth_WE-PD-Typ-LS_Handsoldering
- R8, R9: footprint (none) -> Resistor_SMD:R_0805_2012Metric_Pad1.20x1.40mm_HandSolder
- TP_3V1, TP_5V_MAIN1, TP_5V_PER1: footprint (none) -> TestPoint:TestPoint_THTPad_D2.0mm_Drill1.0mm
- TP_GND1: footprint (none) -> TestPoint:TestPoint_THTPad_2.0x2.0mm_Drill1.0mm
- renumbered U7 to U4, U8 to U5
Other:
- moved on the sheet: C3, C4, C5, C6, C7, D2, D3, D4, J7, J8, J9, L1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

Commit message: ModificacionesByNico
Corregi una eleccion de footprint y arregle un poco el layout tambien detecte una falla que no solucione que es el echo que los smd y lo th van a tener problemas para soldarlos
Parts:
- C4, C5: footprint Capacitor_SMD:C_0805_2012Metric_Pad1.18x1.45mm_HandSolder -> C_Radial_D6.3mm_H11.0mm_P2.50mm
