File: PCB/FSAE-BaseBoard/FSAE-BaseBoard-4.kicad_sch (KiCad schematic)
At the start: 22 parts, among them J11 Zocalo_Resolver, J12 Bornera_Resolver, J13 Zocalo_Resolver, J14 Screw_Terminal_01x03, J15 Bornera_Encoder, U12 LoRa SX1278, U13 MPU 6050, U14 PC817, U15 PC817, U16 PC817

Commit message: Actualizacion de la placa de desarollo - v.2
Parts:
- removed TP_ENC_A1, TP_ENC_B1, TP_ENC_B_GND1, TP_ENC_B_GND2, TP_RPM1, TP_RPM_GND1: TestPoint, symbol Connector:TestPoint
- renumbered J11 to J10, J12 to J11, J13 to J12, J14 to J13, J15 to J14, R7 to R11, R8 to R12, R9 to R13, R10 to R14, R11 to R15, R12 to R16, U13 to U10, U14 to U11, U15 to U12, U16 to U13, U12 to U9
Connections:
- net MISO_RES is gone; now on net MISO: J12.6 (Pin_6)
- net MOSI_RES is gone; now on net MOSI: J12.7 (Pin_7)
- net SCK_RES is gone; now on net SCK: J12.5 (Pin_5)
- net MISO_LORA renamed MISO
- net MOSI_LORA renamed MOSI
- net SCK_LORA renamed SCK

Commit message: Actualizacion diseño BaseBoard
Parts:
- J11: renamed from J10; footprint (none) -> Connector_PinSocket_2.54mm:PinSocket_1x08_P2.54mm_Vertical
- J12: renamed from J11; footprint (none) -> TerminalBlock_Phoenix:TerminalBlock_Phoenix_PT-1,5-6-3.5-H_1x06_P3.50mm_Horizontal
- J13: renamed from J12; footprint (none) -> Connector_PinSocket_2.54mm:PinSocket_1x08_P2.54mm_Vertical
- J14: renamed from J13; footprint (none) -> TerminalBlock_Phoenix:TerminalBlock_Phoenix_PT-1,5-3-3.5-H_1x03_P3.50mm_Horizontal
- J15: renamed from J14; footprint (none) -> TerminalBlock_Phoenix:TerminalBlock_Phoenix_PT-1,5-4-3.5-H_1x04_P3.50mm_Horizontal
- R11, R12, R13, R14, R15, R16: footprint (none) -> Resistor_SMD:R_0805_2012Metric_Pad1.20x1.40mm_HandSolder
- U6: renamed from U9; footprint (none) -> FSAE_Kicad_Footprints:LoRa_SX178
- U7: renamed from U10; footprint (none) -> FSAE_Kicad_Footprints:MPU6050
- renumbered U13 to U10, U11 to U8, U12 to U9
Connections:
- net CS_LORA: now also U6.15 (NSS); no longer U6.10 (NSS)
- net MISO: now also J13.5 (Pin_5), U6.13 (MISO); no longer J13.6 (Pin_6), U6.12 (MISO)
- net MOSI: now also U6.14 (MOSI); no longer U6.11 (MOSI)
- net SCK: now also J13.6 (Pin_6), U6.12 (SCK); no longer J13.5 (Pin_5), U6.13 (SCK)
