File: PCB/FSAE-BaseBoard/FSAE-BaseBoard-5.kicad_sch (KiCad schematic)
At the start: 7 parts, among them J10 Conn_01x03, K2 Relay_SPDT, Q1 BC817

Commit message: Actualizacion de la placa de desarollo - v.2
Parts:
- removed TP_RELE1, TP_RELE_GND1: TestPoint, symbol Connector:TestPoint
- renumbered J10 to J9, R6 to R10
Changed lines of the file:
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@@
 	(title_block
 		(title "Bloque rele")
+		(rev "v2")
 	)
 	(junction
@@
 	)
 	(junction
-		(at 118.11 105.41)
-		(diameter 0)
-		(color 0 0 0 0)
-	)
-	(junction
 		(at 148.59 82.55)
 		(diameter 0)
@@
 	(wire
 		(pts
-			(xy 116.84 105.41) (xy 118.11 105.41)
-		)
-		(stroke
-			(width 0)
-			(type default)
-		)
-	)
-	(wire
-		(pts
 			(xy 129.54 105.41) (xy 140.97 105.41)
 		)
@@
 	(wire
 		(pts
-			(xy 118.11 102.87) (xy 118.11 105.41)
-		)
-		(stroke
-			(width 0)
-			(type default)
-		)
-	)
-	(wire
-		(pts
 			(xy 132.08 86.36) (xy 132.08 82.55)
 		)
@@
 	(wire
 		(pts
-			(xy 118.11 105.41) (xy 121.92 105.41)
+			(xy 116.84 105.41) (xy 121.92 105.41)
 		)
 		(stroke
@@
 		(dnp no)
 		(fields_autoplaced yes)
-		(property "Reference" "J10"
+		(property "Reference" "J9"
 			(at 163.83 72.3899 90)
 			(effects
@@
 			(project ""
 				(path "/b93e2547-308e-44b8-b993-67c2742cde0a/0b38690d-bb9d-4f36-8216-43ed7abbfd42"
-					(reference "J10")
-					(unit 1)
-				)
-			)
-		)
-	)
-	(symbol
-		(lib_id "Connector:TestPoint")
-		(at 118.11 102.87 0)
-		(unit 1)
-		(exclude_from_sim no)
-		(in_bom yes)
-		(on_board yes)
-		(dnp no)
-		(property "Reference" "TP_RELE1"
-			(at 117.094 95.25 0)
-			(effects
-				(font
-					(size 1.27 1.27)
-				)
-				(justify left)
-			)
-		)
-		(property "Value" "TestPoint"
-			(at 117.856 97.028 0)
-			(effects
-				(font
-					(size 1.27 1.27)
-				)
-				(justify left)
-			)
-		)
-		(property "Footprint" ""
-			(at 123.19 102.87 0)
-			(effects
-				(font
-					(size 1.27 1.27)
-				)
-				(hide yes)
-			)
-		)
-		(property "Datasheet" "~"
-			(at 123.19 102.87 0)
-			(effects
-				(font
-					(size 1.27 1.27)
-				)
-				(hide yes)
-			)
-		)
-		(property "Description" "test point"
-			(at 118.11 102.87 0)
-			(effects
-				(font
-					(size 1.27 1.27)
-				)
-				(hide yes)
-			)
-		)
-		(pin "1"
-		)
-		(instances
-			(project "FSAE-BaseBoard"
-				(path "/b93e2547-308e-44b8-b993-67c2742cde0a/0b38690d-bb9d-4f36-8216-43ed7abbfd42"
-					(reference "TP_RELE1")
-					(unit 1)
-				)
-			)
-		)
-	)
-	(symbol
-		(lib_id "Connector:TestPoint")
-		(at 102.87 102.87 0)
-		(unit 1)
-		(exclude_from_sim no)
-		(in_bom yes)
-		(on_board yes)
-		(dnp no)
-		(property "Reference" "TP_RELE_GND1"
-			(at 101.854 95.25 0)
-			(effects
-				(font
-					(size 1.27 1.27)
-				)
-				(justify left)
-			)
-		)
-		(property "Value" "TestPoint"
-			(at 102.616 97.028 0)
-			(effects
-				(font
-					(size 1.27 1.27)
-				)
-				(justify left)
-			)
-		)
-		(property "Footprint" ""
-			(at 107.95 102.87 0)
-			(effects
-				(font
-					(size 1.27 1.27)
-				)
-				(hide yes)
-			)
-		)
-		(property "Datasheet" "~"
-			(at 107.95 102.87 0)
-			(effects
-				(font
-					(size 1.27 1.27)
-				)
-				(hide yes)
-			)
-		)
-		(property "Description" "test point"
-			(at 102.87 102.87 0)
-			(effects
-				(font
-					(size 1.27 1.27)
-				)
-				(hide yes)
-			)
-		)
-		(pin "1"
-		)
-		(instances
-			(project "FSAE-BaseBoard"
-				(path "/b93e2547-308e-44b8-b993-67c2742cde0a/0b38690d-bb9d-4f36-8216-43ed7abbfd42"
-					(reference "TP_RELE_GND1")
+					(reference "J9")
 					(unit 1)
 				)
@@
 	(symbol
 		(lib_id "power:GND")
-		(at 102.87 102.87 0)
-		(unit 1)
-		(exclude_from_sim no)
-		(in_bom yes)
-		(on_board yes)
-		(dnp no)
-		(fields_autoplaced yes)
-		(property "Reference" "#PWR032"
-			(at 102.87 109.22 0)
-			(effects
-				(font
-					(size 1.27 1.27)
-				)
-				(hide yes)
-			)
-		)
-		(property "Value" "GND"
-			(at 102.87 107.95 0)
-			(effects
-				(font
-					(size 1.27 1.27)
-				)
-			)
-		)
-		(property "Footprint" ""
-			(at 102.87 102.87 0)
-			(effects
-				(font
-					(size 1.27 1.27)
-				)
-				(hide yes)
-			)
-		)
-		(property "Datasheet" ""
-			(at 102.87 102.87 0)
-			(effects
-				(font
-					(size 1.27 1.27)
-				)
-				(hide yes)
-			)
-		)
-		(property "Description" "Power symbol creates a global label with name \"GND\" , ground"
-			(at 102.87 102.87 0)
-			(effects
-				(font
-					(size 1.27 1.27)
-				)
-				(hide yes)
-			)
-		)
-		(pin "1"
-		)
-		(instances
-			(project "FSAE-BaseBoard"
-				(path "/b93e2547-308e-44b8-b993-67c2742cde0a/0b38690d-bb9d-4f36-8216-43ed7abbfd42"
-					(reference "#PWR032")
-					(unit 1)
-				)
-			)
-		)
-	)
-	(symbol
-		(lib_id "power:GND")
 		(at 148.59 113.03 0)
 		(unit 1)
@@
 		(dnp no)
 		(fields_autoplaced yes)
-		(property "Reference" "#PWR033"
+		(property "Reference" "#PWR028"
 			(at 148.59 119.38 0)
 			(effects
@@
 			(project ""
 				(path "/b93e2547-308e-44b8-b993-67c2742cde0a/0b38690d-bb9d-4f36-8216-43ed7abbfd42"
-					(reference "#PWR033")
+					(reference "#PWR028")
 					(unit 1)
 				)
@@
 		(dnp no)
 		(fields_autoplaced yes)
-		(property "Reference" "R6"
+		(property "Reference" "R10"
 			(at 125.73 99.06 90)
 			(effects
@@
 			(project ""
 				(path "/b93e2547-308e-44b8-b993-67c2742cde0a/0b38690d-bb9d-4f36-8216-43ed7abbfd42"
-					(reference "R6")
+					(reference "R10")
 					(unit 1)
 				)
@@
 		(dnp no)
 		(fields_autoplaced yes)
-		(property "Reference" "#PWR031"
+		(property "Reference" "#PWR027"
 			(at 148.59 81.28 0)
 			(effects
@@
 			(project ""
 				(path "/b93e2547-308e-44b8-b993-67c2742cde0a/0b38690d-bb9d-4f36-8216-43ed7abbfd42"
-					(reference "#PWR031")
+					(reference "#PWR027")
 					(unit 1)
 				)

Commit message: Actualizacion diseño BaseBoard
Parts:
- J10: renamed from J9; footprint (none) -> Connector_PinHeader_2.54mm:PinHeader_1x03_P2.54mm_Vertical
- K1: renamed from K2; footprint (none) -> Relay_THT:Relay_SPDT_Omron-G5LE-1
- R10: footprint (none) -> Resistor_SMD:R_0805_2012Metric_Pad1.20x1.40mm_HandSolder
Connections:
- net +5V: now also K1.1; no longer K1.A1
- net at J10.1 (Pin_1): now also K1.3; no longer K1.12
- net at J10.2 (Pin_2): now also K1.5; no longer K1.14
- net at J10.3 (Pin_3): now also K1.4; no longer K1.11
- net at D5.2 (A), Q1.3 (C): now also K1.2; no longer K1.A2
