File: PCB/FSAE-BaseBoard/FSAE-BaseBoard.kicad_sch (KiCad schematic)
At the start: 6 parts, among them K1 Relay_SPDT, U1 ESP32 C3, U2 LM2596S-ADJ, U3 ESP32 S3, U4 TJA1050, U5 SN65HVD230

Commit message: Actualizacion de la placa de desarollo - v.2
Parts:
- removed U4: TJA1050, TJA1050:SOT96-1, symbol TJA1050:TJA1050
- removed U5: SN65HVD230, Package_SO:SOIC-8_3.9x4.9mm_P1.27mm, symbol Interface_CAN_LIN:SN65HVD230
Other:
- removed sheet Comunicacion CAN #
- sheet Comunicacion CAN: file FSAE-BaseBoard-2.kicad_sch -> FSAE-BaseBoard-6.kicad_sch
- sheet ESP32 C3 y S3 ports: added MISO, MOSI, SCK; removed MISO_LORA, MISO_RES, MOSI_LORA, MOSI_RES, SCK_LORA, SCK_RES
- sheet Perifericos ports: added MISO, MOSI, SCK; removed MISO_LORA, MISO_RES, MOSI_LORA, MOSI_RES, SCK_LORA, SCK_RES

Commit message: Actualizacion diseño BaseBoard
Parts:
- removed K1: Relay_SPDT, symbol Relay:Relay_SPDT
- removed U1: ESP32 C3, symbol FSAE_Kicad_Symbols.pretty:ESP32_C3_SM
- removed U2: LM2596S-ADJ, Package_TO_SOT_SMD:TO-263-5_TabPin3, symbol Regulator_Switching:LM2596S-ADJ
- removed U3: ESP32 S3, FSAE_Kicad_Footprints:ESP32 S3, symbol FSAE_Kicad_Symbols.pretty:ESP32 S3
Connections:
- no-connect marks 1 -> 0
Other:
- sheet Bloque de Alimentacion ports: added +3.3V; removed 3V3_ESP
- sheet ESP32 C3 y S3 ports: added +3.3V; removed 3V3_ESP
