File: PCB/Inverter/Primero_esquematico/core.kicad_sch (KiCad schematic)
At the start: 0 parts

Commit message: Correcciones incompletas e instalaciones de un par de extensiones copadas
Other:
- removed sheet LogicSupply1
Changed lines of the file:
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@@
 (kicad_sch
-	(version 20231120)
+	(version 20260306)
 	(generator "eeschema")
-	(generator_version "8.0")
+	(generator_version "10.0")
 	(paper "A4")
-	(sheet
-		(at 196.85 52.07)
-		(size 15.24 13.97)
-		(fields_autoplaced yes)
-		(stroke
-			(width 0.1524)
-			(type solid)
-		)
-		(fill
-			(color 0 0 0 0.0000)
-		)
-		(property "Sheetname" "LogicSupply1"
-			(at 196.85 51.3584 0)
-			(effects
-				(font
-					(size 1.27 1.27)
-				)
-				(justify left bottom)
-			)
-		)
-		(property "Sheetfile" "LogicSupply.kicad_sch"
-			(at 196.85 66.6246 0)
-			(effects
-				(font
-					(size 1.27 1.27)
-				)
-				(justify left top)
-			)
-		)
-		(pin "Vin_FB" input
-			(at 196.85 57.15 180)
-			(effects
-				(font
-					(size 1.27 1.27)
-				)
-				(justify left)
-			)
-		)
-		(pin "3,3V" input
-			(at 196.85 60.96 180)
-			(effects
-				(font
-					(size 1.27 1.27)
-				)
-				(justify left)
-			)
-		)
-		(instances
-			(project "Primero_esquematico"
-				(path "/d930f486-f6ac-489c-907e-47f2cb34cf04/f0ff413d-26b0-42cf-a9bd-9bb6e2a05cb0"
-					(page "11")
-				)
-			)
-		)
-	)
 )
