File: PCB/Inverter/Primero_esquematico/untitled.kicad_sch (KiCad schematic)
At the start: 16 parts, among them T8 Trafo 30uH - 3:1, U17 LM25180QNGURQ1

Commit message: Correcciones incompletas e instalaciones de un par de extensiones copadas
Parts:
- added U2: TPS7A2050PDBVR, Snapeda:DBV0005A-IPC_A, symbol Snapeda:TPS7A2050PDBVR
Connections:
- net 5V: now also U2.5 (OUT); no longer C77.2, D94.1 (K), D95.1 (K), R137.1
- net GND: now also U2.2 (GND)
- new net 5V_FB: C77.2, D94.1 (K), D95.1 (K), R137.1, U2.1 (IN), U2.3 (EN)
- no-connect marks 0 -> 1
Other:
- note added: "158k para 5V 174k para 5,5V 187k para 6V"
- note added: "HAY Q AJUSTAR LAS RESISTENCIAS DE FB PARA QUE GANE UN POCO MAS DE TENSION Y DE UN POCO MAS DE MARGEN"
- note added: "La funcion de este integrado es tener una salida con menos ruido y alimentar a los sensores con un sistema mas preciso"
