File: PCB/Inverter/Primero_esquematico/Primero_esquematico.kicad_pcb (KiCad board)
At the start: 2 copper layers, 37 parts, among them T1 750317595, T2 750317595, T3 750317595, T4 750317595, T5 750317595, T6 750317595, U1 UCC21750QDWRQ1, U10 LM25180QNGURQ1, U11 UCC21750QDWRQ1, U12 LM25180QNGURQ1, U13 UCC21750QDWRQ1, U2 LM25180QNGURQ1, U3 FS950R08A6P2BBPSA1, U4 LM25180QNGURQ1, U5 UCC21750QDWRQ1, U6 LM25180QNGURQ1, U7 UCC21750QDWRQ1, U8 LM25180QNGURQ1, U9 UCC21750QDWRQ1

Commit message: Correcciones incompletas e instalaciones de un par de extensiones copadas
Parts:
- added D68: 1N4148WS-Q, Diode_SMD:D_SOD-323F, F.Cu at (-30.3, 115.4)
- added D88: 1N4148WS-Q, Diode_SMD:D_SOD-323F, F.Cu at (-22.8, 115.4)
- added D93: 1N4148WS-Q, Diode_SMD:D_SOD-323F, F.Cu at (-19.2, 102.0)
- added U15: LM25180QNGURQ1, NuevoGui:NGU0008C, F.Cu at (-29.7, 111.2)
- added U16: LM25180QNGURQ1, NuevoGui:NGU0008C, F.Cu at (-22.2, 111.2)
- added U17: LM25180QNGURQ1, NuevoGui:NGU0008C, F.Cu at (-18.7, 97.8)
- added U19: AM26C32IDR, Snapeda:SOIC127P600X175-16N, F.Cu at (-36.0, 96.0)
Connections:
- U1 pad 15: /Gate_Driver/GDsupply/3,3v -> /Gate_Driver/3,3V
- U11 pad 15: /Gate_Driver/GDsupply4/3,3v -> /Gate_Driver/3,3V
- U13 pad 15: /Gate_Driver/GDsupply5/3,3v -> /Gate_Driver/3,3V
- U5 pad 15: /Gate_Driver/GDsupply1/3,3v -> /Gate_Driver/3,3V
- U7 pad 15: /Gate_Driver/GDsupply2/3,3v -> /Gate_Driver/3,3V
- U9 pad 15: /Gate_Driver/GDsupply3/3,3v -> /Gate_Driver/3,3V

Commit message: Coloque filtros y sensores
Parts:
- added REF**: CONN5_05D1509_XPR, Snapeda:CONN5_05D1509_XPR, F.Cu at (40.0, 47.0)
- moved T4 53.2 mm to (255.4, 73.3)
Changed lines of the file:
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@@
 	(footprint "FSAE-footprints:WE-FLYTI_EP7_4436"
 		(layer "F.Cu")
-		(at 204.074 59.3947)
+		(at 255.4 73.3)
 		(property "Reference" "T4"
 			(at 0 -6.135 0)
@@
 		)
 		(embedded_fonts no)
+	)
+	(footprint "Snapeda:CONN5_05D1509_XPR"
+		(layer "F.Cu")
+		(at 40 47)
+		(tags "IHL0205D1509 ")
+		(property "Reference" "REF**"
+			(at 7.62 0 0)
+			(unlocked yes)
+			(layer "F.SilkS")
+			(effects
+				(font
+					(size 1 1)
+					(thickness 0.15)
+				)
+			)
+		)
+		(property "Value" "CONN5_05D1509_XPR"
+			(at 7.62 0 0)
+			(unlocked yes)
+			(layer "F.Fab")
+			(effects
+				(font
+					(size 1 1)
+					(thickness 0.15)
+				)
+			)
+		)
+		(property "Datasheet" ""
+			(at 0 0 0)
+			(layer "F.Fab")
+			(hide yes)
+			(effects
+				(font
+					(size 1.27 1.27)
+				)
+			)
+		)
+		(property "Description" ""
+			(at 0 0 0)
+			(layer "F.Fab")
+			(hide yes)
+			(effects
+				(font
+					(size 1.27 1.27)
+				)
+			)
+		)
+		(attr through_hole)
+		(duplicate_pad_numbers_are_jumpers no)
+		(fp_line
+			(start -2.2606 -2.127)
+			(end -2.2606 5.315199)
+			(stroke
+				(width 0.1524)
+				(type solid)
+			)
+			(layer "F.SilkS")
+		)
+		(fp_line
+			(start -2.2606 5.315199)
+			(end 17.5006 5.315199)
+			(stroke
+				(width 0.1524)
+				(type solid)
+			)
+			(layer "F.SilkS")
+		)
+		(fp_line
+			(start 17.5006 -2.127)
+			(end -2.2606 -2.127)
+			(stroke
+				(width 0.1524)
+				(type solid)
+			)
+			(layer "F.SilkS")
+		)
+		(fp_line
+			(start 17.5006 5.315199)
+			(end 17.5006 -2.127)
+			(stroke
+				(width 0.1524)
+				(type solid)
+			)
+			(layer "F.SilkS")
+		)
+		(fp_circle
+			(center -4.0386 0)
+			(end -3.6576 0)
+			(stroke
+				(width 0.508)
+				(type solid)
+			)
+			(fill no)
+			(layer "F.SilkS")
+		)
+		(fp_circle
+			(center -4.0386 0)
+			(end -3.6576 0)
+			(stroke
+				(width 0.508)
+				(type solid)
+			)
+			(fill no)
+			(layer "B.SilkS")
+		)
+		(fp_line
+			(start -2.3876 -2.254)
+			(end -2.3876 5.442199)
+			(stroke
+				(width 0.1524)
+				(type solid)
+			)
+			(layer "F.CrtYd")
+		)
+		(fp_line
+			(start -2.3876 5.442199)
+			(end 17.6276 5.442199)
+			(stroke
+				(width 0.1524)
+				(type solid)
+			)
+			(layer "F.CrtYd")
+		)
+		(fp_line
+			(start 17.6276 -2.254)
+			(end -2.3876 -2.254)
+			(stroke
+				(width 0.1524)
+				(type solid)
+			)
+			(layer "F.CrtYd")
+		)
+		(fp_line
+			(start 17.6276 5.442199)
+			(end 17.6276 -2.254)
+			(stroke
+				(width 0.1524)
+				(type solid)
+			)
+			(layer "F.CrtYd")
+		)
+		(fp_line
+			(start -2.1336 -2)
+			(end -2.1336 5.188199)
+			(stroke
+				(width 0.0254)
+				(type solid)
+			)
+			(layer "F.Fab")
+		)
+		(fp_line
+			(start -2.1336 5.188199)
+			(end 17.3736 5.188199)
+			(stroke
+				(width 0.0254)
+				(type solid)
+			)
+			(layer "F.Fab")
+		)
+		(fp_line
+			(start 17.3736 -2)
+			(end -2.1336 -2)
+			(stroke
+				(width 0.0254)
+				(type solid)
+			)
+			(layer "F.Fab")
+		)
+		(fp_line
+			(start 17.3736 5.188199)
+			(end 17.3736 -2)
+			(stroke
+				(width 0.0254)
+				(type solid)
+			)
+			(layer "F.Fab")
+		)
+		(fp_circle
+			(center 0 -1.905)
+			(end 0.381 -1.905)
+			(stroke
+				(width 0.508)
+				(type solid)
+			)
+			(fill no)
+			(layer "F.Fab")
+		)
+		(fp_text user "${REFERENCE}"
+			(at 7.62 0 0)
+			(unlocked yes)
+			(layer "F.Fab")
+			(effects
+				(font
+					(size 1 1)
+					(thickness 0.15)
+				)
+			)
+		)
+		(pad "1" thru_hole circle
+			(at 0 0)
+			(size 1.0668 1.0668)
+			(drill 0.5588)
+			(layers "*.Cu" "*.Mask")
+			(remove_unused_layers no)
+		)
+		(pad "2" thru_hole circle
+			(at 2.54 0)
+			(size 1.0668 1.0668)
+			(drill 0.5588)
+			(layers "*.Cu" "*.Mask")
+			(remove_unused_layers no)
+		)
+		(pad "5" thru_hole circle
+			(at 10.16 0)
+			(size 1.0668 1.0668)
+			(drill 0.5588)
+			(layers "*.Cu" "*.Mask")
+			(remove_unused_layers no)
+		)
+		(pad "6" thru_hole circle
+			(at 12.7 0)
+			(size 1.0668 1.0668)
+			(drill 0.5588)
+			(layers "*.Cu" "*.Mask")
+			(remove_unused_layers no)
+		)
+		(pad "7" thru_hole circle
+			(at 15.24 0)
+			(size 1.0668 1.0668)
+			(drill 0.5588)
+			(layers "*.Cu" "*.Mask")
+			(remove_unused_layers no)
+		)
+		(embedded_fonts no)

Commit message: Esquematico Listo
Parts:
- removed D68, D88, D93: 1N4148WS-Q, Diode_SMD:D_SOD-323F
- removed REF**: CONN5_05D1509_XPR, Snapeda:CONN5_05D1509_XPR
- removed T2, T3, T4, T5, T6: 750317595, FSAE-footprints:WE-FLYTI_EP7_4436
- removed U11, U5, U7: UCC21750QDWRQ1, FSAE-footprints:SOIC16_DW_TEX
- removed U15, U16: LM25180QNGURQ1, NuevoGui:NGU0008C
- removed U3: FS950R08A6P2BBPSA1, FSAE-footprints:IC_FS950R08A6P2BBPSA1
- removed U6, U8: LM25180QNGURQ1, FSAE-footprints:NGU0008C
- added C1: 1uF, Capacitor_SMD:C_0603_1608Metric, F.Cu at (-169.0, -24.3)
- added C10: 0.1uF, Capacitor_SMD:C_0603_1608Metric, F.Cu at (258.0, 76.8)
- added C100: 2.2uF, Capacitor_SMD:C_0603_1608Metric, F.Cu at (594.2, 176.5)
- added C101: 2.2uF, Capacitor_SMD:C_0603_1608Metric, F.Cu at (594.2, 179.0)
- added C102: 2.2uF, Capacitor_SMD:C_0603_1608Metric, F.Cu at (594.2, 181.5)
- added C103: 100nF, Capacitor_SMD:C_0603_1608Metric, F.Cu at (594.2, 184.0)
- added C104: 100nF, Capacitor_SMD:C_0603_1608Metric, F.Cu at (594.2, 186.5)
- added C105: 100nF, Capacitor_SMD:C_0603_1608Metric, F.Cu at (594.2, 189.0)
- added C106: 10pF, Capacitor_SMD:C_0402_1005Metric, F.Cu at (586.3, 203.6)
- added C107: 10pF, Capacitor_SMD:C_0402_1005Metric, F.Cu at (586.3, 205.5)
- added C108: 100nF, Capacitor_SMD:C_0603_1608Metric, F.Cu at (594.2, 191.6)
- added C109: 2.2uF, Capacitor_SMD:C_0603_1608Metric, F.Cu at (598.2, 176.5)
- added C11: 1uF, Capacitor_SMD:C_0603_1608Metric, F.Cu at (258.0, 79.3)
- added C110: 2.2uF, Capacitor_SMD:C_0603_1608Metric, F.Cu at (598.2, 179.0)
- added C111: 100nF, Capacitor_SMD:C_0603_1608Metric, F.Cu at (598.2, 181.5)
- added C112: 2.2nF, Capacitor_SMD:C_0603_1608Metric, F.Cu at (-169.0, -21.8)
- added C113: 100nF, Capacitor_SMD:C_0603_1608Metric, F.Cu at (-273.8, 242.2)
- added C114: 100nF, Capacitor_SMD:C_0603_1608Metric, F.Cu at (-273.8, 244.8)
- added C115: 100nF, Capacitor_SMD:C_0603_1608Metric, F.Cu at (-273.8, 247.3)
- added C116: 100nF, Capacitor_SMD:C_0603_1608Metric, F.Cu at (-273.8, 249.8)
- added C117: 100nF, Capacitor_SMD:C_0603_1608Metric, F.Cu at (-273.8, 252.3)
- added C118: 100nF, Capacitor_SMD:C_0603_1608Metric, F.Cu at (-269.8, 239.7)
- added C119: 100nF, Capacitor_SMD:C_0603_1608Metric, F.Cu at (-269.8, 242.2)
- added C12: 100pF, Capacitor_SMD:C_0603_1608Metric_Pad1.08x0.95mm_HandSolder, F.Cu at (105.4, -117.5)
- added C120: 100nF, Capacitor_SMD:C_0603_1608Metric, F.Cu at (-269.8, 244.8)
- added C121: 100nF, Capacitor_SMD:C_0603_1608Metric, F.Cu at (-269.8, 247.3)
- added C122: 10uF, Capacitor_SMD:C_0603_1608Metric, F.Cu at (598.2, 184.0)
- added C13: EEH-ZS1H271UP, Capacitor_SMD:CP_Elec_10x10, F.Cu at (-73.9, -296.6)
- added C14: CL31B475KAHNNNE, Capacitor_SMD:C_1206_3216Metric, F.Cu at (-87.4, -319.4)
- added C15: 10pF, Capacitor_SMD:C_0402_1005Metric, F.Cu at (105.4, -115.5)
- added C16: 220nF, Capacitor_SMD:C_0603_1608Metric, F.Cu at (101.0, -93.7)
- added C17: 100pF, Capacitor_SMD:C_0402_1005Metric, F.Cu at (105.4, -113.5)
- added C18: 100pF, Capacitor_SMD:C_0402_1005Metric, F.Cu at (105.4, -111.6)
- added C19: 0.1uF, Capacitor_SMD:C_0603_1608Metric, F.Cu at (101.0, -91.2)
- added C2: 10uF, Capacitor_SMD:C_0805_2012Metric, F.Cu at (-179.7, -9.88)
- added C20: 1uF, Capacitor_SMD:C_0603_1608Metric, F.Cu at (101.0, -88.7)
- added C21: 100pF, Capacitor_SMD:C_0603_1608Metric_Pad1.08x0.95mm_HandSolder, F.Cu at (160.0, -149.4)
- added C22: EEH-ZS1H271UP, Capacitor_SMD:CP_Elec_10x10, F.Cu at (142.5, -135.4)
- added C23: CL31B475KAHNNNE, Capacitor_SMD:C_1206_3216Metric, F.Cu at (163.5, -119.1)
- added C24: 10pF, Capacitor_SMD:C_0402_1005Metric, F.Cu at (160.0, -147.4)
- added C25: 220nF, Capacitor_SMD:C_0603_1608Metric, F.Cu at (155.7, -125.6)
- added C26: 100pF, Capacitor_SMD:C_0402_1005Metric, F.Cu at (160.0, -145.4)
- added C27: 100pF, Capacitor_SMD:C_0402_1005Metric, F.Cu at (160.0, -143.5)
- added C28: 0.1uF, Capacitor_SMD:C_0603_1608Metric, F.Cu at (155.7, -123.1)
- added C29: 1uF, Capacitor_SMD:C_0603_1608Metric, F.Cu at (155.7, -120.6)
- added C3: 100pF, Capacitor_SMD:C_0603_1608Metric_Pad1.08x0.95mm_HandSolder, F.Cu at (182.5, 68.5)
- added C30: 100pF, Capacitor_SMD:C_0603_1608Metric_Pad1.08x0.95mm_HandSolder, F.Cu at (160.0, -113.9)
- added C31: EEH-ZS1H271UP, Capacitor_SMD:CP_Elec_10x10, F.Cu at (142.5, -99.9)
- added C32: CL31B475KAHNNNE, Capacitor_SMD:C_1206_3216Metric, F.Cu at (163.5, -83.7)
- added C33: 10pF, Capacitor_SMD:C_0402_1005Metric, F.Cu at (160.0, -112.0)
- added C34: 220nF, Capacitor_SMD:C_0603_1608Metric, F.Cu at (155.7, -90.2)
- added C35: 100pF, Capacitor_SMD:C_0402_1005Metric, F.Cu at (160.0, -110.0)
- added C36: 100pF, Capacitor_SMD:C_0402_1005Metric, F.Cu at (160.0, -108.0)
- added C37: 0.1uF, Capacitor_SMD:C_0603_1608Metric, F.Cu at (155.7, -87.6)
- added C38: 1uF, Capacitor_SMD:C_0603_1608Metric, F.Cu at (155.7, -85.1)
- added C39: 100pF, Capacitor_SMD:C_0603_1608Metric_Pad1.08x0.95mm_HandSolder, F.Cu at (160.0, -184.8)
- added C4: EEH-ZS1H271UP, Capacitor_SMD:CP_Elec_10x10, F.Cu at (301.5, 78.0)
- added C40: EEH-ZS1H271UP, Capacitor_SMD:CP_Elec_10x10, F.Cu at (142.5, -170.8)
- added C41: CL31B475KAHNNNE, Capacitor_SMD:C_1206_3216Metric, F.Cu at (163.5, -154.6)
- added C42: 10pF, Capacitor_SMD:C_0402_1005Metric, F.Cu at (160.0, -182.8)
- added C43: 220nF, Capacitor_SMD:C_0603_1608Metric, F.Cu at (155.7, -161.1)
- added C44: 100pF, Capacitor_SMD:C_0402_1005Metric, F.Cu at (160.0, -180.9)
- added C45: 100pF, Capacitor_SMD:C_0402_1005Metric, F.Cu at (160.0, -178.9)
- added C46: 0.1uF, Capacitor_SMD:C_0603_1608Metric, F.Cu at (155.7, -158.5)
- added C47: 1uF, Capacitor_SMD:C_0603_1608Metric, F.Cu at (155.7, -156.0)
- added C48: 100pF, Capacitor_SMD:C_0603_1608Metric_Pad1.08x0.95mm_HandSolder, F.Cu at (105.4, -152.9)
- added C49: EEH-ZS1H271UP, Capacitor_SMD:CP_Elec_10x10, F.Cu at (87.9, -138.9)
- added C5: CL31B475KAHNNNE, Capacitor_SMD:C_1206_3216Metric, F.Cu at (326.3, 77.8)
- added C50: CL31B475KAHNNNE, Capacitor_SMD:C_1206_3216Metric, F.Cu at (108.8, -122.7)
- added C51: 10pF, Capacitor_SMD:C_0402_1005Metric, F.Cu at (105.4, -151.0)
- added C52: 220nF, Capacitor_SMD:C_0603_1608Metric, F.Cu at (101.0, -129.2)
- added C53: 100pF, Capacitor_SMD:C_0402_1005Metric, F.Cu at (105.4, -149.0)
- added C54: 100pF, Capacitor_SMD:C_0402_1005Metric, F.Cu at (105.4, -147.0)
- added C55: 0.1uF, Capacitor_SMD:C_0603_1608Metric, F.Cu at (101.0, -126.7)
- added C56: 1uF, Capacitor_SMD:C_0603_1608Metric, F.Cu at (101.0, -124.2)
- added C57: EEH-ZS1H271UP, Capacitor_SMD:CP_Elec_10x10, F.Cu at (741.0, -383.5)
- added C58: CL31B475KAHNNNE, Capacitor_SMD:C_1206_3216Metric, F.Cu at (727.7, -399.4)
- added C59: 47nF, Capacitor_SMD:C_0603_1608Metric, F.Cu at (661.0, -418.9)
- added C6: 10pF, Capacitor_SMD:C_0402_1005Metric, F.Cu at (176.5, 84.5)
- added C60: 0,1uF, Capacitor_SMD:C_0603_1608Metric, F.Cu at (581.7, 119.3)
- added C61: 0,1uF, Capacitor_SMD:C_0603_1608Metric, F.Cu at (581.7, 121.8)
- added C62: 0,1uF, Capacitor_SMD:C_0603_1608Metric, F.Cu at (581.7, 124.3)
- added C63: 10uF, Capacitor_SMD:C_0805_2012Metric, F.Cu at (654.7, -402.7)
- added C64: 100nF, Capacitor_SMD:C_0603_1608Metric, F.Cu at (-277.9, 239.7)
- added C65: 100nF, Capacitor_SMD:C_0603_1608Metric, F.Cu at (-277.9, 242.2)
- added C66: 100nF, Capacitor_SMD:C_0603_1608Metric, F.Cu at (-277.9, 244.8)
- added C67: 100nF, Capacitor_SMD:C_0603_1608Metric, F.Cu at (-277.9, 247.3)
- added C68: 0,1uF, Capacitor_SMD:C_0603_1608Metric, F.Cu at (-277.9, 249.8)
- added C69: 0,1uF, Capacitor_SMD:C_0603_1608Metric, F.Cu at (-277.9, 252.3)
- added C7: 220nF, Capacitor_SMD:C_0603_1608Metric, F.Cu at (258.0, 74.3)
- added C70: 0,1uF, Capacitor_SMD:C_0603_1608Metric, F.Cu at (-273.8, 239.7)
- added C71: 2.2nF, Capacitor_SMD:C_0603_1608Metric, F.Cu at (-232.7, -17.5)
- added C72: 2.2nF, Capacitor_SMD:C_0603_1608Metric, F.Cu at (-232.7, -15.0)
- added C73: 2.2nF, Capacitor_SMD:C_0603_1608Metric, F.Cu at (-232.7, -12.5)
- added C74: 100nF, Capacitor_SMD:C_0603_1608Metric, F.Cu at (-232.7, -9.99)
- added C75: 100nF, Capacitor_SMD:C_0603_1608Metric, F.Cu at (-232.7, -7.48)
- added C76: 100nF, Capacitor_SMD:C_0603_1608Metric, F.Cu at (-232.7, -4.97)
- added C77: 220nF, Capacitor_SMD:C_0603_1608Metric, F.Cu at (540.8, 196.3)
- added C78: 220nF, Capacitor_SMD:C_0603_1608Metric, F.Cu at (540.8, 198.8)
- added C79: 220nF, Capacitor_SMD:C_0603_1608Metric, F.Cu at (540.8, 201.3)
- added C8: 100pF, Capacitor_SMD:C_0402_1005Metric, F.Cu at (262.3, 54.4)
- added C80: 220nF, Capacitor_SMD:C_0603_1608Metric, F.Cu at (540.8, 203.8)
- added C81: 10nF, Capacitor_SMD:C_0603_1608Metric, F.Cu at (583.0, 160.2)
- added C82: 10nF, Capacitor_SMD:C_0603_1608Metric, F.Cu at (583.0, 162.7)
- added C83: 10nF, Capacitor_SMD:C_0603_1608Metric, F.Cu at (583.0, 165.2)
- added C84: 10nF, Capacitor_SMD:C_0603_1608Metric, F.Cu at (583.0, 167.7)
- added C85: 10nF, Capacitor_SMD:C_0603_1608Metric, F.Cu at (583.0, 170.2)
- added C86: 100nF, Capacitor_SMD:C_0603_1608Metric, F.Cu at (618.0, 104.9)
- added C87: 100nF, Capacitor_SMD:C_0603_1608Metric, F.Cu at (618.0, 107.4)
- added C88: 100nF, Capacitor_SMD:C_0603_1608Metric, F.Cu at (618.0, 109.9)
- added C89: 100nF, Capacitor_SMD:C_0603_1608Metric, F.Cu at (618.0, 112.4)
- added C9: 100pF, Capacitor_SMD:C_0402_1005Metric, F.Cu at (262.3, 56.4)
- added C90: 10uF, Capacitor_SMD:C_0805_2012Metric, F.Cu at (580.0, 198.3)
- added C91: 10uF, Capacitor_SMD:C_0805_2012Metric, F.Cu at (580.0, 201.3)
- added C92: 100nF, Capacitor_SMD:C_0603_1608Metric, F.Cu at (590.2, 176.5)
- added C93: 100nF, Capacitor_SMD:C_0603_1608Metric, F.Cu at (590.2, 179.0)
- added C94: 100nF, Capacitor_SMD:C_0603_1608Metric, F.Cu at (590.2, 181.5)
- added C95: 100nF, Capacitor_SMD:C_0603_1608Metric, F.Cu at (590.2, 184.0)
- added C96: 10uF, Capacitor_SMD:C_0805_2012Metric, F.Cu at (580.0, 204.3)
- added C97: 100nF, Capacitor_SMD:C_0603_1608Metric, F.Cu at (590.2, 186.5)
- added C98: 100nF, Capacitor_SMD:C_0603_1608Metric, F.Cu at (590.2, 189.0)
- added C99: 2.2uF, Capacitor_SMD:C_0603_1608Metric, F.Cu at (590.2, 191.6)
- added D10: APT2012EC, LED_SMD:LED_0805_2012Metric, F.Cu at (325.7, 71.5)
- added D11: APT2012EC, LED_SMD:LED_0805_2012Metric, F.Cu at (325.7, 74.6)
- added D14: BAT54WS-7-F, Diode_SMD:D_SOD-323_HandSoldering, F.Cu at (109.4, -117.0)
- added D15: BZT52C2V7-TP, Diode_SMD:D_SOD-123, F.Cu at (102.0, -100.0)
- added D16: MMSZ5242B-7-F, Diode_SMD:D_SOD-123, F.Cu at (102.0, -96.7)
- added D17: SMDJ13A, Diode_SMD:D_SMC, F.Cu at (-61.6, -298.6)
- added D19: APT2012EC, LED_SMD:LED_0805_2012Metric, F.Cu at (-87.9, -322.6)
- added D2: APT2012EC, LED_SMD:LED_0805_2012Metric, F.Cu at (108.2, -223.3)
- added D20: STTH112A, Diode_SMD:D_SOD-323F, F.Cu at (162.4, -139.8)
- added D21: STTH112A, Diode_SMD:D_SOD-323F, F.Cu at (162.4, -136.9)
- added D22: BAT54WS-7-F, Diode_SMD:D_SOD-323_HandSoldering, F.Cu at (164.0, -148.9)
- added D25: SMDJ13A, Diode_SMD:D_SMC, F.Cu at (154.8, -137.4)
- added D26: APT2012EC, LED_SMD:LED_0805_2012Metric, F.Cu at (162.9, -125.3)
- added D27: APT2012EC, LED_SMD:LED_0805_2012Metric, F.Cu at (162.9, -122.3)
- added D28: STTH112A, Diode_SMD:D_SOD-323F, F.Cu at (162.4, -104.4)
- added D3: APT2012EC, LED_SMD:LED_0805_2012Metric, F.Cu at (108.2, -220.3)
- added D30: BAT54WS-7-F, Diode_SMD:D_SOD-323_HandSoldering, F.Cu at (164.0, -113.4)
- added D31: BZT52C2V7-TP, Diode_SMD:D_SOD-123, F.Cu at (156.6, -96.4)
- added D32: MMSZ5242B-7-F, Diode_SMD:D_SOD-123, F.Cu at (156.6, -93.1)
- added D33: SMDJ13A, Diode_SMD:D_SMC, F.Cu at (154.8, -102.0)
- added D36: STTH112A, Diode_SMD:D_SOD-323F, F.Cu at (162.4, -175.3)
- added D37: STTH112A, Diode_SMD:D_SOD-323F, F.Cu at (162.4, -172.3)
- added D38: BAT54WS-7-F, Diode_SMD:D_SOD-323_HandSoldering, F.Cu at (164.0, -184.3)
- added D39: BZT52C2V7-TP, Diode_SMD:D_SOD-123, F.Cu at (156.6, -167.3)
- added D4: STTH112A, Diode_SMD:D_SOD-323F, F.Cu at (182.5, 61.0)
- added D41: SMDJ13A, Diode_SMD:D_SMC, F.Cu at (154.8, -172.9)
- added D42: APT2012EC, LED_SMD:LED_0805_2012Metric, F.Cu at (162.9, -160.8)
- added D43: APT2012EC, LED_SMD:LED_0805_2012Metric, F.Cu at (162.9, -157.7)
- added D44: STTH112A, Diode_SMD:D_SOD-323F, F.Cu at (107.7, -143.4)
- added D47: BZT52C2V7-TP, Diode_SMD:D_SOD-123, F.Cu at (102.0, -135.4)
- added D48: MMSZ5242B-7-F, Diode_SMD:D_SOD-123, F.Cu at (102.0, -132.1)
- added D49: SMDJ13A, Diode_SMD:D_SMC, F.Cu at (100.1, -141.0)
- added D5: STTH112A, Diode_SMD:D_SOD-323F, F.Cu at (186.0, 61.0)
- added D50: APT2012EC, LED_SMD:LED_0805_2012Metric, F.Cu at (108.2, -128.9)
- added D52: SMDJ13A, Diode_SMD:D_SMC, F.Cu at (739.5, -397.5)
- added D53: DFLZ24Q-7, Diode_SMD:D_PowerDI-123, F.Cu at (661.0, -416.5)
- added D54: 1N4148WS-Q, Diode_SMD:D_SOD-323F, F.Cu at (671.0, -415.7)
- added D55: VS-10MQ100NTRPBF, Diode_SMD:D_SMA, F.Cu at (663.0, -405.3)
- added D58: PESD2CANFD24LT-QR, Package_TO_SOT_SMD:SOT-23, F.Cu at (605.4, 126.7)
- added D59: PESD2CANFD24LT-QR, Package_TO_SOT_SMD:SOT-23, F.Cu at (605.4, 131.2)
- added D6: BAT54WS-7-F, Diode_SMD:D_SOD-323_HandSoldering, F.Cu at (183.0, 66.5)
- added D60: APT2012EC, LED_SMD:LED_0805_2012Metric, F.Cu at (575.6, 198.3)
- added D61: APT2012EC, LED_SMD:LED_0805_2012Metric, F.Cu at (575.6, 201.3)
- added D63: APT2012EC, LED_SMD:LED_0805_2012Metric, F.Cu at (-175.2, -9.87)
- added D64: SMDJ13A, Diode_SMD:D_SMC, F.Cu at (-176.4, -21.7)
- added D9: SMDJ13A, Diode_SMD:D_SMC, F.Cu at (311.0, 53.0)
- added FB1: 220 Ohms, Inductor_SMD:L_01005_0402Metric_Pad0.57x0.30mm_HandSolder, F.Cu at (591.2, 193.8)
- added FB2: 60 Ohm, Inductor_SMD:L_01005_0402Metric_Pad0.57x0.30mm_HandSolder, F.Cu at (591.2, 195.5)
- added J1: IHL0212D1509, NuevoGui:CONN5_05D1509_XPR, F.Cu at (213.5, 89.0)
- added J10: 430450414, Snapeda:CONN_SD-43045-005_04_MOL, F.Cu at (610.3, 110.8)
- added J11: 430450414, Snapeda:CONN_SD-43045-005_04_MOL, F.Cu at (610.3, 121.2)
- added J12: 348268125, Snapeda:CONN_SD-34826-001_12_MOL, F.Cu at (577.8, 139.5)
- added J2: IHL0212D1509, NuevoGui:CONN5_05D1509_XPR, F.Cu at (-76.0, -308.5)
- added J3: IHL0212D1509, NuevoGui:CONN5_05D1509_XPR, F.Cu at (140.4, -147.3)
- added J4: IHL0212D1509, NuevoGui:CONN5_05D1509_XPR, F.Cu at (140.4, -111.9)
- added J5: IHL0212D1509, NuevoGui:CONN5_05D1509_XPR, F.Cu at (140.4, -182.8)
- added J6: IHL0212D1509, NuevoGui:CONN5_05D1509_XPR, F.Cu at (85.7, -150.9)
- added J7: GT8E-5P-2H(55), NuevoGui:HRS_GT8E-5P-2H_55_, F.Cu at (-112.0, -88.5)
- added J8: 20021521-00010T1LF, Snapeda:AMPHENOL_20021521-00010T1LF, F.Cu at (613.7, 140.4)
- added L1: MLZ2012N6R8LT000, Inductor_SMD:L_0805_2012Metric, F.Cu at (326.6, 50.8)
- added L2: MLZ2012N6R8LT000, Inductor_SMD:L_0805_2012Metric, F.Cu at (-52.7, -307.2)
- added L3: MLZ2012N6R8LT000, Inductor_SMD:L_0805_2012Metric, F.Cu at (163.7, -146.0)
- added L4: MLZ2012N6R8LT000, Inductor_SMD:L_0805_2012Metric, F.Cu at (163.7, -110.6)
- added L5: MLZ2012N6R8LT000, Inductor_SMD:L_0805_2012Metric, F.Cu at (163.7, -181.5)
- added L6: MLZ2012N6R8LT000, Inductor_SMD:L_0805_2012Metric, F.Cu at (109.1, -149.6)
- added L7: MLZ2012N6R8LT000, Inductor_SMD:L_0805_2012Metric, F.Cu at (739.6, -406.0)
- added PS1: TES_1-1211, Snapeda:CONV_TES_1-1211, F.Cu at (-287.5, 245.4)
- added R10: 5.1, Resistor_SMD:R_1206_3216Metric, F.Cu at (213.7, 65.0)
- added R100: 100k, Resistor_SMD:R_0805_2012Metric, F.Cu at (-284.1, 234.1)
- added R101: 100k, Resistor_SMD:R_0805_2012Metric, F.Cu at (-284.1, 237.0)
- added R102: 1k13, Resistor_SMD:R_0805_2012Metric, F.Cu at (-279.7, 216.3)
- added R103: 1k13, Resistor_SMD:R_0805_2012Metric, F.Cu at (-279.7, 219.3)
- added R104: 1k13, Resistor_SMD:R_0805_2012Metric, F.Cu at (-279.7, 222.2)
- added R105: 1k13, Resistor_SMD:R_0805_2012Metric, F.Cu at (-279.7, 225.2)
- added R106: 3k9, Resistor_SMD:R_0805_2012Metric, F.Cu at (-279.7, 228.2)
- added R107: 3k9, Resistor_SMD:R_0805_2012Metric, F.Cu at (-279.7, 231.1)
- added R108: 3k9, Resistor_SMD:R_0805_2012Metric, F.Cu at (-279.7, 234.1)
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Connections:
- D1 pad 1: Net-(D1-K) -> GND1
- D1 pad 2: Net-(D1-A) -> /pcb_potencia/GD_FLT
- D12 pad 1: /Gate_Driver/GDsupply1/Colector -> /pcb_potencia/Gate_Driver/GDsupply1/Colector
- D18 pad 1: Net-(D17-K) -> /pcb_potencia/Gate_Driver/GDsupply1/-8V
- D23 pad 1: /Gate_Driver/GDsupply2/Colector -> Net-(D23-K)
- D23 pad 2: Net-(D23-A) -> Net-(D21-A)
- D24 pad 1: Net-(D23-A) -> /pcb_potencia/Gate_Driver/GDsupply2/DESAT
- D24 pad 2: Net-(D24-A) -> /pcb_potencia/Gate_Driver/GDsupply2/ISO_GND
- D34 pad 1: /Gate_Driver/GDsupply3/Colector -> /pcb_potencia/Gate_Driver/GDsupply3/-8V
- D35 pad 1: Net-(D34-A) -> /pcb_potencia/Gate_Driver/GDsupply3/ISO_GND
- D40 pad 1: Net-(D39-K) -> /pcb_potencia/Gate_Driver/GDsupply4/DESAT
- D40 pad 2: Net-(D40-A) -> /pcb_potencia/Gate_Driver/GDsupply4/ISO_GND
- D45 pad 1: /Gate_Driver/GDsupply4/Colector -> Net-(D44-A)
- D46 pad 1: Net-(D45-A) -> /pcb_potencia/Gate_Driver/GDsupply5/DESAT
- D46 pad 2: Net-(D46-A) -> /pcb_potencia/Gate_Driver/GDsupply5/ISO_GND
- D51 pad 1: Net-(D50-K) -> /pcb_potencia/Gate_Driver/GDsupply5/ISO_GND
- D56 pad 1: /Gate_Driver/GDsupply5/Colector -> /pcb_logica/LogicSupply/5V_FB
- D56 pad 2: Net-(D56-A) -> GND
- D57 pad 1: Net-(D56-A) -> GND
- D62 pad 1: Net-(D61-K) -> GND
- D7 pad 1: /Gate_Driver/GDsupply/Colector -> Net-(D7-K)
- D7 pad 2: Net-(D7-A) -> Net-(D5-A)
- D8 pad 1: Net-(D7-A) -> /pcb_potencia/Gate_Driver/GDsupply/DESAT
- D8 pad 2: Net-(D8-A) -> /pcb_potencia/Gate_Driver/GDsupply/ISO_GND
- T1 pad 1: /Gate_Driver/15V -> Net-(D52-A1)
- T1 pad 2: (no net) -> Net-(D54-A)
- T1 pad 3: (no net) -> GND
- T1 pad 4: Net-(D1-A) -> Net-(D55-A)
- T1 pad 5: Net-(D3-A) -> (no net)
- T1 pad 6: /Gate_Driver/GDsupply/ISO_GND -> (no net)
- T1 pad 7: /Gate_Driver/GDsupply/ISO_GND -> (no net)
- T1 pad 8: Net-(D41-K) -> (no net)
- U1 pad 1: Net-(U1-AIN) -> GND1
- U1 pad 10: /Gate_Driver/C1_In_neg -> (no net)
- U1 pad 11: /Gate_Driver/C1_In_pos -> (no net)
- U1 pad 12: /Gate_Driver/RDY -> (no net)
- U1 pad 13: /Gate_Driver/~FLT -> (no net)
- U1 pad 14: /Gate_Driver/Reset -> (no net)
- U1 pad 15: /Gate_Driver/3,3V -> (no net)
- U1 pad 2: /Gate_Driver/GDsupply/DESAT -> Net-(U1-DVDT)
- U1 pad 3: /Gate_Driver/GDsupply/ISO_GND -> Net-(U1-EN/UVLO)
- U1 pad 4: /Gate_Driver/GDsupply/ISO_GND -> +12VA
- U1 pad 5: /Gate_Driver/GDsupply/+15V -> +12VF
- U1 pad 6: Net-(U1-OUTL) -> /pcb_potencia/12V_Filtrada/Led_12V_Ok
- U1 pad 7: /Gate_Driver/GDsupply/Gate -> Net-(U1-ILM)
- U1 pad 8: /Gate_Driver/GDsupply/-8V -> Net-(U1-OVCSEL)
- U1 pad 9: GND -> GND1
- U10 pad 1: Net-(D51-A) -> Net-(U10-AIN)
- U10 pad 2: Net-(U10-FB) -> /pcb_potencia/Gate_Driver/GDsupply4/DESAT
- U10 pad 3: /Gate_Driver/15V -> /pcb_potencia/Gate_Driver/GDsupply4/ISO_GND
- U10 pad 4: Net-(U10-EN_UVLO) -> /pcb_potencia/Gate_Driver/GDsupply4/ISO_GND
- U10 pad 5: Net-(U10-SS_BIAS) -> /pcb_potencia/Gate_Driver/GDsupply4/+15V
- U10 pad 7: Net-(U10-RSET) -> /pcb_potencia/Gate_Driver/GDsupply4/Gate
- U10 pad 8: GND -> /pcb_potencia/Gate_Driver/GDsupply4/-8V
- U10 pad 9: GND -> GND1
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Other:
- board outline added: 258 x 242 mm

Commit message: Un par de cosas mas
Parts:
- removed C13, C22, C31, C4, C40, C49, C57: EEH-ZS1H271UP, Capacitor_SMD:CP_Elec_10x10
- removed C14, C23, C32, C41, C5, C50: CL31B475KAHNNNE, Capacitor_SMD:C_1206_3216Metric
- removed D10, D11, D18, D19, D26, D27, D34, D35, D42, D43, D50, D51: APT2012EC, LED_SMD:LED_0805_2012Metric
- removed D17, D25, D33, D41, D49, D9: SMDJ13A, Diode_SMD:D_SMC
- removed J1, J2, J3, J4, J5, J6: IHL0212D1509, NuevoGui:CONN5_05D1509_XPR
- removed L1, L2, L3, L4, L5, L6: MLZ2012N6R8LT000, Inductor_SMD:L_0805_2012Metric
- removed R14, R25, R36, R47, R58, R69: 6k8, Resistor_SMD:R_0402_1005Metric
- removed R16, R27, R38, R49, R60, R71: 15k, Resistor_SMD:R_0402_1005Metric
- added C123: 10 uF, Capacitor_SMD:C_1206_3216Metric, F.Cu at (199.9, 357.9)
- added C124: 47nF, Capacitor_SMD:C_0402_1005Metric_Pad0.74x0.62mm_HandSolder, F.Cu at (211.9, 360.1)
- added C125: 10uF, Capacitor_SMD:C_0805_2012Metric, F.Cu at (208.0, 344.4)
- added C126: 10 uF, Capacitor_SMD:C_1206_3216Metric, F.Cu at (266.6, 357.9)
- added C127: 47nF, Capacitor_SMD:C_0402_1005Metric_Pad0.74x0.62mm_HandSolder, F.Cu at (278.6, 360.1)
- added C128: 10uF, Capacitor_SMD:C_0805_2012Metric, F.Cu at (274.7, 344.4)
- added C129: 10 uF, Capacitor_SMD:C_1206_3216Metric, F.Cu at (233.3, 357.9)
- added C130: 47nF, Capacitor_SMD:C_0402_1005Metric_Pad0.74x0.62mm_HandSolder, F.Cu at (245.2, 360.1)
- added C131: 10uF, Capacitor_SMD:C_0805_2012Metric, F.Cu at (241.4, 344.4)
- added C132: 10 uF, Capacitor_SMD:C_1206_3216Metric, F.Cu at (233.3, 390.3)
- added C133: 47nF, Capacitor_SMD:C_0402_1005Metric_Pad0.74x0.62mm_HandSolder, F.Cu at (245.2, 392.5)
- added C134: 10uF, Capacitor_SMD:C_0805_2012Metric, F.Cu at (241.4, 376.8)
- added C135: 10 uF, Capacitor_SMD:C_1206_3216Metric, F.Cu at (199.9, 390.3)
- added C136: 47nF, Capacitor_SMD:C_0402_1005Metric_Pad0.74x0.62mm_HandSolder, F.Cu at (211.9, 392.5)
- added C137: 10uF, Capacitor_SMD:C_0805_2012Metric, F.Cu at (208.0, 376.8)
- added C138: 10 uF, Capacitor_SMD:C_1206_3216Metric, F.Cu at (199.3, 40.8)
- added C139: 47nF, Capacitor_SMD:C_0402_1005Metric_Pad0.74x0.62mm_HandSolder, F.Cu at (197.6, 40.0)
- added C140: 10uF, Capacitor_SMD:C_0805_2012Metric, F.Cu at (197.5, 62.1)
- added C141: 22uF, Capacitor_SMD:C_0805_2012Metric, F.Cu at (208.0, 347.4)
- added C142: 22uF, Capacitor_SMD:C_0805_2012Metric, F.Cu at (274.7, 347.4)
- added C143: 22uF, Capacitor_SMD:C_0805_2012Metric, F.Cu at (241.4, 347.4)
- added C144: 22uF, Capacitor_SMD:C_0805_2012Metric, F.Cu at (241.4, 379.8)
- added C145: 22uF, Capacitor_SMD:C_0805_2012Metric, F.Cu at (208.0, 379.8)
- added C146: 22uF, Capacitor_SMD:C_0805_2012Metric, F.Cu at (188.0, 62.1)
- added C151: 100nF, Capacitor_SMD:C_0402_1005Metric, F.Cu at (226.0, 349.8)
- added C152: 100nF, Capacitor_SMD:C_0402_1005Metric, F.Cu at (292.7, 349.8)
- added C153: 100nF, Capacitor_SMD:C_0402_1005Metric, F.Cu at (259.3, 349.8)
- added C154: 100nF, Capacitor_SMD:C_0402_1005Metric, F.Cu at (259.3, 382.1)
- added C155: 100nF, Capacitor_SMD:C_0402_1005Metric, F.Cu at (226.0, 382.1)
- added C156: 100nF, Capacitor_SMD:C_0402_1005Metric, F.Cu at (201.0, 40.6)
- added C157: 10uF, Capacitor_SMD:C_0805_2012Metric, F.Cu at (208.0, 350.4)
- added C158: 10uF, Capacitor_SMD:C_0805_2012Metric, F.Cu at (274.7, 350.4)
- added C159: 10uF, Capacitor_SMD:C_0805_2012Metric, F.Cu at (241.4, 350.4)
- added C160: 10uF, Capacitor_SMD:C_0805_2012Metric, F.Cu at (241.4, 382.8)
- added C161: 10uF, Capacitor_SMD:C_0805_2012Metric, F.Cu at (208.0, 382.8)
- added C162: 10uF, Capacitor_SMD:C_0805_2012Metric, F.Cu at (194.7, 61.4)
- added C163: 22uF, Capacitor_SMD:C_0805_2012Metric, F.Cu at (208.0, 353.4)
- added C164: 22uF, Capacitor_SMD:C_0805_2012Metric, F.Cu at (274.7, 353.4)
- added C165: 22uF, Capacitor_SMD:C_0805_2012Metric, F.Cu at (241.4, 353.4)
- added C166: 22uF, Capacitor_SMD:C_0805_2012Metric, F.Cu at (241.4, 385.8)
- added C167: 22uF, Capacitor_SMD:C_0805_2012Metric, F.Cu at (208.0, 385.8)
- added C168: 22uF, Capacitor_SMD:C_0805_2012Metric, F.Cu at (190.8, 61.4)
- added D101: SDM1U100S1F-7, Diode_SMD:D_SOD-123F, F.Cu at (217.4, 356.7)
- added D102: SDM1U100S1F-7, Diode_SMD:D_SOD-123F, F.Cu at (284.1, 356.7)
- added D103: SDM1U100S1F-7, Diode_SMD:D_SOD-123F, F.Cu at (250.8, 356.7)
- added D104: SDM1U100S1F-7, Diode_SMD:D_SOD-123F, F.Cu at (250.8, 389.1)
- added D105: SDM1U100S1F-7, Diode_SMD:D_SOD-123F, F.Cu at (217.4, 389.1)
- added D106: SDM1U100S1F-7, Diode_SMD:D_SOD-123F, F.Cu at (186.2, 57.8)
- added D65: BZT52C18-7-F, Diode_SMD:D_SOD-123, F.Cu at (200.0, 351.2)
- added D66: DFLZ24Q-7, Diode_SMD:D_PowerDI-123, F.Cu at (225.4, 338.3)
- added D67: 1N4148WS-Q, Diode_SMD:D_SOD-323F, F.Cu at (216.8, 350.2)
- added D68: SDM1U100S1F-7, Diode_SMD:D_SOD-123F, F.Cu at (217.4, 353.4)
- added D69: BZT52C18-7-F, Diode_SMD:D_SOD-123, F.Cu at (266.7, 351.2)
- added D71: BZT52C18-7-F, Diode_SMD:D_SOD-123, F.Cu at (233.4, 351.2)
- added D72: DFLZ24Q-7, Diode_SMD:D_PowerDI-123, F.Cu at (292.1, 338.3)
- added D73: 1N4148WS-Q, Diode_SMD:D_SOD-323F, F.Cu at (283.5, 350.2)
- added D74: SDM1U100S1F-7, Diode_SMD:D_SOD-123F, F.Cu at (284.1, 353.4)
- added D75: BZT52C18-7-F, Diode_SMD:D_SOD-123, F.Cu at (233.4, 383.6)
- added D77: BZT52C18-7-F, Diode_SMD:D_SOD-123, F.Cu at (200.0, 383.6)
- added D78: DFLZ24Q-7, Diode_SMD:D_PowerDI-123, F.Cu at (258.8, 338.3)
- added D79: 1N4148WS-Q, Diode_SMD:D_SOD-323F, F.Cu at (250.2, 350.2)
- added D80: SDM1U100S1F-7, Diode_SMD:D_SOD-123F, F.Cu at (250.8, 353.4)
- added D81: BZT52C18-7-F, Diode_SMD:D_SOD-123, F.Cu at (195.3, 59.2)
- added D83: BZT52B8V2-E3-08, Diode_SMD:D_SOD-123, F.Cu at (200.0, 354.6)
- added D84: DFLZ24Q-7, Diode_SMD:D_PowerDI-123, F.Cu at (258.8, 370.7)
- added D85: 1N4148WS-Q, Diode_SMD:D_SOD-323F, F.Cu at (250.2, 382.6)
- added D86: SDM1U100S1F-7, Diode_SMD:D_SOD-123F, F.Cu at (250.8, 385.8)
- added D87: BZT52B8V2-E3-08, Diode_SMD:D_SOD-123, F.Cu at (266.7, 354.6)
- added D89: BZT52B8V2-E3-08, Diode_SMD:D_SOD-123, F.Cu at (233.4, 354.6)
- added D90: DFLZ24Q-7, Diode_SMD:D_PowerDI-123, F.Cu at (225.4, 370.7)
- added D91: 1N4148WS-Q, Diode_SMD:D_SOD-323F, F.Cu at (216.8, 382.6)
- added D92: SDM1U100S1F-7, Diode_SMD:D_SOD-123F, F.Cu at (217.4, 385.8)
- added D93: BZT52B8V2-E3-08, Diode_SMD:D_SOD-123, F.Cu at (233.4, 387.0)
- added D95: BZT52B8V2-E3-08, Diode_SMD:D_SOD-123, F.Cu at (200.0, 387.0)
- added D96: DFLZ24Q-7, Diode_SMD:D_PowerDI-123, F.Cu at (195.4, 45.8)
- added D97: 1N4148WS-Q, Diode_SMD:D_SOD-323F, F.Cu at (191.1, 46.2)
- added D98: SDM1U100S1F-7, Diode_SMD:D_SOD-123F, F.Cu at (199.1, 57.8)
- added D99: BZT52B8V2-E3-08, Diode_SMD:D_SOD-123, F.Cu at (190.2, 59.1)
- added R178: 246k, Resistor_SMD:R_0402_1005Metric, F.Cu at (204.3, 349.8)
- added R196: 37k, Resistor_SMD:R_0402_1005Metric, F.Cu at (204.3, 351.8)
- added R197: 12k1, Resistor_SMD:R_0402_1005Metric, F.Cu at (204.3, 353.8)
- added R198: 110k, Resistor_SMD:R_0402_1005Metric, F.Cu at (204.3, 355.8)
- added R199: 154k, Resistor_SMD:R_0402_1005Metric_Pad0.72x0.64mm_HandSolder, F.Cu at (211.9, 358.2)
- added R201: 246k, Resistor_SMD:R_0402_1005Metric, F.Cu at (271.0, 349.8)
- added R202: 37k, Resistor_SMD:R_0402_1005Metric, F.Cu at (271.0, 351.8)
- added R203: 12k1, Resistor_SMD:R_0402_1005Metric, F.Cu at (271.0, 353.8)
- added R204: 110k, Resistor_SMD:R_0402_1005Metric, F.Cu at (271.0, 355.8)
- added R205: 154k, Resistor_SMD:R_0402_1005Metric_Pad0.72x0.64mm_HandSolder, F.Cu at (278.6, 358.2)
- added R207: 246k, Resistor_SMD:R_0402_1005Metric, F.Cu at (237.7, 349.8)
- added R208: 37k, Resistor_SMD:R_0402_1005Metric, F.Cu at (237.7, 351.8)
- added R209: 12k1, Resistor_SMD:R_0402_1005Metric, F.Cu at (237.7, 353.8)
- added R210: 110k, Resistor_SMD:R_0402_1005Metric, F.Cu at (237.7, 355.8)
- added R211: 154k, Resistor_SMD:R_0402_1005Metric_Pad0.72x0.64mm_HandSolder, F.Cu at (245.2, 358.2)
- added R213: 246k, Resistor_SMD:R_0402_1005Metric, F.Cu at (237.7, 382.2)
- added R214: 37k, Resistor_SMD:R_0402_1005Metric, F.Cu at (237.7, 384.2)
- added R215: 12k1, Resistor_SMD:R_0402_1005Metric, F.Cu at (237.7, 386.2)
- added R216: 110k, Resistor_SMD:R_0402_1005Metric, F.Cu at (237.7, 388.2)
- added R217: 154k, Resistor_SMD:R_0402_1005Metric_Pad0.72x0.64mm_HandSolder, F.Cu at (245.2, 390.6)
- added R219: 246k, Resistor_SMD:R_0402_1005Metric, F.Cu at (204.3, 382.2)
- added R220: 37k, Resistor_SMD:R_0402_1005Metric, F.Cu at (204.3, 384.2)
- added R221: 12k1, Resistor_SMD:R_0402_1005Metric, F.Cu at (204.3, 386.2)
- added R222: 110k, Resistor_SMD:R_0402_1005Metric, F.Cu at (204.3, 388.2)
- added R223: 154k, Resistor_SMD:R_0402_1005Metric_Pad0.72x0.64mm_HandSolder, F.Cu at (211.9, 390.6)
- added R225: 246k, Resistor_SMD:R_0402_1005Metric, F.Cu at (196.0, 43.8)
- added R226: 37k, Resistor_SMD:R_0402_1005Metric, F.Cu at (197.6, 42.2)
- added R227: 12k1, Resistor_SMD:R_0402_1005Metric, F.Cu at (197.0, 38.2)
- added R228: 110k, Resistor_SMD:R_0402_1005Metric, F.Cu at (195.1, 38.2)
- added R229: 154k, Resistor_SMD:R_0402_1005Metric_Pad0.72x0.64mm_HandSolder, F.Cu at (193.9, 43.8)
- added T2: 750317595, Snapeda:WE-FLYTI_EP7_4436, F.Cu at (283.3, 336.7)
- added T3: 750317595, Snapeda:WE-FLYTI_EP7_4436, F.Cu at (250.0, 336.7)
- added T4: 750317595, Snapeda:WE-FLYTI_EP7_4436, F.Cu at (250.0, 369.1)
- added T5: 750317595, Snapeda:WE-FLYTI_EP7_4436, F.Cu at (216.6, 369.1)
- added T6: 750317595, Snapeda:WE-FLYTI_EP7_4436, F.Cu at (192.7, 52.5)
- added TP53: TestPoint, TestPoint:TestPoint_Pad_D2.0mm, F.Cu at (222.2, 353.7)
- added TP54: TestPoint, TestPoint:TestPoint_Pad_D2.0mm, F.Cu at (288.9, 353.7)
- added TP55: TestPoint, TestPoint:TestPoint_Pad_D2.0mm, F.Cu at (255.5, 353.7)
- added TP56: TestPoint, TestPoint:TestPoint_Pad_D2.0mm, F.Cu at (255.5, 386.1)
- added TP57: TestPoint, TestPoint:TestPoint_Pad_D2.0mm, F.Cu at (222.2, 386.1)
- added TP58: TestPoint, TestPoint:TestPoint_Pad_D2.0mm, F.Cu at (346.8, 24.4)
- added TP59: TestPoint, TestPoint:TestPoint_Pad_D2.0mm, F.Cu at (222.2, 357.8)
- added TP60: TestPoint, TestPoint:TestPoint_Pad_D2.0mm, F.Cu at (288.9, 357.8)
- added TP61: TestPoint, TestPoint:TestPoint_Pad_D2.0mm, F.Cu at (255.5, 357.8)
- added TP62: TestPoint, TestPoint:TestPoint_Pad_D2.0mm, F.Cu at (255.5, 390.2)
- added TP63: TestPoint, TestPoint:TestPoint_Pad_D2.0mm, F.Cu at (222.2, 390.2)
- added TP64: TestPoint, TestPoint:TestPoint_Pad_D2.0mm, F.Cu at (346.8, 28.4)
- added Te1: Trafo 30uH - 3:1, Snapeda:WE-FLYTI_EP7_4436, F.Cu at (762.0, 25.9)
- added U40: LM25180QNGURQ1, NuevoGui:NGU0008C, F.Cu at (225.2, 333.7)
- added U41: LM25180QNGURQ1, NuevoGui:NGU0008C, F.Cu at (291.9, 333.7)
- added U42: LM25180QNGURQ1, NuevoGui:NGU0008C, F.Cu at (258.5, 333.7)
- added U43: LM25180QNGURQ1, NuevoGui:NGU0008C, F.Cu at (258.6, 366.3)
- added U45: LM25180QNGURQ1, NuevoGui:NGU0008C, F.Cu at (225.2, 366.1)
- added U47: LM25180QNGURQ1, NuevoGui:NGU0008C, F.Cu at (194.9, 41.0)
- C1: value 1uF -> 10uF
- C16, C25, C34, C43, C52, C7: footprint Capacitor_SMD:C_0603_1608Metric -> Capacitor_SMD:C_0402_1005Metric
- C59: footprint Capacitor_SMD:C_0603_1608Metric -> Capacitor_SMD:C_0402_1005Metric_Pad0.74x0.62mm_HandSolder
- D55: value VS-10MQ100NTRPBF -> SDM1U100S1F-7; footprint Diode_SMD:D_SMA -> Diode_SMD:D_SOD-123F
- R15, R26, R37, R48, R59, R70: footprint Resistor_SMD:R_0805_2012Metric -> Resistor_SMD:R_0402_1005Metric
- R72: value 307k -> 246k
- R76: footprint Resistor_SMD:R_0603_1608Metric -> Resistor_SMD:R_0402_1005Metric_Pad0.72x0.64mm_HandSolder
- T1: value Trafo 30uH - 3:1 -> 750317595
- moved T1 878.7 mm to (216.6, 336.7)
- moved D1 625.1 mm to (271.7, 377.0)
- moved D2 625.1 mm to (271.7, 380.1)
- moved D3 625.1 mm to (271.7, 383.1)
- moved R3 625.1 mm to (275.9, 376.8)
- moved R4 625.1 mm to (275.9, 379.3)
- moved R5 625.1 mm to (275.9, 381.8)
- moved TH1 621.6 mm to (265.4, 377.3)
- moved D46 555.3 mm to (217.2, 392.3)
- moved C48 551.7 mm to (212.4, 388.3)
- moved D38 546.8 mm to (217.2, 359.9)
- moved C39 543.3 mm to (212.4, 355.9)
- moved TP27 542.7 mm to (281.9, 365.4)
- moved TP28 542.7 mm to (281.9, 369.4)
- moved TP29 542.7 mm to (281.9, 373.5)
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Connections:
- T1 pad 1: Net-(D52-A1) -> Net-(D67-A)
- T1 pad 2: Net-(D54-A) -> (no net)
- T1 pad 3: GND -> (no net)
- T1 pad 4: Net-(D55-A) -> +12VF
- T1 pad 5: (no net) -> Net-(D68-A)
- T1 pad 6: (no net) -> /pcb_potencia/Gate_Driver/GDsupply4/ISO_GND
- T1 pad 7: (no net) -> /pcb_potencia/Gate_Driver/GDsupply4/ISO_GND
- T1 pad 8: (no net) -> Net-(D101-K)
Other:
- board size 258 x 242 mm -> 18.8 x 2.4 mm
- copper layers 2 -> 4
- board text added: "1 -> Layer: Power Signal 2 -> Layer: Gnd 3 -> Layer: Power 4 -> Layer: Signal"
- board text added: "IPC‑2221, ΔT = 20 °C 1 -> Layer: 2 oz"

Commit message: Sigo con la placa padre
Parts:
- R110, R111, R112, R113: footprint Resistor_SMD:R_0402_1005Metric -> Resistor_SMD:R_0805_2012Metric
- moved TP12 625.0 mm to (598.5, 153.9)
- moved TP3 625.0 mm to (594.5, 153.9)
- moved U18 625.0 mm to (606.8, 158.3)
- moved PS1 598.8 mm to (549.7, 149.6)
- moved C66 587.3 mm to (570.1, 144.4)
- moved R118 587.3 mm to (572.5, 156.1)
- moved R119 587.3 mm to (572.5, 158.1)
- moved C121 587.3 mm to (578.1, 146.9)
- moved R124 587.3 mm to (575.4, 154.1)
- moved R128 587.3 mm to (575.4, 162.1)
- moved R132 587.3 mm to (578.3, 156.1)
- moved U19 561.4 mm to (536.6, 148.1)
- moved C116 448.7 mm to (432.4, 166.9)
- moved C12 410.8 mm to (147.9, -10.7)
- moved C132 410.8 mm to (135.4, -8.68)
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Connections:
- D12 pad 1: /pcb_potencia/Gate_Driver/GDsupply1/Colector -> /pcb_potencia/Gate_Driver/VCC_DC
- D20 pad 1: /pcb_potencia/Gate_Driver/GDsupply2/Colector -> /pcb_potencia/Gate_Driver/VCC_DC
- D4 pad 1: /pcb_potencia/Gate_Driver/GDsupply/Colector -> /pcb_potencia/Gate_Driver/VCC_DC
- U2 pad C1: /pcb_potencia/Gate_Driver/GDsupply/Colector -> /pcb_potencia/Gate_Driver/VCC_DC
- U2 pad C3: /pcb_potencia/Gate_Driver/GDsupply1/Colector -> /pcb_potencia/Gate_Driver/VCC_DC
- U2 pad C5: /pcb_potencia/Gate_Driver/GDsupply2/Colector -> /pcb_potencia/Gate_Driver/VCC_DC
- U2 pad E1: GNDPWR -> /pcb_potencia/Gate_Driver/MP_1
- U2 pad E2: /pcb_potencia/Gate_Driver/VCC_DC -> GNDPWR
- U2 pad E3: GNDPWR -> /pcb_potencia/Gate_Driver/MP_2
- U2 pad E4: /pcb_potencia/Gate_Driver/VCC_DC -> GNDPWR
- U2 pad E5: GNDPWR -> /pcb_potencia/Gate_Driver/MP_3
- U2 pad E6: /pcb_potencia/Gate_Driver/VCC_DC -> GNDPWR
Routing:
- net (no net): track 0.00 -> 0.54 mm

Commit message: Ordene los gate drivers
Parts:
- removed PS1: TES_1-1211, Snapeda:CONV_TES_1-1211
- added PS2: NTE1205MC-R, Snapeda:CONV_NTE1205MC-R, F.Cu at (142.4, 99.9)
- moved U19 543.3 mm to (-3.67, 90.2)
- moved C27 386.1 mm to (87.2, 2.21)
- moved C28 386.1 mm to (87.4, 9.90)
- moved R211 386.1 mm to (73.1, 12.6)
- moved R34 386.1 mm to (65.6, 0.27)
- moved TP61 386.1 mm to (83.4, 12.2)
- moved U42 386.1 mm to (86.4, -11.9)
- moved C129 386.1 mm to (61.2, 12.4)
- moved C130 386.1 mm to (73.1, 14.6)
- moved C153 386.1 mm to (87.2, 4.18)
- moved C25 386.1 mm to (87.4, 7.39)
- moved C26 386.1 mm to (87.2, 0.24)
- moved C29 386.1 mm to (87.4, 12.4)
- moved D78 386.1 mm to (86.7, -7.28)
- moved D79 386.1 mm to (78.1, 4.66)
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Other:
- board size 18.8 x 2.4 mm -> 171.2 x 137.4 mm

Commit message: Casi todo padre
Parts:
- removed C33, C42, C51: 10pF, Capacitor_SMD:C_0402_1005Metric
- removed PS2: NTE1205MC-R, Snapeda:CONV_NTE1205MC-R
- removed R44, R55, R66: 10, Resistor_SMD:R_0402_1005Metric
- added U3: R1S12-1205/HP, NuevoGui:SMD12_15.24X10.7X6.7_SINGLE&slash_DUAL_RCP-L, F.Cu at (143.1, 98.6)
- C68, C69: footprint Capacitor_SMD:C_0603_1608Metric -> Capacitor_SMD:C_0805_2012Metric
- moved TP1 474.7 mm to (405.4, 112.8)
- moved TP13 474.7 mm to (413.5, 116.9)
- moved TP14 474.7 mm to (417.6, 112.8)
- moved TP15 474.7 mm to (417.6, 116.9)
- moved TP2 474.7 mm to (405.4, 116.9)
- moved TP4 474.7 mm to (409.5, 116.9)
- moved R130 469.0 mm to (425.6, 121.9)
- moved R129 469.0 mm to (425.6, 119.9)
- moved C1 465.6 mm to (431.0, 132.2)
- moved C112 465.6 mm to (431.0, 134.7)
- moved C2 465.6 mm to (420.4, 146.7)
- moved D64 465.6 mm to (423.6, 134.8)
- moved R193 465.6 mm to (431.0, 137.2)
- moved D63 465.6 mm to (424.8, 146.7)
- moved R190 465.6 mm to (434.1, 139.7)
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