File: PCB/Inverter/Primero_esquematico/g_driver.kicad_sch (KiCad schematic)
At the start: 17 parts, among them U2 FS950R08A6P2BBPSA1

Commit message: Sigo con la placa padre
Connections:
- net GDsupply/Colector is gone; now on net VCC_DC: U2.C1
- net GDsupply1/Colector is gone; now on net VCC_DC: U2.C3
- net GDsupply2/Colector is gone; now on net VCC_DC: U2.C5
- net GNDPWR: now also U2.E2, U2.E4, U2.E6; no longer U2.E1, U2.E3, U2.E5
- net MP_1: now also U2.E1
- net MP_2: now also U2.E3
- net MP_3: now also U2.E5
- net VCC_DC: no longer U2.E2, U2.E4, U2.E6

Commit message: correcciones
Parts:
- TP10: renamed from TP19; footprint TestPoint:TestPoint_Pad_D2.0mm -> TestPoint:TestPoint_Pad_D1.0mm
- TP11: renamed from TP20; footprint TestPoint:TestPoint_Pad_D2.0mm -> TestPoint:TestPoint_Pad_D1.0mm
- TP3: renamed from TP24; footprint TestPoint:TestPoint_Pad_D2.0mm -> TestPoint:TestPoint_Pad_D1.0mm
- TP4: renamed from TP16; footprint TestPoint:TestPoint_Pad_D2.0mm -> TestPoint:TestPoint_Pad_D1.0mm
- TP5: renamed from TP22; footprint TestPoint:TestPoint_Pad_D2.0mm -> TestPoint:TestPoint_Pad_D1.0mm
- TP6: renamed from TP17; footprint TestPoint:TestPoint_Pad_D2.0mm -> TestPoint:TestPoint_Pad_D1.0mm
- TP7: renamed from TP23; footprint TestPoint:TestPoint_Pad_D2.0mm -> TestPoint:TestPoint_Pad_D1.0mm
- TP8: renamed from TP18; footprint TestPoint:TestPoint_Pad_D2.0mm -> TestPoint:TestPoint_Pad_D1.0mm
- TP9: renamed from TP21; footprint TestPoint:TestPoint_Pad_D2.0mm -> TestPoint:TestPoint_Pad_D1.0mm
- renumbered D1 to D3, D2 to D4, D3 to D5, R3 to R6, R4 to R7, R5 to R8
