File: PCB/Inverter/Primero_esquematico/SensorTension.kicad_sch (KiCad schematic)
At the start: 86 parts, among them U17 AMC1301QDWVRQ1, U18 TLV9004QDRQ1, U19 ADR130BUJZ-REEL7, U37 AMC1301QDWVRQ1, U38 AMC1301QDWVRQ1, U39 AMC1301QDWVRQ1

Commit message: Casi todo padre
Parts:
- added U3: R1S12-1205/HP, NuevoGui:SMD12_15.24X10.7X6.7_SINGLE&slash_DUAL_RCP-L, symbol Snapeda:R1S12-1205_HP
- C68, C69: footprint Capacitor_SMD:C_0603_1608Metric -> Capacitor_SMD:C_0805_2012Metric
Connections:
- net +12VF: now also U3.1 (-VIN)
- net 5V_ISO: now also U3.8 (+VOUT)
- net GND1: now also U3.2 (+VIN)
- net GNDPWR: now also U3.5 (-VOUT)
Other:
- moved on the sheet: C68, C69

Commit message: correcciones
Parts:
- C113: renamed from C64; footprint Capacitor_SMD:C_0603_1608Metric -> Capacitor_SMD:C_0402_1005Metric
- C114: renamed from C65; footprint Capacitor_SMD:C_0603_1608Metric -> Capacitor_SMD:C_0402_1005Metric
- C115: renamed from C66; footprint Capacitor_SMD:C_0603_1608Metric -> Capacitor_SMD:C_0402_1005Metric
- C116: renamed from C67; footprint Capacitor_SMD:C_0603_1608Metric -> Capacitor_SMD:C_0402_1005Metric
- TP24: renamed from TP15; footprint TestPoint:TestPoint_Pad_D2.0mm -> TestPoint:TestPoint_Pad_D1.0mm
- TP25: renamed from TP1; footprint TestPoint:TestPoint_Pad_D2.0mm -> TestPoint:TestPoint_Pad_D1.0mm
- TP26: renamed from TP2; footprint TestPoint:TestPoint_Pad_D2.0mm -> TestPoint:TestPoint_Pad_D1.0mm
- TP27: renamed from TP14; footprint TestPoint:TestPoint_Pad_D2.0mm -> TestPoint:TestPoint_Pad_D1.0mm
- TP28: renamed from TP3; footprint TestPoint:TestPoint_Pad_D2.0mm -> TestPoint:TestPoint_Pad_D1.0mm
- TP29: renamed from TP12; footprint TestPoint:TestPoint_Pad_D2.0mm -> TestPoint:TestPoint_Pad_D1.0mm
- TP30: renamed from TP13; footprint TestPoint:TestPoint_Pad_D2.0mm -> TestPoint:TestPoint_Pad_D1.0mm
- TP31: renamed from TP4; footprint TestPoint:TestPoint_Pad_D2.0mm -> TestPoint:TestPoint_Pad_D1.0mm
- renumbered C116 to C105, C114 to C106, C117 to C107, C115 to C108, C118 to C109, C119 to C110, C121 to C111, C120 to C112, C113 to C117, C68 to C118, C70 to C119, C69 to C120, R78 to R100, R79 to R101, R80 to R102, R81 to R103, R82 to R104, R83 to R105, R84 to R106, R85 to R107, R86 to R108, R87 to R109, R88 to R110, R89 to R111, R90 to R112, R91 to R113, R92 to R114, R93 to R115, R94 to R116, R95 to R117, R96 to R118, R97 to R119, R98 to R120, R99 to R121, R100 to R122, R101 to R123, R102 to R124, R103 to R125, R104 to R126, R105 to R127, R106 to R128, R107 to R129, R108 to R130, R109 to R131, R110 to R132, R111 to R133, R112 to R134, R113 to R135, R114 to R136, R115 to R137, R122 to R138, R116 to R139, R117 to R140, R123 to R141, R118 to R142, R119 to R143, R124 to R144, R120 to R145, R121 to R146, R125 to R147, R126 to R148, R127 to R149, R128 to R150, R129 to R151, R130 to R152, R131 to R153, R132 to R154, R133 to R155, U37 to U17, U38 to U18, U39 to U19, U17 to U20, U18 to U21, U19 to U22, U3 to U23
Other:
- moved on the sheet: C109, R139, R140

Commit message: Algunos cambios
Parts:
- removed C118, C120: 0,1uF, Capacitor_SMD:C_0805_2012Metric, symbol Device:C_Small
- removed U23: R1S12-1205/HP, NuevoGui:SMD12_15.24X10.7X6.7_SINGLE&slash_DUAL_RCP-L, symbol Snapeda:R1S12-1205_HP
Connections:
- net +3.3VA renamed +3.3V_analog
Other:
- note removed: "El AMC1301 tiene una tension en la entrada maxima entre +-250mV (V+-V-)/V(MP_x)=0.25V/500V=5*10^-4 Con nuestra configuracion esa realacion es de 4.9*10^-4 La rama VINN debe tener la misma impedancia hacia el bias que la rama VINP, para que el modo común sea idéntico en ambas entradas y no se introduzca un offset diferencial."
