File: PCB/Inverter/Primero_esquematico/12V_Filtrada.kicad_sch (KiCad schematic)
At the start: 12 parts, among them U1 TPS259621DDAT

Commit message: Corregi cosas de la placa
Parts:
- renumbered C1 to C2, C2 to C3, C153 to C4, D1 to D2
Changed lines of the file:
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@@
 		(dnp no)
 		(fields_autoplaced yes)
-		(property "Reference" "#PWR02"
+		(property "Reference" "#PWR08"
 			(at 76.2 120.65 0)
 			(hide yes)
@@
 			(project "Primero_esquematico"
 				(path "/d930f486-f6ac-489c-907e-47f2cb34cf04/d101e913-ebd1-4e08-b728-82218f47123b/3145a225-26ad-4004-be15-8a1076c951ad"
-					(reference "#PWR02")
+					(reference "#PWR08")
 					(unit 1)
 				)
@@
 		(dnp no)
 		(fields_autoplaced yes)
-		(property "Reference" "#PWR01"
+		(property "Reference" "#PWR07"
 			(at 76.2 99.06 0)
 			(hide yes)
@@
 			(project "Primero_esquematico"
 				(path "/d930f486-f6ac-489c-907e-47f2cb34cf04/d101e913-ebd1-4e08-b728-82218f47123b/3145a225-26ad-4004-be15-8a1076c951ad"
-					(reference "#PWR01")
+					(reference "#PWR07")
 					(unit 1)
 				)
@@
 		(dnp no)
 		(fields_autoplaced yes)
-		(property "Reference" "D1"
+		(property "Reference" "D2"
 			(at 80.01 110.8074 90)
 			(show_name no)
@@
 			(project "Primero_esquematico"
 				(path "/d930f486-f6ac-489c-907e-47f2cb34cf04/d101e913-ebd1-4e08-b728-82218f47123b/3145a225-26ad-4004-be15-8a1076c951ad"
-					(reference "D1")
+					(reference "D2")
 					(unit 1)
 				)
@@
 		(in_pos_files yes)
 		(dnp no)
-		(property "Reference" "C2"
+		(property "Reference" "C3"
 			(at 196.85 114.3062 0)
 			(show_name no)
@@
 			(project "Primero_esquematico"
 				(path "/d930f486-f6ac-489c-907e-47f2cb34cf04/d101e913-ebd1-4e08-b728-82218f47123b/3145a225-26ad-4004-be15-8a1076c951ad"
-					(reference "C2")
+					(reference "C3")
 					(unit 1)
 				)
@@
 		(dnp no)
 		(fields_autoplaced yes)
-		(property "Reference" "#PWR06"
+		(property "Reference" "#PWR012"
 			(at 204.47 125.73 0)
 			(hide yes)
@@
 			(project "Primero_esquematico"
 				(path "/d930f486-f6ac-489c-907e-47f2cb34cf04/d101e913-ebd1-4e08-b728-82218f47123b/3145a225-26ad-4004-be15-8a1076c951ad"
-					(reference "#PWR06")
+					(reference "#PWR012")
 					(unit 1)
 				)
@@
 		(dnp no)
 		(fields_autoplaced yes)
-		(property "Reference" "#PWR04"
+		(property "Reference" "#PWR010"
 			(at 129.54 125.73 0)
 			(hide yes)
@@
 			(project "Primero_esquematico"
 				(path "/d930f486-f6ac-489c-907e-47f2cb34cf04/d101e913-ebd1-4e08-b728-82218f47123b/3145a225-26ad-4004-be15-8a1076c951ad"
-					(reference "#PWR04")
+					(reference "#PWR010")
 					(unit 1)
 				)
@@
 		(dnp no)
 		(fields_autoplaced yes)
-		(property "Reference" "C153"
+		(property "Reference" "C4"
 			(at 213.36 101.903 90)
 			(show_name no)
@@
 			(project "Primero_esquematico"
 				(path "/d930f486-f6ac-489c-907e-47f2cb34cf04/d101e913-ebd1-4e08-b728-82218f47123b/3145a225-26ad-4004-be15-8a1076c951ad"
-					(reference "C153")
+					(reference "C4")
 					(unit 1)
 				)
@@
 		(dnp no)
 		(fields_autoplaced yes)
-		(property "Reference" "#PWR03"
+		(property "Reference" "#PWR09"
 			(at 119.38 97.79 0)
 			(hide yes)
@@
 			(project "Primero_esquematico"
 				(path "/d930f486-f6ac-489c-907e-47f2cb34cf04/d101e913-ebd1-4e08-b728-82218f47123b/3145a225-26ad-4004-be15-8a1076c951ad"
-					(reference "#PWR03")
+					(reference "#PWR09")
 					(unit 1)
 				)
@@
 		(dnp no)
 		(fields_autoplaced yes)
-		(property "Reference" "#PWR08"
+		(property "Reference" "#PWR014"
 			(at 212.09 102.87 0)
 			(hide yes)
@@
 			(project "Primero_esquematico"
 				(path "/d930f486-f6ac-489c-907e-47f2cb34cf04/d101e913-ebd1-4e08-b728-82218f47123b/3145a225-26ad-4004-be15-8a1076c951ad"
-					(reference "#PWR08")
+					(reference "#PWR014")
 					(unit 1)
 				)
@@
 		(in_pos_files yes)
 		(dnp no)
-		(property "Reference" "C1"
+		(property "Reference" "C2"
 			(at 124.46 104.902 0)
 			(show_name no)
@@
 			(project "Primero_esquematico"
 				(path "/d930f486-f6ac-489c-907e-47f2cb34cf04/d101e913-ebd1-4e08-b728-82218f47123b/3145a225-26ad-4004-be15-8a1076c951ad"
-					(reference "C1")
+					(reference "C2")
 					(unit 1)
 				)
@@
 		(dnp no)
 		(fields_autoplaced yes)
-		(property "Reference" "#PWR05"
+		(property "Reference" "#PWR011"
 			(at 194.31 127 0)
 			(hide yes)
@@
 			(project "Primero_esquematico"
 				(path "/d930f486-f6ac-489c-907e-47f2cb34cf04/d101e913-ebd1-4e08-b728-82218f47123b/3145a225-26ad-4004-be15-8a1076c951ad"
-					(reference "#PWR05")
+					(reference "#PWR011")
 					(unit 1)
 				)
@@
 		(in_pos_files yes)
 		(dnp no)
-		(property "Reference" "#PWR07"
+		(property "Reference" "#PWR013"
 			(at 209.55 114.3 0)
 			(hide yes)
@@
 			(project "Primero_esquematico"
 				(path "/d930f486-f6ac-489c-907e-47f2cb34cf04/d101e913-ebd1-4e08-b728-82218f47123b/3145a225-26ad-4004-be15-8a1076c951ad"
-					(reference "#PWR07")
+					(reference "#PWR013")
 					(unit 1)
 				)
