File: PCB/Inverter/Primero_esquematico/GD_HS.kicad_sch (KiCad schematic)
At the start: 46 parts, among them T3 750317595, U7 LM25180QNGURQ1, U8 UCC21750QDWRQ1

Commit message: Solo falta routear algo
Parts:
- C38: value 47pF -> 56pF
Other:
- note added: "CASO SiC C_BLK · dV/dt = Ichg + (V_DD − V_Z − V) / R_ext V_ss = (V_DD − V_Z) + Ichg·R_ext τ = R_ext · C_BLK t_BLK = τ · ln[ V_ss / (V_ss − V_DESAT) ] Para nuestro caso el tiempo de blanking es 121ns"
- note added: "Caso IGBT t_BLK = C_BLK · V_DESAT / Ichg t_BLK = 1,05 us"
- note added: "LAS Ressitencias estas no iran en el diseño final solo para el caso de usar SiC"
Changed lines of the file:
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@@
 		)
 	)
+	(text "CASO SiC\nC_BLK · dV/dt = Ichg + (V_DD − V_Z − V) / R_ext\n\nV_ss = (V_DD − V_Z) + Ichg·R_ext\nτ = R_ext · C_BLK\nt_BLK = τ · ln[ V_ss / (V_ss − V_DESAT) ]\n\nPara nuestro caso el tiempo de blanking es 121ns"
+		(exclude_from_sim no)
+		(at 70.104 171.196 0)
+		(effects
+			(font
+				(size 1.27 1.27)
+				(thickness 0.254)
+				(bold yes)
+			)
+		)
+	)
 	(text "El Rst/En se suele juntar con +IN pero creo que no es obligatorio\nSi se junta con +IN revisar un tiempo que te limita el datasheet\n"
 		(exclude_from_sim no)
@@
 		)
 	)
+	(text "LAS Ressitencias estas no\niran en el diseño final\nsolo para el caso de usar SiC"
+		(exclude_from_sim no)
+		(at 83.566 101.092 0)
+		(effects
+			(font
+				(size 1.27 1.27)
+			)
+		)
+	)
 	(text "Ejemplo de Teaxas de su implementacion\nhttps://www.ti.com/lit/ug/sluuck0a/sluuck0a.pdf?ts=1781860744035"
 		(exclude_from_sim no)
@@
 		)
 	)
+	(text "Caso IGBT\nt_BLK = C_BLK · V_DESAT / Ichg\nt_BLK = 1,05 us"
+		(exclude_from_sim no)
+		(at 55.372 128.524 0)
+		(effects
+			(font
+				(size 1.27 1.27)
+				(thickness 0.254)
+				(bold yes)
+			)
+		)
+	)
 	(text "Frecuencia de corte en 2khz (Comentario para componentes colocados en APWM)\nEsto se coloca para pasar de un PWM a una señal ADC para monitorear tension\ny temperatura, esta frecuencia de corte es elevada para temperatura pero\nquiero usar menos variedad de componentes y no deberia cambiar\n"
 		(exclude_from_sim no)
-		(at 131.572 179.07 0)
+		(at 149.098 178.054 0)
 		(effects
 			(font
@@
 	(text "Esta etapa vigila la saturación del IGBT midiendo su tensión colector-emisor (V_CE) mientras está encendido:\n- Si el IGBT satura, V_CE es baja → OK.\n- Si V_CE queda alta con el IGBT en ON (desaturación) → sobrecorriente/cortocircuito → dispara el soft turn-off.\n- El C de blanking (47 pF) fija una ventana inicial tras el encendido en la que la protección se ignora, para dar tiempo a que el IGBT sature.\n- Si hay disparos falsos en el encendido → subir un poco el C (alarga el blanking).\n- No subirlo de más: alarga la ventana sin protección; un cortocircuito real debe detectarse antes del aguante del módulo (≤3 µs en caliente)."
 		(exclude_from_sim no)
-		(at 78.232 165.354 0)
+		(at 148.844 166.878 0)
 		(effects
 			(font
@@
 			)
 		)
-		(property "Value" "47pF"
+		(property "Value" "56pF"
 			(at 60.96 142.2399 0)
 			(show_name no)

Commit message: correcciones de apps
Parts:
- renumbered C37 to C34, C38 to C35, C39 to C36, C40 to C37, C41 to C38, C42 to C39, C43 to C40, C44 to C41, C45 to C42, C46 to C43, C47 to C44, C48 to C45, C49 to C46, C50 to C47, C51 to C48, C52 to C49, D28 to D27, D29 to D28, D30 to D29, D31 to D30, D32 to D31, D33 to D32, D34 to D33, D35 to D34, D36 to D35, D37 to D36, D38 to D37, R37 to R30, R38 to R31, R39 to R32, R40 to R33, R41 to R34, R42 to R35, R43 to R36, R44 to R37, R45 to R38, R46 to R39, R47 to R40, R48 to R41, R49 to R42, R50 to R43, TP16 to TP11, TP17 to TP12, U7 to U8, U8 to U9

Commit message: EsqumaticoCuasifinalizado
Ya hice varias correcciones creo q solo falta cambiar algunas resistencias en los limites q tendrian que estar en el notion
Connections:
- net 15V_ISO renamed +15V
Changed lines of the file:
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@@
-	(wire
-		(pts
-			(xy 266.7 35.56) (xy 266.7 36.83)
-		)
-		(stroke
-			(width 0)
-			(type default)
-		)
-	)
 	(wire
 		(pts
@@
 	(wire
 		(pts
-			(xy 266.7 35.56) (xy 271.78 35.56)
+			(xy 266.7 36.83) (xy 276.86 36.83)
 		)
 		(stroke
@@
 	)
 	(label "+15V"
-		(at 271.78 35.56 180)
+		(at 276.86 36.83 180)
 		(effects
 			(font
@@
 		(effects
 			(font
-				(size 1.27 1.27)
-			)
-			(justify left)
-		)
-	)
-	(hierarchical_label "15V_ISO"
-		(shape bidirectional)
-		(at 271.78 35.56 0)
-		(effects
-			(font
