File: PCB/Inverter/Primero_esquematico/GD_LS.kicad_sch (KiCad schematic)
At the start: 46 parts, among them T1 750317595, U3 LM25180QNGURQ1, U4 UCC21750QDWRQ1, U42 LP2951-5.0_VSSOP

Commit message: Solo falta routear algo
Parts:
- C6: value 47pF -> 56pF
Other:
- note added: "CASO SiC C_BLK · dV/dt = Ichg + (V_DD − V_Z − V) / R_ext V_ss = (V_DD − V_Z) + Ichg·R_ext τ = R_ext · C_BLK t_BLK = τ · ln[ V_ss / (V_ss − V_DESAT) ] Para nuestro caso el tiempo de blanking es 121ns"
- note added: "Caso IGBT t_BLK = C_BLK · V_DESAT / Ichg t_BLK = 1,05 us"
- note added: "LAS Ressitencias estas no iran en el diseño final solo para el caso de usar SiC"
Changed lines of the file:
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@@
 	(text "Frecuencia de corte en 2khz (Comentario para componentes colocados en APWM)\nEsto se coloca para pasar de un PWM a una señal ADC para monitorear tension\ny temperatura, esta frecuencia de corte es elevada para temperatura pero\nquiero usar menos variedad de componentes y no deberia cambiar\n"
 		(exclude_from_sim no)
-		(at 106.68 175.768 0)
+		(at 128.016 175.768 0)
 		(effects
 			(font
@@
 		)
 	)
+	(text "Caso IGBT\nt_BLK = C_BLK · V_DESAT / Ichg\nt_BLK = 1,05 us"
+		(exclude_from_sim no)
+		(at 37.338 127.508 0)
+		(effects
+			(font
+				(size 1.27 1.27)
+				(thickness 0.254)
+				(bold yes)
+			)
+		)
+	)
 	(text "Aca hay q conciderar el DC Bias\nDesteriora la capacitancia de los capacitores"
 		(exclude_from_sim no)
@@
 		)
 	)
+	(text "LAS Ressitencias estas no\niran en el diseño final\nsolo para el caso de usar SiC"
+		(exclude_from_sim no)
+		(at 67.31 100.838 0)
+		(effects
+			(font
+				(size 1.27 1.27)
+			)
+		)
+	)
 	(text "Ejemplo de Teaxas de su implementacion\nhttps://www.ti.com/lit/ug/sluuck0a/sluuck0a.pdf?ts=1781860744035"
 		(exclude_from_sim no)
@@
 	(text "Esta etapa vigila la saturación del IGBT midiendo su tensión colector-emisor (V_CE) mientras está encendido:\n- Si el IGBT satura, V_CE es baja → OK.\n- Si V_CE queda alta con el IGBT en ON (desaturación) → sobrecorriente/cortocircuito → dispara el soft turn-off.\n- El C de blanking (47 pF) fija una ventana inicial tras el encendido en la que la protección se ignora, para dar tiempo a que el IGBT sature.\n- Si hay disparos falsos en el encendido → subir un poco el C (alarga el blanking).\n- No subirlo de más: alarga la ventana sin protección; un cortocircuito real debe detectarse antes del aguante del módulo (≤3 µs en caliente)."
 		(exclude_from_sim no)
-		(at 58.42 164.592 0)
+		(at 130.302 165.608 0)
 		(effects
 			(font
@@
 		)
 	)
+	(text "CASO SiC\nC_BLK · dV/dt = Ichg + (V_DD − V_Z − V) / R_ext\n\nV_ss = (V_DD − V_Z) + Ichg·R_ext\nτ = R_ext · C_BLK\nt_BLK = τ · ln[ V_ss / (V_ss − V_DESAT) ]\n\nPara nuestro caso el tiempo de blanking es 121ns"
+		(exclude_from_sim no)
+		(at 53.848 171.958 0)
+		(effects
+			(font
+				(size 1.27 1.27)
+				(thickness 0.254)
+				(bold yes)
+			)
+		)
+	)
 	(text "Pagina 23"
 		(exclude_from_sim no)
@@
 			)
 		)
-		(property "Value" "47pF"
+		(property "Value" "56pF"
 			(at 43.18 142.2399 0)
 			(show_name no)

Commit message: correcciones de apps
Parts:
- renumbered C14 to C10, C189 to C11, C16 to C12, C17 to C13, C18 to C14, C19 to C15, C20 to C16, C190 to C17, C6 to C2, C5 to C3, C7 to C4, C9 to C5, C11 to C6, C12 to C7, C15 to C8, C13 to C9, D11 to D10, D12 to D11, D13 to D12, D14 to D13, D15 to D14, D16 to D15, D6 to D5, D7 to D6, D8 to D7, D9 to D8, D10 to D9, R15 to R10, R16 to R11, R17 to R12, R19 to R13, R21 to R14, R22 to R15, R226 to R16, R11 to R4, R13 to R5, R14 to R6, R9 to R7, R10 to R8, R12 to R9, TP12 to TP7, TP13 to TP8, U4 to U2, U42 to U4

Commit message: EsqumaticoCuasifinalizado
Ya hice varias correcciones creo q solo falta cambiar algunas resistencias en los limites q tendrian que estar en el notion
Parts:
- added C181: 100nF, Capacitor_SMD:C_0402_1005Metric, symbol Device:C_Small
- C11, C17: value 1uF -> 4.8uF
Connections:
- net 5V_ISO: now also C181.1
- net ISO_GND: now also C181.2
Other:
- note added: "Pagina 26 del datasheet"
- moved on the sheet: C17
Changed lines of the file:
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@@
 		)
 	)
+	(text "Pagina 26 del datasheet\n"
+		(exclude_from_sim no)
+		(at 253.746 151.892 0)
+		(effects
+			(font
+				(size 1.27 1.27)
+			)
+		)
+	)
 	(text "Corriente pico:\nI(on)=8,33A\nI(off)=4,92A\nCada 50us\n"
 		(exclude_from_sim no)
@@
 	)
 	(junction
+		(at 271.78 144.78)
+		(diameter 0)
+		(color 0 0 0 0)
+	)
+	(junction
 		(at 240.03 49.53)
 		(diameter 0)
@@
 	)
 	(junction
+		(at 275.59 124.46)
+		(diameter 0)
+		(color 0 0 0 0)
+	)
+	(junction
+		(at 271.78 124.46)
+		(diameter 0)
+		(color 0 0 0 0)
+	)
+	(junction
 		(at 74.93 115.57)
 		(diameter 0)
@@
 	)
 	(junction
-		(at 273.05 124.46)
-		(diameter 0)
-		(color 0 0 0 0)
-	)
-	(junction
 		(at 240.03 62.23)
 		(diameter 0)
@@
 	(wire
 		(pts
+			(xy 275.59 137.16) (xy 275.59 144.78)
+		)
+		(stroke
+			(width 0)
+			(type default)
+		)
+	)
+	(wire
+		(pts
 			(xy 135.89 43.18) (xy 135.89 39.37)
 		)
@@
 	(wire
 		(pts
+			(xy 275.59 124.46) (xy 279.4 124.46)
+		)
+		(stroke
+			(width 0)
+			(type default)
+		)
+	)
+	(wire
+		(pts
 			(xy 228.6 59.69) (xy 228.6 62.23)
 		)
@@
 	(wire
 		(pts
-			(xy 160.02 114.3) (xy 214.63 114.3)
+			(xy 275.59 144.78) (xy 271.78 144.78)
 		)
 		(stroke
@@
 	(wire
 		(pts
-			(xy 240.03 40.64) (xy 240.03 36.83)
+			(xy 160.02 114.3) (xy 214.63 114.3)
 		)
 		(stroke
@@
 	(wire
 		(pts
-			(xy 71.12 115.57) (xy 74.93 115.57)
+			(xy 240.03 40.64) (xy 240.03 36.83)
 		)
 		(stroke
@@
 	(wire
 		(pts
-			(xy 240.03 49.53) (xy 228.6 49.53)
+			(xy 71.12 115.57) (xy 74.93 115.57)
 		)
 		(stroke
@@
 	(wire
 		(pts
-			(xy 275.59 124.46) (xy 273.05 124.46)
+			(xy 240.03 49.53) (xy 228.6 49.53)
 		)
 		(stroke
@@
 	(wire
 		(pts
+			(xy 271.78 124.46) (xy 275.59 124.46)
+		)
+		(stroke
+			(width 0)
+			(type default)
+		)
+	)
+	(wire
+		(pts
 			(xy 50.8 144.78) (xy 50.8 147.32)
 		)
@@
 	(wire
 		(pts
-			(xy 264.16 124.46) (xy 273.05 124.46)
+			(xy 264.16 124.46) (xy 271.78 124.46)
 		)
 		(stroke
@@
 	(wire
 		(pts
-			(xy 273.05 124.46) (xy 273.05 125.73)
+			(xy 271.78 124.46) (xy 271.78 132.08)
 		)
 		(stroke
@@
 	(wire
 		(pts
-			(xy 273.05 144.78) (xy 250.19 144.78)
+			(xy 271.78 144.78) (xy 250.19 144.78)
 		)
 		(stroke
@@
 	(wire
 		(pts
-			(xy 273.05 130.81) (xy 273.05 144.78)
+			(xy 271.78 137.16) (xy 271.78 144.78)
 		)
 		(stroke
@@
 	(wire
 		(pts
+			(xy 275.59 124.46) (xy 275.59 132.08)
+		)
+		(stroke
+			(width 0)
+			(type default)
+		)
+	)
+	(wire
+		(pts
 			(xy 50.8 147.32) (xy 69.85 147.32)
 		)
@@
 	(hierarchical_label "5V_ISO"
 		(shape bidirectional)
-		(at 275.59 124.46 0)
+		(at 279.4 124.46 0)
 		(effects
 			(font
@@
 			)
 		)
-		(property "Value" "1uF"
+		(property "Value" "4.8uF"
 			(at 232.41 128.2762 0)
 			(show_name no)
@@
 	(symbol
 		(lib_id "Device:C_Small")
-		(at 273.05 128.27 0)
+		(at 271.78 134.62 0)
+		(mirror y)
 		(unit 1)
 		(body_style 1)
@@
 		(dnp no)
 		(property "Reference" "C17"
-			(at 275.59 127.0062 0)
+			(at 269.24 133.3562 0)
 			(show_name no)
 			(do_not_autoplace no)
@@
 			)
 		)
-		(property "Value" "1uF"
-			(at 275.59 129.5462 0)
+		(property "Value" "4.8uF"
+			(at 269.24 135.8962 0)
 			(show_name no)
 			(do_not_autoplace no)
@@
 		)
 		(property "Footprint" "Capacitor_SMD:C_0603_1608Metric"
-			(at 273.05 128.27 0)
+			(at 271.78 134.62 0)
 			(hide yes)
 			(show_name no)
@@
 		)
 		(property "Datasheet" ""
-			(at 273.05 128.27 0)
+			(at 271.78 134.62 0)
 			(hide yes)
 			(show_name no)
@@
 		)
 		(property "Description" "Unpolarized capacitor, small symbol"
-			(at 273.05 128.27 0)
+			(at 271.78 134.62 0)
 			(hide yes)
 			(show_name no)
@@
 		)
 		(property "Description_1" ""
-			(at 273.05 128.27 0)
+			(at 271.78 134.62 0)
 			(hide yes)
 			(show_name no)
@@
 		)
 		(property "Purchase-URL" ""
-			(at 273.05 128.27 0)
+			(at 271.78 134.62 0)
 			(hide yes)
 			(show_name no)
@@
 					(unit 1)
 				)
+			)
+		)
+	)
+	(symbol
+		(lib_id "Device:C_Small")
+		(at 275.59 134.62 0)
+		(unit 1)
+		(body_style 1)
+		(exclude_from_sim no)
+		(in_bom yes)
+		(on_board yes)
+		(in_pos_files yes)
+		(dnp no)
+		(property "Reference" "C181"
+			(at 278.13 133.3562 0)
+			(show_name no)
+			(do_not_autoplace no)
+			(effects
+				(font
+					(size 1.27 1.27)
+				)
+				(justify left)
+			)
+		)
+		(property "Value" "100nF"
+			(at 278.13 135.8962 0)
+			(show_name no)
+			(do_not_autoplace no)
+			(effects
+				(font
+					(size 1.27 1.27)
+				)
+				(justify left)
+			)
+		)
+		(property "Footprint" "Capacitor_SMD:C_0402_1005Metric"
+			(at 275.59 134.62 0)
+			(hide yes)
+			(show_name no)
+			(do_not_autoplace no)
+			(effects
+				(font
+					(size 1.27 1.27)
+				)
+			)
+		)
+		(property "Datasheet" ""
+			(at 275.59 134.62 0)
+			(hide yes)
+			(show_name no)
+			(do_not_autoplace no)
+			(effects
+				(font
+					(size 1.27 1.27)
+				)
+			)
+		)
+		(property "Description" "Unpolarized capacitor, small symbol"
+			(at 275.59 134.62 0)
+			(hide yes)
+			(show_name no)
+			(do_not_autoplace no)
+			(effects
+				(font
+					(size 1.27 1.27)
+				)
+			)
+		)
+		(property "Description_1" ""
+			(at 275.59 134.62 0)
+			(hide yes)
+			(show_name no)
+			(do_not_autoplace no)
+			(effects
+				(font
+					(size 1.27 1.27)
+				)
+			)
+		)
+		(property "Purchase-URL" ""
+			(at 275.59 134.62 0)
+			(hide yes)
+			(show_name no)
+			(do_not_autoplace no)
+			(effects
+				(font
+					(size 1.27 1.27)
+				)
+			)
+		)
+		(pin "1"
+		)
+		(pin "2"
+		)
+		(instances
+			(project "Primero_esquematico"
+				(path "/d930f486-f6ac-489c-907e-47f2cb34cf04/d101e913-ebd1-4e08-b728-82218f47123b/f5297dcd-d9e2-4174-98d4-ada2947e9df5/5cdf39cf-afbe-4cc8-b2fc-5cff4a76438c"
+					(reference "C181")
+					(unit 1)
+				)
+				(path "/d930f486-f6ac-489c-907e-47f2cb34cf04/d101e913-ebd1-4e08-b728-82218f47123b/f5297dcd-d9e2-4174-98d4-ada2947e9df5/78ffa60a-7e25-44e8-bbd6-bfc8ed5e55d3"
+					(reference "C183")
+					(unit 1)
+				)
+				(path "/d930f486-f6ac-489c-907e-47f2cb34cf04/d101e913-ebd1-4e08-b728-82218f47123b/f5297dcd-d9e2-4174-98d4-ada2947e9df5/e0d894c7-fa45-4b97-bd7c-86f3d038d141"
+					(reference "C182")
+					(unit 1)
+				)
