File: PCB/Inverter/Primero_esquematico/LogicSupply.kicad_sch (KiCad schematic)
At the start: 34 parts, among them U24 LM25180QNGURQ1, U27 TPS7A2050PDBVR, U28 REF2033QDDCRQ1, U39 TLV76733QWDRBRQ1, U40 LP5907QMFX-3.3Q1

Commit message: Algunos cambios
Parts:
- removed C121: CL31B475KAHNNNE, Capacitor_SMD:C_1206_3216Metric, symbol Device:C
- removed D75: SMDJ13A, Diode_SMD:D_SMC, symbol Device:D_TVS
- U28: value REF2033QDDCRQ1 -> REF2030-Q1
Connections:
- net +3.3V renamed +3.3_digital
- net +3.3_digital: now also TP34.1; no longer TP32.1
- net +3.3VP renamed +3.3V_analog
- net +3.3V_analog: now also TP32.1; no longer TP34.1
Other:
- note added: "Alimentacion Digital"
- note added: "Hay dos distintas para repartir potencia y para que el ruido digital con sus armonicos no ensucie las mediciones"
- moved on the sheet: C122, C123, C148, C149, D76, D77, D78, D79, D80, L1, R156, R157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

Commit message: Corregi cosas de la placa
Parts:
- removed TP36: TestPoint, TestPoint:TestPoint_Pad_D1.0mm, symbol Connector:TestPoint
- added C169: 10uF, Capacitor_SMD:C_0805_2012Metric, symbol Device:C
- R161: footprint Resistor_SMD:R_0402_1005Metric -> Resistor_SMD:R_0603_1608Metric
- renumbered C122 to C138, C149 to C139, C150 to C140, C123 to C141, C151 to C142, C148 to C143, C124 to C144, C125 to C145, C126 to C146, D76 to D75, D77 to D76, D78 to D77, D79 to D78, D80 to D79, U24 to U23, U40 to U24, U39 to U25, U27 to U26, U28 to U27
Connections:
- net +5V: now also C169.2
- net GND: now also C169.1

Commit message: a
Parts:
- added C174: 10uF, Capacitor_SMD:C_0805_2012Metric, symbol Device:C
- added U37: TPS7A2050PDBVR, Snapeda:DBV0005A-IPC_A, symbol Snapeda:TPS7A2050PDBVR
Connections:
- net +5V: no longer C169.2, U26.5 (OUT)
- net 5V_FB: now also U37.1 (IN), U37.3 (EN)
- net GND: now also C174.1, U37.2 (GND)
- new net +5V_analog: C174.2, U37.5 (OUT)
- new net +5V_digital: C169.2, U26.5 (OUT)
Other:
- note added: "Alimentacion 5V"
- moved on the sheet: C145, C146, TP32, TP33, TP34, TP35
