File: PCB/Inverter/Primero_esquematico/LogicSupply.kicad_sch (KiCad schematic)
At the start: 34 parts, among them U23 LM25180QNGURQ1, U24 LP5907QMFX-3.3Q1, U25 TLV76733QWDRBRQ1, U26 TPS7A2050PDBVR, U27 REF2030-Q1, U37 TPS7A2050PDBVR

Commit message: Falta poco
Parts:
- removed TP32, TP33, TP34, TP35: TestPoint, TestPoint:TestPoint_Pad_D1.0mm, symbol Connector:TestPoint

Commit message: Solo falta routear algo
Connections:
- net +5V is gone; now on net +5V_digital: C144.1, U27.3 (EN), U27.4 (VIN)
Changed lines of the file:
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@@
+	)
+	(symbol
+		(lib_id "power:+5V")
+		(at 222.25 123.19 0)
+		(unit 1)
+		(body_style 1)
+		(exclude_from_sim no)
+		(in_bom yes)
+		(on_board yes)
+		(in_pos_files yes)
+		(dnp no)
+		(fields_autoplaced yes)
+		(property "Reference" "#PWR0270"
+			(at 222.25 127 0)
+			(hide yes)
+			(show_name no)
+			(do_not_autoplace no)
+			(effects
+				(font
+					(size 1.27 1.27)
+				)
+			)
+		)
+		(property "Value" "+5V_digital"
+			(at 222.25 118.11 0)
+			(show_name no)
+			(do_not_autoplace no)
+			(effects
+				(font
+					(size 1.27 1.27)
+				)
+			)
+		)
+		(property "Footprint" ""
+			(at 222.25 123.19 0)
+			(hide yes)
+			(show_name no)
+			(do_not_autoplace no)
+			(effects
+				(font
+					(size 1.27 1.27)
+				)
+			)
+		)
+		(property "Datasheet" ""
+			(at 222.25 123.19 0)
+			(hide yes)
+			(show_name no)
+			(do_not_autoplace no)
+			(effects
+				(font
+					(size 1.27 1.27)
+				)
+			)
+		)
+		(property "Description" "Power symbol creates a global label with name \"+5V\""
+			(at 222.25 123.19 0)
+			(hide yes)
+			(show_name no)
+			(do_not_autoplace no)
+			(effects
+				(font
+					(size 1.27 1.27)
+				)
+			)
+		)
+		(pin "1"
+		)
+		(instances
+			(project "Primero_esquematico"
+				(path "/d930f486-f6ac-489c-907e-47f2cb34cf04/0bcc01e0-1903-49c9-8a02-17640b3194e7/d69e10c3-78b1-4a5f-bd39-c4f4dfb65e7e"
+					(reference "#PWR0270")
+					(unit 1)
+				)
+			)
+		)
 	)
 	(symbol
@@
 					(unit 1)
 				)
-			)
-		)
-	)
-	(symbol
-		(lib_id "power:+5V")
-		(at 222.25 123.19 0)
-		(unit 1)
-		(body_style 1)
-		(exclude_from_sim no)
-		(in_bom yes)
-		(on_board yes)
-		(in_pos_files yes)
-		(dnp no)
-		(fields_autoplaced yes)
-		(property "Reference" "#PWR0177"
-			(at 222.25 127 0)
-			(hide yes)
-			(show_name no)
-			(do_not_autoplace no)
-			(effects
-				(font
-					(size 1.27 1.27)
-				)
-			)
-		)
-		(property "Value" "+5V"
-			(at 222.25 118.11 0)
-			(show_name no)
-			(do_not_autoplace no)
-			(effects
-				(font
-					(size 1.27 1.27)
-				)
-			)
-		)
-		(property "Footprint" ""
-			(at 222.25 123.19 0)
-			(hide yes)
-			(show_name no)
-			(do_not_autoplace no)
-			(effects
-				(font
-					(size 1.27 1.27)
-				)
-			)
-		)
-		(property "Datasheet" ""
-			(at 222.25 123.19 0)
-			(hide yes)
-			(show_name no)
-			(do_not_autoplace no)
-			(effects
-				(font
-					(size 1.27 1.27)
-				)
-			)
-		)
-		(property "Description" "Power symbol creates a global label with name \"+5V\""
-			(at 222.25 123.19 0)
-			(hide yes)
-			(show_name no)
-			(do_not_autoplace no)
-			(effects
-				(font
-					(size 1.27 1.27)
-				)
-			)
-		)
-		(pin "1"
-		)
-		(instances
-			(project "Primero_esquematico"
-				(path "/d930f486-f6ac-489c-907e-47f2cb34cf04/0bcc01e0-1903-49c9-8a02-17640b3194e7/d69e10c3-78b1-4a5f-bd39-c4f4dfb65e7e"
-					(reference "#PWR0177")
-					(unit 1)
-				)

Commit message: correcciones de apps
Parts:
- renumbered C174 to C138, C138 to C139, C139 to C140, C169 to C141, C140 to C142, C141 to C143, C142 to C144, C143 to C145, C144 to C146, C145 to C147, C146 to C148, D75 to D74, D76 to D75, D77 to D76, D78 to D77, D79 to D78, R156 to R140, R157 to R141, R158 to R142, R159 to R143, R160 to R144, R161 to R145, U37 to U24, U23 to U25, U24 to U26, U26 to U27, U25 to U28, U27 to U29

Commit message: EsqumaticoCuasifinalizado
Ya hice varias correcciones creo q solo falta cambiar algunas resistencias en los limites q tendrian que estar en el notion
Parts:
- removed C148: 0,1uF, Capacitor_SMD:C_0603_1608Metric, symbol Device:C_Small
- U25: footprint NGU0008C -> Snapeda:NGU0008C
Connections:
- net +1V5: no longer names the net of U29.1 (VBIAS)
- no-connect marks 0 -> 1

Commit message: Modificaciones por falta de stock
Connections:
- net +1V5: now reaches U29.1 (VBIAS)
- no-connect marks 1 -> 0
Other:
- note added: "Power Flags"
