File: PCB/Inverter/Primero_esquematico/conectores_externos.kicad_sch (KiCad schematic)
At the start: 5 parts, among them J8 20021521-00010T1LF

Commit message: Un par de cosas q corregi del ERC pero sigue mal
Parts:
- J8: footprint Snapeda:AMPHENOL_20021521-00010T1LF -> 20021521-00010T1LF:AMPHENOL_20021521-00010T1LF
Changed lines of the file:
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@@
 			)
 		)
-		(property "Description" "-- valores mixtos --"
+		(property "Description" "Resistor"
 			(at 191.77 87.63 0)
 			(hide yes)
@@
 			)
 		)
-		(property "Description" "-- valores mixtos --"
+		(property "Description" "Resistor"
 			(at 191.77 97.79 0)
 			(hide yes)
@@
 			)
 		)
-		(property "Footprint" "Snapeda:AMPHENOL_20021521-00010T1LF"
+		(property "Footprint" "20021521-00010T1LF:AMPHENOL_20021521-00010T1LF"
 			(at 184.15 22.86 0)
 			(hide yes)
@@
 			)
 		)
-		(property "Description" "-- valores mixtos --"
+		(property "Description" "Resistor"
 			(at 177.8 97.79 0)
 			(hide yes)
@@
 			)
 		)
-		(property "Description" "-- valores mixtos --"
+		(property "Description" "Resistor"
 			(at 177.8 87.63 0)
 			(hide yes)

Commit message: Esquematico Listo
Parts:
- J8: footprint 20021521-00010T1LF:AMPHENOL_20021521-00010T1LF -> Snapeda:AMPHENOL_20021521-00010T1LF
Changed lines of the file:
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@@
 			)
 		)
-		(property "Footprint" "20021521-00010T1LF:AMPHENOL_20021521-00010T1LF"
+		(property "Footprint" "Snapeda:AMPHENOL_20021521-00010T1LF"
 			(at 184.15 22.86 0)
 			(hide yes)

Commit message: correcciones
Parts:
- removed R184, R186: 10k, Resistor_SMD:R_0402_1005Metric, symbol Device:R
- added R193, R195: 0, Resistor_SMD:R_0402_1005Metric, symbol Device:R
- added SW2, SW3: IT-1181-180G-G, FSAE_footprints:Sin título, symbol Switch:SW_Push
- renumbered J8 to J4, R183 to R192, R185 to R194
Connections:
- net GND: now also R193.2, R195.2
- net GP_24_BOOT_MODE_2: now also SW3.2
- net GP_32_BOOT_MODE_1: now also SW2.2
- net +3.3VP renamed +3.3V
- new net: R193.1, SW2.1
- new net: R195.1, SW3.1
Other:
- moved on the sheet: R194

Commit message: Algunos cambios
Parts:
- removed J4: 20021521-00010T1LF, Snapeda:AMPHENOL_20021521-00010T1LF, symbol Snapeda:20021521-00010T1LF
- removed SW2, SW3: IT-1181-180G-G, FSAE_footprints:Sin título, symbol Switch:SW_Push
- added J4: 347928082, Snapeda:CONN08_34792_MOL, symbol Snapeda:347928082
- added S1: DS04-254-2-02BK-SMT-TR, Snapeda:SW_DS04-254-2-02BK-SMT-TR, symbol Snapeda:DS04-254-2-02BK-SMT-TR
Connections:
- net GND: now also J4.7, J4.8
- net GP_24_BOOT_MODE_2: now also S1.2B
- net GP_32_BOOT_MODE_1: now also S1.1B
- net Mcu_Reset: now also J4.2
- net TCK: now also J4.5
- net TDI: now also J4.3
- net TDO: now also J4.4
- net TMS: now also J4.6
- net at R193.1: now also S1.1A
- net at R195.1: now also S1.2A
- net +3.3V renamed +3.3_digital
- net +3.3_digital: now also J4.1
- no-connect marks 1 -> 0
Other:
- note added: "Con el sistema finalizado se recomienda sacar las resistencias de 0 Ohms para no tener problemas con la degradacion de los interruptores"
- moved on the sheet: R192, R193, R194, R195

Commit message: Corregi cosas de la placa
Parts:
- renumbered J4 to J5
Changed lines of the file:
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@@
 		(in_pos_files yes)
 		(dnp no)
-		(property "Reference" "J4"
+		(property "Reference" "J5"
 			(at 247.65 94.996 0)
 			(show_name no)
@@
 			(project "Primero_esquematico"
 				(path "/d930f486-f6ac-489c-907e-47f2cb34cf04/0bcc01e0-1903-49c9-8a02-17640b3194e7/49867297-e849-416a-bae2-6d0463384f96"
-					(reference "J4")
+					(reference "J5")
 					(unit 1)
 				)
@@
 		(in_pos_files yes)
 		(dnp no)
-		(property "Reference" "#PWR0335"
+		(property "Reference" "#PWR0245"
 			(at 227.33 91.44 0)
 			(hide yes)
@@
 			(project "Primero_esquematico"
 				(path "/d930f486-f6ac-489c-907e-47f2cb34cf04/0bcc01e0-1903-49c9-8a02-17640b3194e7/49867297-e849-416a-bae2-6d0463384f96"
-					(reference "#PWR0335")
+					(reference "#PWR0245")
 					(unit 1)
 				)
@@
 		(dnp no)
 		(fields_autoplaced yes)
-		(property "Reference" "#PWR0238"
+		(property "Reference" "#PWR0246"
 			(at 231.14 113.03 0)
 			(hide yes)
@@
 			(project "Primero_esquematico"
 				(path "/d930f486-f6ac-489c-907e-47f2cb34cf04/0bcc01e0-1903-49c9-8a02-17640b3194e7/49867297-e849-416a-bae2-6d0463384f96"
-					(reference "#PWR0238")
+					(reference "#PWR0246")
 					(unit 1)
 				)
@@
 		(in_pos_files yes)
 		(dnp no)
-		(property "Reference" "#PWR0336"
+		(property "Reference" "#PWR0243"
 			(at 172.72 80.01 0)
 			(hide yes)
@@
 			(project "Primero_esquematico"
 				(path "/d930f486-f6ac-489c-907e-47f2cb34cf04/0bcc01e0-1903-49c9-8a02-17640b3194e7/49867297-e849-416a-bae2-6d0463384f96"
-					(reference "#PWR0336")
+					(reference "#PWR0243")
 					(unit 1)
 				)
@@
 		(dnp no)
 		(fields_autoplaced yes)
-		(property "Reference" "#PWR0243"
+		(property "Reference" "#PWR0244"
 			(at 175.26 118.11 0)
 			(hide yes)
@@
 			(project "Primero_esquematico"
 				(path "/d930f486-f6ac-489c-907e-47f2cb34cf04/0bcc01e0-1903-49c9-8a02-17640b3194e7/49867297-e849-416a-bae2-6d0463384f96"
-					(reference "#PWR0243")
+					(reference "#PWR0244")
 					(unit 1)
 				)
@@
 		(dnp no)
 		(fields_autoplaced yes)
-		(property "Reference" "#PWR0241"
+		(property "Reference" "#PWR0242"
 			(at 170.18 118.11 0)
 			(hide yes)
@@
 			(project "Primero_esquematico"
 				(path "/d930f486-f6ac-489c-907e-47f2cb34cf04/0bcc01e0-1903-49c9-8a02-17640b3194e7/49867297-e849-416a-bae2-6d0463384f96"
-					(reference "#PWR0241")
+					(reference "#PWR0242")
 					(unit 1)
 				)
