File: PCB/Inverter/Primero_esquematico/conectores_externos.kicad_sch (KiCad schematic)
At the start: 6 parts, among them J5 347928082

Commit message: Puse areas sin de aisleamento
Connections:
- net GP_24_BOOT_MODE_2: now also R192.2, S1.1B; no longer R194.2, S1.2B
- net GP_32_BOOT_MODE_1: now also R194.2, S1.2B; no longer R192.2, S1.1B
Changed lines of the file:
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@@
 		)
 	)
-	(hierarchical_label "GP_24_BOOT_MODE_2"
+	(hierarchical_label "GP_32_BOOT_MODE_1"
 		(shape bidirectional)
 		(at 176.53 87.63 0)
@@
 		)
 	)
-	(hierarchical_label "Mcu_Reset"
+	(hierarchical_label "GP_24_BOOT_MODE_2"
 		(shape bidirectional)
-		(at 232.41 90.17 180)
+		(at 168.91 87.63 180)
 		(effects
 			(font
@@
 		)
 	)
-	(hierarchical_label "GP_32_BOOT_MODE_1"
+	(hierarchical_label "Mcu_Reset"
 		(shape bidirectional)
-		(at 168.91 87.63 180)
+		(at 232.41 90.17 180)
 		(effects
 			(font

Commit message: correcciones de apps
Parts:
- renumbered J5 to J4, R192 to R176, R193 to R177, R194 to R178, R195 to R179
Changed lines of the file:
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@@
 		(in_pos_files yes)
 		(dnp no)
-		(property "Reference" "J5"
+		(property "Reference" "J4"
 			(at 247.65 94.996 0)
 			(show_name no)
@@
 			(project "Primero_esquematico"
 				(path "/d930f486-f6ac-489c-907e-47f2cb34cf04/0bcc01e0-1903-49c9-8a02-17640b3194e7/49867297-e849-416a-bae2-6d0463384f96"
-					(reference "J5")
+					(reference "J4")
 					(unit 1)
 				)
@@
 		(in_pos_files yes)
 		(dnp no)
-		(property "Reference" "#PWR0245"
+		(property "Reference" "#PWR0236"
 			(at 227.33 91.44 0)
 			(hide yes)
@@
 			(project "Primero_esquematico"
 				(path "/d930f486-f6ac-489c-907e-47f2cb34cf04/0bcc01e0-1903-49c9-8a02-17640b3194e7/49867297-e849-416a-bae2-6d0463384f96"
-					(reference "#PWR0245")
+					(reference "#PWR0236")
 					(unit 1)
 				)
@@
 		(dnp no)
 		(fields_autoplaced yes)
-		(property "Reference" "#PWR0246"
+		(property "Reference" "#PWR0237"
 			(at 231.14 113.03 0)
 			(hide yes)
@@
 			(project "Primero_esquematico"
 				(path "/d930f486-f6ac-489c-907e-47f2cb34cf04/0bcc01e0-1903-49c9-8a02-17640b3194e7/49867297-e849-416a-bae2-6d0463384f96"
-					(reference "#PWR0246")
+					(reference "#PWR0237")
 					(unit 1)
 				)
@@
 		(in_pos_files yes)
 		(dnp no)
-		(property "Reference" "R193"
+		(property "Reference" "R177"
 			(at 167.64 106.6799 0)
 			(show_name no)
@@
 			(project "Primero_esquematico"
 				(path "/d930f486-f6ac-489c-907e-47f2cb34cf04/0bcc01e0-1903-49c9-8a02-17640b3194e7/49867297-e849-416a-bae2-6d0463384f96"
-					(reference "R193")
+					(reference "R177")
 					(unit 1)
 				)
@@
 		(dnp no)
 		(fields_autoplaced yes)
-		(property "Reference" "R194"
+		(property "Reference" "R178"
 			(at 177.8 81.2799 0)
 			(show_name no)
@@
 			(project "Primero_esquematico"
 				(path "/d930f486-f6ac-489c-907e-47f2cb34cf04/0bcc01e0-1903-49c9-8a02-17640b3194e7/49867297-e849-416a-bae2-6d0463384f96"
-					(reference "R194")
+					(reference "R178")
 					(unit 1)
 				)
@@
 		(in_pos_files yes)
 		(dnp no)
-		(property "Reference" "#PWR0243"
+		(property "Reference" "#PWR0234"
 			(at 172.72 80.01 0)
 			(hide yes)
@@
 			(project "Primero_esquematico"
 				(path "/d930f486-f6ac-489c-907e-47f2cb34cf04/0bcc01e0-1903-49c9-8a02-17640b3194e7/49867297-e849-416a-bae2-6d0463384f96"
-					(reference "#PWR0243")
+					(reference "#PWR0234")
 					(unit 1)
 				)
@@
 		(dnp no)
 		(fields_autoplaced yes)
-		(property "Reference" "#PWR0244"
+		(property "Reference" "#PWR0235"
 			(at 175.26 118.11 0)
 			(hide yes)
@@
 			(project "Primero_esquematico"
 				(path "/d930f486-f6ac-489c-907e-47f2cb34cf04/0bcc01e0-1903-49c9-8a02-17640b3194e7/49867297-e849-416a-bae2-6d0463384f96"
-					(reference "#PWR0244")
+					(reference "#PWR0235")
 					(unit 1)
 				)
@@
 		(in_pos_files yes)
 		(dnp no)
-		(property "Reference" "R195"
+		(property "Reference" "R179"
 			(at 177.8 106.6799 0)
 			(show_name no)
@@
 			(project "Primero_esquematico"
 				(path "/d930f486-f6ac-489c-907e-47f2cb34cf04/0bcc01e0-1903-49c9-8a02-17640b3194e7/49867297-e849-416a-bae2-6d0463384f96"
-					(reference "R195")
+					(reference "R179")
 					(unit 1)
 				)
@@
 		(dnp no)
 		(fields_autoplaced yes)
-		(property "Reference" "#PWR0242"
+		(property "Reference" "#PWR0233"
 			(at 170.18 118.11 0)
 			(hide yes)
@@
 			(project "Primero_esquematico"
 				(path "/d930f486-f6ac-489c-907e-47f2cb34cf04/0bcc01e0-1903-49c9-8a02-17640b3194e7/49867297-e849-416a-bae2-6d0463384f96"
-					(reference "#PWR0242")
+					(reference "#PWR0233")
 					(unit 1)
 				)
@@
 		(in_pos_files yes)
 		(dnp no)
-		(property "Reference" "R192"
+		(property "Reference" "R176"
 			(at 167.64 81.2799 0)
 			(show_name no)
@@
 			(project "Primero_esquematico"
 				(path "/d930f486-f6ac-489c-907e-47f2cb34cf04/0bcc01e0-1903-49c9-8a02-17640b3194e7/49867297-e849-416a-bae2-6d0463384f96"
-					(reference "R192")
+					(reference "R176")
 					(unit 1)
 				)
