File: PCB/Inverter/Primero_esquematico/SistemasProteccion.kicad_sch (KiCad schematic)
At the start: 34 parts, among them U28 TLV1704AQPWRQ1, U29 TLV1704AQPWRQ1

Commit message: Puse areas sin de aisleamento
Parts:
- added C175, C176: 220nF, Capacitor_SMD:C_0402_1005Metric, symbol Device:C_Small
Connections:
- net +3.3V_analog: now also C175.1, C176.1; no longer U28.12 (V-), U29.12 (V-)
- net GND: now also U28.12 (V-), U29.12 (V-), C175.2, C176.2
