File: PCB/Inverter/Primero_esquematico/pcb_logica.kicad_sch (KiCad schematic)
At the start: 13 parts

Commit message: Puse areas sin de aisleamento
Other:
- sheet F280049C ports: added GP_56_GD_FLT, GP_57_GD_RDY, GP_58_Reset_Pote; removed GP_22_GD_FLT, GP_34_Reset_Pote, GP_40_GD_RDY
Changed lines of the file:
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@@
 	)
 	(no_connect
-		(at 119.38 129.54)
+		(at 119.38 127)
 	)
 	(no_connect
@@
 	(wire
 		(pts
-			(xy 120.65 102.87) (xy 121.92 102.87)
-		)
-		(stroke
-			(width 0)
-			(type default)
-		)
-	)
-	(wire
-		(pts
 			(xy 33.02 110.49) (xy 40.64 110.49)
 		)
@@
 	(wire
 		(pts
-			(xy 119.38 104.14) (xy 120.65 104.14)
-		)
-		(stroke
-			(width 0)
-			(type default)
-		)
-	)
-	(wire
-		(pts
-			(xy 120.65 104.14) (xy 120.65 102.87)
-		)
-		(stroke
-			(width 0)
-			(type default)
-		)
-	)
-	(wire
-		(pts
 			(xy 218.44 135.89) (xy 232.41 135.89)
 		)
@@
 	(wire
 		(pts
-			(xy 121.92 125.73) (xy 120.65 125.73)
-		)
-		(stroke
-			(width 0)
-			(type default)
-		)
-	)
-	(wire
-		(pts
 			(xy 133.35 96.52) (xy 119.38 96.52)
 		)
@@
 	(wire
 		(pts
-			(xy 120.65 127) (xy 119.38 127)
+			(xy 119.38 135.89) (xy 120.65 135.89)
 		)
 		(stroke
@@
 	(wire
 		(pts
-			(xy 119.38 132.08) (xy 120.65 132.08)
+			(xy 119.38 133.35) (xy 120.65 133.35)
 		)
 		(stroke
@@
 	(wire
 		(pts
-			(xy 120.65 125.73) (xy 120.65 127)
-		)
-		(stroke
-			(width 0)
-			(type default)
-		)
-	)
-	(wire
-		(pts
 			(xy 219.71 90.17) (xy 220.98 90.17)
 		)
@@
 	(wire
 		(pts
-			(xy 120.65 132.08) (xy 120.65 130.81)
-		)
-		(stroke
-			(width 0)
-			(type default)
-		)
-	)
-	(wire
-		(pts
 			(xy 39.37 78.74) (xy 40.64 78.74)
 		)
@@
 	(wire
 		(pts
-			(xy 120.65 130.81) (xy 121.92 130.81)
+			(xy 218.44 128.27) (xy 232.41 128.27)
 		)
 		(stroke
@@
 	(wire
 		(pts
-			(xy 218.44 128.27) (xy 232.41 128.27)
+			(xy 39.37 83.82) (xy 40.64 83.82)
 		)
 		(stroke
@@
 	(wire
 		(pts
-			(xy 39.37 83.82) (xy 40.64 83.82)
+			(xy 219.71 85.09) (xy 220.98 85.09)
 		)
 		(stroke
@@
 	(wire
 		(pts
-			(xy 219.71 85.09) (xy 220.98 85.09)
+			(xy 264.16 92.71) (xy 259.08 92.71)
 		)
 		(stroke
@@
 	(wire
 		(pts
-			(xy 264.16 92.71) (xy 259.08 92.71)
+			(xy 119.38 130.81) (xy 120.65 130.81)
 		)
 		(stroke
@@
 		)
 	)
-	(hierarchical_label "GD_FLT"
+	(hierarchical_label "PWM_H_C"
 		(shape bidirectional)
-		(at 121.92 102.87 0)
+		(at 62.23 24.13 90)
 		(effects
 			(font
@@
 		)
 	)
-	(hierarchical_label "PWM_H_C"
+	(hierarchical_label "GD_FLT"
 		(shape bidirectional)
-		(at 62.23 24.13 90)
+		(at 120.65 130.81 0)
 		(effects
 			(font
@@
 	(hierarchical_label "Reset_Pote"
 		(shape bidirectional)
-		(at 121.92 125.73 0)
+		(at 120.65 135.89 0)
 		(effects
 			(font
@@
 	(hierarchical_label "GD_RDY"
 		(shape bidirectional)
-		(at 121.92 130.81 0)
+		(at 120.65 133.35 0)
 		(effects
 			(font
@@
 			)
 		)
-		(pin "GP_34_Reset_Pote" bidirectional
-			(at 119.38 127 0)
-			(effects
-				(font
-					(size 1.27 1.27)
-				)
-				(justify right)
-			)
-		)
 		(pin "GP_39_E_STOP" bidirectional
-			(at 119.38 129.54 0)
-			(effects
-				(font
-					(size 1.27 1.27)
-				)
-				(justify right)
-			)
-		)
-		(pin "GP_40_GD_RDY" bidirectional
-			(at 119.38 132.08 0)
+			(at 119.38 127 0)
 			(effects
 				(font
@@
 			)
 		)
-		(pin "GP_22_GD_FLT" bidirectional
-			(at 119.38 104.14 0)
+		(pin "GP_56_GD_FLT" bidirectional
+			(at 119.38 130.81 0)
+			(effects
+				(font
+					(size 1.27 1.27)
+				)
+				(justify right)
+			)
+		)
+		(pin "GP_57_GD_RDY" bidirectional
+			(at 119.38 133.35 0)
+			(effects
+				(font
+					(size 1.27 1.27)
+				)
+				(justify right)
+			)
+		)
+		(pin "GP_58_Reset_Pote" bidirectional
+			(at 119.38 135.89 0)
 			(effects
 				(font

Commit message: Falta poco
Parts:
- removed TP52, TP53, TP54, TP55, TP56, TP57, TP58, TP59, TP60, TP61, TP62, TP63, TP64: TestPoint, TestPoint:TestPoint_Pad_D1.0mm, symbol Connector:TestPoint
