File: PCB/Inverter/Primero_esquematico/comunicacionCAN.kicad_sch (KiCad schematic)
At the start: 12 parts, among them J3 347920040, J4 347920040, U31 ISO1042DWR, U32 ISO1042DWR

Commit message: correcciones de apps
Parts:
- removed D80, D81: PESD2CANFD24LT-QR, Package_TO_SOT_SMD:SOT-23, symbol Diode:SM712_SOT23
- added D82, D83: PESD5V0S2UAT,215, Package_TO_SOT_SMD:SOT-23, symbol Diode:SM712_SOT23
- renumbered C151 to C155, C152 to C156, C153 to C157, C154 to C158, J3 to J2, J4 to J3, R190 to R174, R191 to R175, U31 to U33, U32 to U34
Connections:
- net GND_Can_1: now also D82.3 (common)
- net GND_Can_2: now also D83.3 (common)
- net at J2.1, R174.2, U33.12 (CANL): now also D82.2 (A2)
- net at J2.2, R174.1, U33.13 (CANH): now also D82.1 (A1)
- net at J3.2, R175.1, U34.13 (CANH): now also D83.1 (A1)
- net at J3.1, R175.2, U34.12 (CANL): now also D83.2 (A2)
