File: PCB/FSAE-BaseBoard_v2/FSAE-BaseBoard.kicad_pcb (KiCad board)
At the start: 2 copper layers, 100 x 100 mm, 71 parts, among them J1 Conn_01x14_Socket, J10 Conn_01x03, J11 Zocalo_Resolver, J12 Bornera_Resolver, J13 Zocalo_Resolver, J14 Screw_Terminal_01x03, J15 Bornera_Encoder, J3 Conn_01x03, J4 Conn_01x02, J5 Conn_01x02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

Commit message: Actualizacion BaseBoard v2
Routing:
- net GND: track 10.1 -> 29.6 mm, vias 1 -> 3
- net +3.3V: track 356.6 -> 360.4 mm
- net /ESP32 C3 y S3/SENSOR_RPM: track 85.5 -> 87.3 mm
