File: PCB/Inverter/Primero_esquematico/_cowork_backup_20260628_231627/Primero_esquematico.kicad_pcb (KiCad board)
At the start: 4 copper layers, 342.5 x 268 mm, 586 parts, among them J1 349128023, J2 GT8E-5P-2H(55), J3 347920040, J4 347920040, J5 347928082, J6 348250125, SW1 IT-1181-180G-G, T1 750317595, T2 750317595, T3 750317595, T4 750317595, T5 750317595, T6 750317595, U10 UCC21750QDWRQ1, U11 LM25180QNGURQ1, U12 UCC21750QDWRQ1, U13 LM25180QNGURQ1, U14 UCC21750QDWRQ1, U15 F280049CPZS, U16 TPS3823-33DBVR, U17 AMC1301QDWVRQ1, U18 AMC1301QDWVRQ1, U19 AMC1301QDWVRQ1, U2 FS950R08A6P2BBPSA1, U20 AMC1301QDWVRQ1, U21 TLV9004QDRQ1, U23 LM25180QNGURQ1, U24 LP5907QMFX-3.3Q1, U25 TLV76733QWDRBRQ1, U26 TPS7A2050PDBVR, U27 REF2030-Q1, U28 TLV1704AQPWRQ1, U29 TLV1704AQPWRQ1, U3 LM25180QNGURQ1, U30 HAH3DR 800-S07/SP4, U31 ISO1042DWR, U32 ISO1042DWR, U33 SN65HVD82DR, U34 AM26LS32AIDR, U35 SN74LVC245ANSR, U36 TLV9004QDRQ1, U4 UCC21750QDWRQ1, U42 LP2951-5.0_VSSOP, U43 LP2951-5.0_VSSOP, U44 LP2951-5.0_VSSOP, U5 LM25180QNGURQ1, U6 UCC21750QDWRQ1, U7 LM25180QNGURQ1, U8 UCC21750QDWRQ1, U9 LM25180QNGURQ1, Y1 ABM8GAIG-20.000MHZ-8-7Z-T3

Commit message: Corregi cosas de la placa
Parts:
- removed the C10 at (282.8, 132.5)
- removed the C138 at (-67.8, 29.0)
- removed the C139 at (70.5, 255.8)
- removed the C140 at (70.5, 258.8)
- removed the C141 at (-54.3, 250.6)
- removed the C142 at (70.5, 264.9)
- removed the C143 at (-45.1, 32.5)
- removed the C144 at (77.7, 255.6)
- removed the C145 at (77.7, 258.1)
- removed the C146 at (77.7, 260.6)
- removed the C168 at (97.3, 280.2)
- removed the C169 at (-46.6, 250.6)
- removed the C170 at (83.1, 278.9)
- removed the C171 at (83.1, 281.4)
- removed the C172 at (83.1, 284.0)
- removed the C173 at (83.1, 286.5)
- removed C189, C190, C191, C192, C193, C194: 1uF, Capacitor_SMD:C_0603_1608Metric
- removed the C37 at (94.7, 294.1)
- removed the C39 at (96.1, 291.4)
- removed the C53 at (96.7, 275.9)
- removed C55: 10 uF, Capacitor_SMD:C_1206_3216Metric
- removed the C72 at (282.8, 134.5)
- removed the D75 at (-61.7, 29.4)
- removed the J1 at (-99.6, 30.3)
- removed the R20 at (279.9, 132.6)
- removed R217, R219, R221, R223: 780, Resistor_SMD:R_0402_1005Metric
- removed R218, R220, R222, R224: 6420, Resistor_SMD:R_0402_1005Metric
- removed R226, R227, R228: 330k, Resistor_SMD:R_0402_1005Metric
- removed U25: TLV76733QWDRBRQ1, Package_SON:VSON-8-1EP_3x3mm_P0.65mm_EP1.65x2.4mm
- removed U26: TPS7A2050PDBVR, Snapeda:DBV0005A-IPC_A
- removed U42, U43, U44: LP2951-5.0_VSSOP, Package_SO:VSSOP-8_3x3mm_P0.65mm
- added C117: 100nF, Capacitor_SMD:C_0603_1608Metric, F.Cu at (68.4, 253.9)
- added C118: 0,1uF, Capacitor_SMD:C_0805_2012Metric, F.Cu at (183.1, 91.4)
- added C119: 0,1uF, Capacitor_SMD:C_0603_1608Metric, F.Cu at (68.4, 256.4)
- added C120: 0,1uF, Capacitor_SMD:C_0805_2012Metric, F.Cu at (190.1, 105.9)
- added C122: 47nF, Capacitor_SMD:C_0402_1005Metric_Pad0.74x0.62mm_HandSolder, F.Cu at (14.5, 305.0)
- added C123: 1uF, Capacitor_SMD:C_0805_2012Metric, F.Cu at (3.71, 297.7)
- added C124: 0,1uF, Capacitor_SMD:C_0603_1608Metric, F.Cu at (10.9, 305.2)
- added C125: 0,1uF, Capacitor_SMD:C_0603_1608Metric, F.Cu at (10.9, 307.8)
- added C126: 0,1uF, Capacitor_SMD:C_0603_1608Metric, F.Cu at (10.9, 310.3)
- added C148: 220uF, Snapeda:WCAP-PSLC_8X11.7_DXL_, F.Cu at (-4.83, 291.2)
- added C149: 1uF, Capacitor_SMD:C_0805_2012Metric, F.Cu at (3.71, 300.8)
- added C150: 1uF, Capacitor_SMD:C_0805_2012Metric, F.Cu at (3.71, 303.8)
- added C151: 1uF, Capacitor_SMD:C_0805_2012Metric, F.Cu at (3.71, 306.8)
- added C152: 100nF, Capacitor_SMD:C_0603_1608Metric, F.Cu at (84.0, 244.2)
- added C153: 220uF, Snapeda:WCAP-PSLC_8X11.7_DXL_, F.Cu at (191.4, 254.8)
- added C178: 220uF, Snapeda:WCAP-PSLC_8X11.7_DXL_, F.Cu at (142.4, 234.8)
- added C2: 2.2nF, Capacitor_SMD:C_0603_1608Metric, F.Cu at (200.4, 263.5)
- added C20: 10pF, Capacitor_SMD:C_0402_1005Metric, F.Cu at (162.0, 248.6)
- added C31: 100nF, Capacitor_SMD:C_0402_1005Metric, F.Cu at (88.2, 222.3)
- added C32: 10 uF, Capacitor_SMD:C_1206_3216Metric, F.Cu at (89.6, 219.6)
- added C44: 100nF, Capacitor_SMD:C_0402_1005Metric, F.Cu at (59.3, 234.1)
- added C45: 10 uF, Capacitor_SMD:C_1206_3216Metric, F.Cu at (60.7, 231.5)
- added C59: 10pF, Capacitor_SMD:C_0402_1005Metric, F.Cu at (157.1, 248.6)
- added C7: 10pF, Capacitor_SMD:C_0402_1005Metric, F.Cu at (152.2, 248.6)
- added D75: SMDJ13A, Diode_SMD:D_SMC, F.Cu at (-11.6, 210.2)
- added D75: SMDJ13A, Diode_SMD:D_SMC, F.Cu at (141.5, 243.7)
- added D80: APT2012EC, LED_SMD:LED_0805_2012Metric, F.Cu at (13.8, 292.4)
- added J3: 349128023, Snapeda:CONN_SD-34912-001_02_MOL, F.Cu at (-51.9, 221.8)
- added PS1: NXJ1S0505T6MC-R7, Snapeda:CONV_NXJ1S0505T6MC-R7, F.Cu at (207.9, 221.6)
- added R1: 2k2, Resistor_SMD:R_0603_1608Metric, F.Cu at (200.4, 266.0)
- added R18: 10, Resistor_SMD:R_0402_1005Metric, F.Cu at (152.2, 246.7)
- added R2: 487k, Resistor_SMD:R_0402_1005Metric, F.Cu at (196.9, 260.7)
- added R3: 11k, Resistor_SMD:R_0402_1005Metric, F.Cu at (196.9, 262.7)
- added R32: 10, Resistor_SMD:R_0402_1005Metric, F.Cu at (162.0, 246.7)
- added R4: 49k9, Resistor_SMD:R_0402_1005Metric, F.Cu at (196.9, 264.7)
- added R5: 550, Resistor_SMD:R_0402_1005Metric, F.Cu at (196.9, 266.7)
- added TP1: TestPoint, TestPoint:TestPoint_Pad_D1.0mm, F.Cu at (199.3, 251.3)
- added TP2: TestPoint, TestPoint:TestPoint_Pad_D1.0mm, F.Cu at (199.3, 254.3)
- added TP36: TestPoint, TestPoint:TestPoint_Pad_D1.0mm, F.Cu at (-12.7, 300.0)
- added U1: TPS259621DDAT, Snapeda:IC_TPS259621DDAT, F.Cu at (190.7, 263.0)
- added U22: ADR130BUJZ-REEL7, NuevoGui:UJ_6_ADI-L, F.Cu at (181.7, 104.7)
- added U28: REF2030-Q1, Snapeda:SOT95P0280X110-5N, F.Cu at (-7.98, 313.6)
- added U39: TLV76733QWDRBRQ1, Package_SON:VSON-8-1EP_3x3mm_P0.65mm_EP1.65x2.4mm, F.Cu at (-2.10, 310.0)
- added U40: LP5907QMFX-3.3Q1, Package_TO_SOT_SMD:SC-74A-5_1.55x2.9mm_P0.95mm, F.Cu at (9.74, 288.6)
- C1: value 220uF -> 10uF; footprint Snapeda:WCAP-PSLC_8X11.7_DXL_ -> Capacitor_SMD:C_0603_1608Metric
- D1: value SMDJ13A -> APT2012EC; footprint Diode_SMD:D_SMC -> LED_SMD:LED_0805_2012Metric
- D76: value 1N4148WS-Q -> DFLZ24Q-7; footprint Diode_SMD:D_SOD-323F -> Diode_SMD:D_PowerDI-123
- D77: value SDM1U100S1F-7 -> 1N4148WS-Q; footprint Diode_SMD:D_SOD-123F -> Diode_SMD:D_SOD-323F
- D78: value SZMM5Z5V6T1G -> SDM1U100S1F-7; footprint Diode_SMD:D_SOD-523 -> Diode_SMD:D_SOD-123F
- D79: value APT2012EC -> SZMM5Z5V6T1G; footprint LED_SMD:LED_0805_2012Metric -> Diode_SMD:D_SOD-523
- R161: footprint Resistor_SMD:R_0603_1608Metric -> Resistor_SMD:R_0402_1005Metric
- U23: value LM25180QNGURQ1 -> R1S12-1205/HP; footprint NuevoGui:NGU0008C -> NuevoGui:SMD12_15.24X10.7X6.7_SINGLE&slash_DUAL_RCP-L
- U24: value LP5907QMFX-3.3Q1 -> LM25180QNGURQ1; footprint Package_TO_SOT_SMD:SC-74A-5_1.55x2.9mm_P0.95mm -> NuevoGui:NGU0008C
- U27: value REF2030-Q1 -> TPS7A2050PDBVR; footprint Snapeda:SOT95P0280X110-5N -> Snapeda:DBV0005A-IPC_A
- moved D1 365.9 mm to (200.0, 257.4), turned to 0 degrees
- moved C1 362.3 mm to (200.4, 261.0), turned to 0 degrees
- moved R159 289.6 mm to (7.39, 311.0), turned to 0 degrees
- moved R158 289.5 mm to (7.39, 309.0), turned to 0 degrees
- moved R157 287.4 mm to (7.39, 307.0), turned to 0 degrees
- moved R156 284.5 mm to (7.39, 305.0), turned to 0 degrees
- moved R161 283.5 mm to (7.39, 312.9), turned to 0 degrees
- moved D76 281.1 mm to (-8.15, 309.5), turned to 0 degrees
- moved L1 274.9 mm to (9.29, 292.2)
- moved Te1 274.7 mm to (-4.28, 302.0)
- moved R160 273.0 mm to (13.2, 294.9), turned to 0 degrees
- moved D79 269.2 mm to (8.84, 294.8), turned to 0 degrees
- moved U23 265.3 mm to (190.5, 97.0), turned to 0 degrees
- moved D78 265.2 mm to (4.29, 293.4), turned to 0 degrees
- moved D77 257.3 mm to (14.6, 287.7), turned to 0 degrees
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- renumbered C11 to C10, C120 to C100, C119 to C101, C121 to C102, C122 to C103, C123 to C104, C124 to C105, C125 to C106, C126 to C107, C127 to C108, C128 to C109, C12 to C11, C129 to C110, C130 to C111, C131 to C112, C132 to C113, C133 to C114, C134 to C115, C135 to C116, C15 to C12, C147 to C127, C148 to C128, C149 to C129, C150 to C130, C151 to C131, C152 to C132, C153 to C133, C154 to C134, C155 to C135, C156 to C136, C157 to C137, C158 to C138, C159 to C139, C160 to C140, C161 to C141, C162 to C142, C163 to C143, C164 to C144, C165 to C145, C166 to C146, C167 to C147, C16 to C15, C18 to C154, C34 to C155, C50 to C156, C66 to C157, C82 to C158, C98 to C159, C20 to C160, C36 to C161, C52 to C162, C68 to C163, C84 to C164, C100 to C165, C17 to C166, C19 to C167, C33 to C168, C35 to C169, C22 to C17, C49 to C170, C51 to C171, C65 to C172, C67 to C173, C81 to C174, C83 to C175, C97 to C176, C99 to C177, C21 to C18, C23 to C19, C25 to C21, C26 to C22, C27 to C23, C28 to C24, C31 to C25, C29 to C26, C30 to C27, C32 to C28, C38 to C30, C40 to C33, C41 to C34, C42 to C35, C43 to C36, C44 to C37, C47 to C38, C45 to C39, C6 to C4, C46 to C40, C48 to C41, C54 to C43, C56 to C46, C57 to C47, C58 to C48, C59 to C49, C60 to C50, C63 to C51, C61 to C52, C62 to C53, C64 to C54, C70 to C56, C69 to C57, C71 to C58, C7 to C6, C73 to C60, C74 to C61, C75 to C62, C76 to C63, C79 to C64, C77 to C65, C78 to C66, C80 to C67, C86 to C69, C85 to C70, C87 to C71, C88 to C72, C89 to C73, C90 to C74, C91 to C75, C92 to C76, C95 to C77, C93 to C78, C94 to C79, C9 to C8, C96 to C80, C101 to C82, C102 to C83, C103 to C84, C104 to C85, C105 to C86, C106 to C87, C107 to C88, C108 to C89, C10 to C9, C109 to C90, C110 to C91, C111 to C92, C112 to C93, C113 to C94, C114 to C95, C115 to C96, C116 to C97, C117 to C98, C118 to C99, D80 to D81, D81 to D82, J2 to J1, J6 to J2, J5 to J4, J4 to J6, J3 to J7, R9 to R10, R10 to R11, R13 to R12, R14 to R13, R12 to R14, R25 to R23, R23 to R24, R24 to R25, R27 to R26, R28 to R27, R26 to R28, R39 to R37, R37 to R38, R38 to R39, R41 to R40, R42 to R41, R40 to R42, R53 to R51, R51 to R52, R52 to R53, R55 to R54, R56 to R55, R54 to R56, R67 to R65, R65 to R66, R66 to R67, R69 to R68, R70 to R69, R68 to R70, R81 to R79, R79 to R80, R80 to R81, R83 to R82, R84 to R83, R82 to R84, R11 to R9, U28 to U29, U29 to U30, U30 to U31, U31 to U32, U32 to U33, U33 to U34, U34 to U35, U35 to U36, U36 to U37
Connections:
- net /pcb_potencia/Gate_Driver/GD_HS_1/+15V renamed /pcb_potencia/Gate_Driver/GDsupply/+15V
- net /pcb_potencia/Gate_Driver/GD_HS_1/-8V renamed /pcb_potencia/Gate_Driver/GDsupply/-8V
- net /pcb_potencia/Gate_Driver/GD_HS_1/DESAT renamed /pcb_potencia/Gate_Driver/GDsupply/DESAT
- net /pcb_potencia/Gate_Driver/GD_HS_1/Gate renamed /pcb_potencia/Gate_Driver/GDsupply/Gate
- net /pcb_potencia/Gate_Driver/GD_HS_1/ISO_GND renamed /pcb_potencia/Gate_Driver/GDsupply/ISO_GND
- net /pcb_potencia/Gate_Driver/GD_HS_2/+15V renamed /pcb_potencia/Gate_Driver/GDsupply1/+15V
- net /pcb_potencia/Gate_Driver/GD_HS_2/-8V renamed /pcb_potencia/Gate_Driver/GDsupply1/-8V
- net /pcb_potencia/Gate_Driver/GD_HS_2/DESAT renamed /pcb_potencia/Gate_Driver/GDsupply1/DESAT
- net /pcb_potencia/Gate_Driver/GD_HS_2/Gate renamed /pcb_potencia/Gate_Driver/GDsupply1/Gate
- net /pcb_potencia/Gate_Driver/GD_HS_2/S_HV renamed /pcb_potencia/Gate_Driver/GDsupply1/S_HV
- net /pcb_potencia/Gate_Driver/GD_HS_3/+15V renamed /pcb_potencia/Gate_Driver/GDsupply2/+15V
- net /pcb_potencia/Gate_Driver/GD_HS_3/-8V renamed /pcb_potencia/Gate_Driver/GDsupply2/-8V
- net /pcb_potencia/Gate_Driver/GD_HS_3/DESAT renamed /pcb_potencia/Gate_Driver/GDsupply2/DESAT
- net /pcb_potencia/Gate_Driver/GD_HS_3/Gate renamed /pcb_potencia/Gate_Driver/GDsupply2/Gate
- net /pcb_potencia/Gate_Driver/GD_HS_3/S_HV renamed /pcb_potencia/Gate_Driver/GDsupply2/S_HV
- net /pcb_potencia/Gate_Driver/GD_LS_1/+15V renamed /pcb_potencia/Gate_Driver/GDsupply5/+15V
- net /pcb_potencia/Gate_Driver/GD_LS_1/-8V renamed /pcb_potencia/Gate_Driver/GDsupply5/-8V
- net /pcb_potencia/Gate_Driver/GD_LS_1/DESAT renamed /pcb_potencia/Gate_Driver/GDsupply5/DESAT
- net /pcb_potencia/Gate_Driver/GD_LS_1/Gate renamed /pcb_potencia/Gate_Driver/GDsupply5/Gate
- net /pcb_potencia/Gate_Driver/GD_LS_2/+15V renamed /pcb_potencia/Gate_Driver/GDsupply4/+15V
- net /pcb_potencia/Gate_Driver/GD_LS_2/-8V renamed /pcb_potencia/Gate_Driver/GDsupply4/-8V
- net /pcb_potencia/Gate_Driver/GD_LS_2/DESAT renamed /pcb_potencia/Gate_Driver/GDsupply4/DESAT
- net /pcb_potencia/Gate_Driver/GD_LS_2/Gate renamed /pcb_potencia/Gate_Driver/GDsupply4/Gate
- net /pcb_potencia/Gate_Driver/GD_LS_3/+15V renamed /pcb_potencia/Gate_Driver/GDsupply3/+15V
- net /pcb_potencia/Gate_Driver/GD_LS_3/-8V renamed /pcb_potencia/Gate_Driver/GDsupply3/-8V
- net /pcb_potencia/Gate_Driver/GD_LS_3/DESAT renamed /pcb_potencia/Gate_Driver/GDsupply3/DESAT
- net /pcb_potencia/Gate_Driver/GD_LS_3/Gate renamed /pcb_potencia/Gate_Driver/GDsupply3/Gate
- C1 pad 1: +12V -> +12VA
- C1 pad 2: GND -> GND1
- C10 pad 1: GND -> GND1
- C11 pad 1: GND -> GND1
- C113 pad 2: GND -> GND1
- C114 pad 2: GND -> GND1
- C115 pad 2: GND -> GND1
- C116 pad 2: GND -> GND1
- C12 pad 1: GND -> GND1
- C13 pad 1: GNDPWR -> /pcb_potencia/Gate_Driver/GDsupply4/ISO_GND
- C14 pad 2: GNDPWR -> /pcb_potencia/Gate_Driver/GDsupply4/ISO_GND
- C142 pad 1: GND -> GND1
- C143 pad 1: GND -> GND1
- C144 pad 1: GND -> GND1
- C145 pad 2: GND -> GND1
- C146 pad 2: GND -> GND1
- C147 pad 2: GND -> GND1
- C15 pad 1: GNDPWR -> /pcb_potencia/Gate_Driver/GDsupply4/ISO_GND
- C154 pad 1: GNDPWR -> /pcb_potencia/Gate_Driver/GDsupply4/ISO_GND
- C155 pad 1: GNDPWR -> /pcb_potencia/Gate_Driver/GDsupply3/ISO_GND
- C156 pad 1: /pcb_potencia/Gate_Driver/GD_HS_3/ISO_GND -> /pcb_potencia/Gate_Driver/GDsupply2/ISO_GND
- C157 pad 1: /pcb_potencia/Gate_Driver/GD_HS_2/ISO_GND -> /pcb_potencia/Gate_Driver/GDsupply1/ISO_GND
- C158 pad 1: GNDPWR -> /pcb_potencia/Gate_Driver/GDsupply5/ISO_GND
- C160 pad 1: GNDPWR -> /pcb_potencia/Gate_Driver/GDsupply4/ISO_GND
- C161 pad 1: GNDPWR -> /pcb_potencia/Gate_Driver/GDsupply3/ISO_GND
- C162 pad 1: /pcb_potencia/Gate_Driver/GD_HS_3/ISO_GND -> /pcb_potencia/Gate_Driver/GDsupply2/ISO_GND
- C163 pad 1: /pcb_potencia/Gate_Driver/GD_HS_2/ISO_GND -> /pcb_potencia/Gate_Driver/GDsupply1/ISO_GND
- C164 pad 1: GNDPWR -> /pcb_potencia/Gate_Driver/GDsupply5/ISO_GND
- C166 pad 2: GNDPWR -> /pcb_potencia/Gate_Driver/GDsupply4/ISO_GND
- C167 pad 2: GNDPWR -> /pcb_potencia/Gate_Driver/GDsupply4/ISO_GND
- C168 pad 2: GNDPWR -> /pcb_potencia/Gate_Driver/GDsupply3/ISO_GND
- C169 pad 2: GNDPWR -> /pcb_potencia/Gate_Driver/GDsupply3/ISO_GND
- C17 pad 1: GNDPWR -> /pcb_potencia/Gate_Driver/GDsupply3/ISO_GND
- C170 pad 2: /pcb_potencia/Gate_Driver/GD_HS_3/ISO_GND -> /pcb_potencia/Gate_Driver/GDsupply2/ISO_GND
- C171 pad 2: /pcb_potencia/Gate_Driver/GD_HS_3/ISO_GND -> /pcb_potencia/Gate_Driver/GDsupply2/ISO_GND
- C172 pad 2: /pcb_potencia/Gate_Driver/GD_HS_2/ISO_GND -> /pcb_potencia/Gate_Driver/GDsupply1/ISO_GND
- C173 pad 2: /pcb_potencia/Gate_Driver/GD_HS_2/ISO_GND -> /pcb_potencia/Gate_Driver/GDsupply1/ISO_GND
- C174 pad 2: GNDPWR -> /pcb_potencia/Gate_Driver/GDsupply5/ISO_GND
- C175 pad 2: GNDPWR -> /pcb_potencia/Gate_Driver/GDsupply5/ISO_GND
- C18 pad 2: +12V -> +12VA
- C19 pad 1: +12V -> +12VA
- C23 pad 1: GND -> GND1
- C24 pad 1: GND -> GND1
- C25 pad 1: GND -> GND1
- C26 pad 1: GNDPWR -> /pcb_potencia/Gate_Driver/GDsupply3/ISO_GND
- C27 pad 2: GNDPWR -> /pcb_potencia/Gate_Driver/GDsupply3/ISO_GND
- C28 pad 1: GNDPWR -> /pcb_potencia/Gate_Driver/GDsupply3/ISO_GND
- C30 pad 1: /pcb_potencia/Gate_Driver/GD_HS_3/ISO_GND -> /pcb_potencia/Gate_Driver/GDsupply2/ISO_GND
- C33 pad 2: /pcb_potencia/Gate_Driver/GD_HS_3/ISO_GND -> /pcb_potencia/Gate_Driver/GDsupply2/ISO_GND
- C35 pad 2: GND -> GND1
- C36 pad 1: GND -> GND1
- C37 pad 1: GND -> GND1
- C38 pad 1: GND -> GND1
- C39 pad 1: /pcb_potencia/Gate_Driver/GD_HS_3/ISO_GND -> /pcb_potencia/Gate_Driver/GDsupply2/ISO_GND
- C4 pad 1: GNDPWR -> /pcb_potencia/Gate_Driver/GDsupply4/ISO_GND
- C40 pad 2: /pcb_potencia/Gate_Driver/GD_HS_3/ISO_GND -> /pcb_potencia/Gate_Driver/GDsupply2/ISO_GND
- C41 pad 1: /pcb_potencia/Gate_Driver/GD_HS_3/ISO_GND -> /pcb_potencia/Gate_Driver/GDsupply2/ISO_GND
- C43 pad 1: /pcb_potencia/Gate_Driver/GD_HS_2/ISO_GND -> /pcb_potencia/Gate_Driver/GDsupply1/ISO_GND
- C46 pad 2: /pcb_potencia/Gate_Driver/GD_HS_2/ISO_GND -> /pcb_potencia/Gate_Driver/GDsupply1/ISO_GND
- C48 pad 2: GND -> GND1
- C49 pad 1: GND -> GND1
- C5 pad 2: +12V -> +12VA
- C50 pad 1: GND -> GND1
- C51 pad 1: GND -> GND1
- C52 pad 1: /pcb_potencia/Gate_Driver/GD_HS_2/ISO_GND -> /pcb_potencia/Gate_Driver/GDsupply1/ISO_GND
- C53 pad 2: /pcb_potencia/Gate_Driver/GD_HS_2/ISO_GND -> /pcb_potencia/Gate_Driver/GDsupply1/ISO_GND
- C54 pad 1: /pcb_potencia/Gate_Driver/GD_HS_2/ISO_GND -> /pcb_potencia/Gate_Driver/GDsupply1/ISO_GND
- C56 pad 1: GNDPWR -> /pcb_potencia/Gate_Driver/GDsupply5/ISO_GND
- C57 pad 2: +12V -> +12VA
- C58 pad 1: +12V -> +12VA
- C6 pad 1: +12V -> +12VA
- C62 pad 1: GND -> GND1
- C63 pad 1: GND -> GND1
- C64 pad 1: GND -> GND1
- C65 pad 1: GNDPWR -> /pcb_potencia/Gate_Driver/GDsupply5/ISO_GND
- C66 pad 2: GNDPWR -> /pcb_potencia/Gate_Driver/GDsupply5/ISO_GND
- C67 pad 1: GNDPWR -> /pcb_potencia/Gate_Driver/GDsupply5/ISO_GND
- C70 pad 2: +12V -> +12VA
- C71 pad 1: +12V -> +12VA
- C72 pad 1: /pcb_potencia/Gate_Driver/GD_HS_1/S_HV -> /pcb_potencia/Gate_Driver/GDsupply/S_HV
- C74 pad 2: GND -> GND1
- C75 pad 1: GND -> GND1
- C76 pad 1: GND -> GND1
- C77 pad 1: GND -> GND1
- D1 pad 1: +12V -> GND1
- D1 pad 2: GND -> /pcb_potencia/12V_Filtrada/Led_12V_Ok
- D10 pad 2: GNDPWR -> /pcb_potencia/Gate_Driver/GDsupply4/ISO_GND
- D11 pad 2: +12V -> +12VA
- D15 pad 2: GNDPWR -> /pcb_potencia/Gate_Driver/GDsupply4/ISO_GND
- D16 pad 1: GNDPWR -> /pcb_potencia/Gate_Driver/GDsupply4/ISO_GND
- D19 pad 2: GNDPWR -> /pcb_potencia/Gate_Driver/GDsupply3/ISO_GND
- D21 pad 2: GNDPWR -> /pcb_potencia/Gate_Driver/GDsupply3/ISO_GND
- D22 pad 2: +12V -> +12VA
- D26 pad 2: GNDPWR -> /pcb_potencia/Gate_Driver/GDsupply3/ISO_GND
- D27 pad 1: GNDPWR -> /pcb_potencia/Gate_Driver/GDsupply3/ISO_GND
- D3 pad 1: GND -> GND1
- D30 pad 2: /pcb_potencia/Gate_Driver/GD_HS_3/ISO_GND -> /pcb_potencia/Gate_Driver/GDsupply2/ISO_GND
- D32 pad 2: /pcb_potencia/Gate_Driver/GD_HS_3/ISO_GND -> /pcb_potencia/Gate_Driver/GDsupply2/ISO_GND
- D33 pad 2: +12V -> +12VA
- D37 pad 2: /pcb_potencia/Gate_Driver/GD_HS_3/ISO_GND -> /pcb_potencia/Gate_Driver/GDsupply2/ISO_GND
- D38 pad 1: /pcb_potencia/Gate_Driver/GD_HS_3/ISO_GND -> /pcb_potencia/Gate_Driver/GDsupply2/ISO_GND
- D4 pad 1: GND -> GND1
- D41 pad 2: /pcb_potencia/Gate_Driver/GD_HS_2/ISO_GND -> /pcb_potencia/Gate_Driver/GDsupply1/ISO_GND
- D43 pad 2: /pcb_potencia/Gate_Driver/GD_HS_2/ISO_GND -> /pcb_potencia/Gate_Driver/GDsupply1/ISO_GND
- D44 pad 2: +12V -> +12VA
- D48 pad 2: /pcb_potencia/Gate_Driver/GD_HS_2/ISO_GND -> /pcb_potencia/Gate_Driver/GDsupply1/ISO_GND
- D49 pad 1: /pcb_potencia/Gate_Driver/GD_HS_2/ISO_GND -> /pcb_potencia/Gate_Driver/GDsupply1/ISO_GND
- D5 pad 1: GND -> GND1
- D52 pad 2: GNDPWR -> /pcb_potencia/Gate_Driver/GDsupply5/ISO_GND
- D54 pad 2: GNDPWR -> /pcb_potencia/Gate_Driver/GDsupply5/ISO_GND
- D55 pad 2: +12V -> +12VA
- D59 pad 2: GNDPWR -> /pcb_potencia/Gate_Driver/GDsupply5/ISO_GND
- D60 pad 1: GNDPWR -> /pcb_potencia/Gate_Driver/GDsupply5/ISO_GND
- D66 pad 2: +12V -> +12VA
- D76 pad 1: Net-(D75-K) -> Net-(D76-K)
- D77 pad 1: /pcb_logica/LogicSupply/5V_FB -> Net-(D76-K)
- D78 pad 2: GND -> Net-(D78-A)
- D79 pad 1: GND -> /pcb_logica/LogicSupply/5V_FB
- D79 pad 2: Net-(D79-A) -> GND
- D8 pad 2: GNDPWR -> /pcb_potencia/Gate_Driver/GDsupply4/ISO_GND
- J1 pad 1: +5V -> +5VA
- J1 pad 2: GND -> GND1
- L1 pad 2: Net-(D75-A) -> Net-(D76-A)
- R10 pad 1: +12V -> +12VA
- R138 pad 1: +1V5 -> +1VA5
- R141 pad 1: +1V5 -> +1VA5
- R144 pad 1: +1V5 -> +1VA5
- R147 pad 1: +1V5 -> +1VA5
- R156 pad 1: Net-(D75-A) -> Net-(D76-A)
- R156 pad 2: Net-(U23-EN_UVLO) -> Net-(U24-EN_UVLO)
- R157 pad 1: Net-(U23-EN_UVLO) -> Net-(U24-EN_UVLO)
- R158 pad 1: Net-(U23-TC) -> Net-(U24-TC)
- R159 pad 1: Net-(U23-TC) -> Net-(U24-TC)
- R159 pad 2: Net-(U23-RSET) -> Net-(U24-RSET)
- R160 pad 1: Net-(D76-A) -> Net-(D77-A)
- R160 pad 2: Net-(U23-FB) -> Net-(U24-FB)
- R161 pad 2: Net-(D79-A) -> Net-(D80-A)
- R205 pad 2: GND -> GND1
- R206 pad 2: GND -> GND1
- R207 pad 2: GND -> GND1
- R24 pad 1: +12V -> +12VA
- R38 pad 1: +12V -> +12VA
- R52 pad 1: +12V -> +12VA
- R6 pad 2: +3.3_digital -> +3.3VA
- R66 pad 1: +12V -> +12VA
- R7 pad 2: +3.3_digital -> +3.3VA
- R74 pad 1: Net-(C72-Pad1) -> /pcb_potencia/Gate_Driver/GDsupply5/S_HV
- R74 pad 2: /pcb_potencia/Gate_Driver/GD_LS_2/S_HV -> Net-(U12-AIN)
- R8 pad 2: +3.3_digital -> +3.3VA
- R80 pad 1: +12V -> +12VA
- R88 pad 1: /pcb_potencia/Gate_Driver/GD_HS_1/S_HV -> /pcb_potencia/Gate_Driver/GDsupply/S_HV
- T1 pad 4: +12V -> +12VA
- T1 pad 6: GNDPWR -> /pcb_potencia/Gate_Driver/GDsupply4/ISO_GND
- T1 pad 7: GNDPWR -> /pcb_potencia/Gate_Driver/GDsupply4/ISO_GND
- T2 pad 4: +12V -> +12VA
- T2 pad 6: GNDPWR -> /pcb_potencia/Gate_Driver/GDsupply3/ISO_GND
- T2 pad 7: GNDPWR -> /pcb_potencia/Gate_Driver/GDsupply3/ISO_GND
- T3 pad 4: +12V -> +12VA
- T3 pad 6: /pcb_potencia/Gate_Driver/GD_HS_3/ISO_GND -> /pcb_potencia/Gate_Driver/GDsupply2/ISO_GND
- T3 pad 7: /pcb_potencia/Gate_Driver/GD_HS_3/ISO_GND -> /pcb_potencia/Gate_Driver/GDsupply2/ISO_GND
- T4 pad 4: +12V -> +12VA
- T4 pad 6: /pcb_potencia/Gate_Driver/GD_HS_2/ISO_GND -> /pcb_potencia/Gate_Driver/GDsupply1/ISO_GND
- T4 pad 7: /pcb_potencia/Gate_Driver/GD_HS_2/ISO_GND -> /pcb_potencia/Gate_Driver/GDsupply1/ISO_GND
- T5 pad 4: +12V -> +12VA
- T5 pad 6: GNDPWR -> /pcb_potencia/Gate_Driver/GDsupply5/ISO_GND
- T5 pad 7: GNDPWR -> /pcb_potencia/Gate_Driver/GDsupply5/ISO_GND
- T6 pad 4: +12V -> +12VA
- TH1 pad 1: GNDPWR -> /pcb_potencia/Gate_Driver/GDsupply4/ISO_GND
- TH1 pad 2: /pcb_potencia/Gate_Driver/GD_LS_2/S_HV -> /pcb_potencia/Gate_Driver/GDsupply4/S_HV
- TP24 pad 1: GND -> GND1
- TP27 pad 1: GND -> GND1
- TP29 pad 1: GND -> GND1
- TP30 pad 1: GND -> GND1
- TP40 pad 1: GND -> GND1
- TP49 pad 1: +5VA -> +5V
- TP50 pad 1: +3.3VA -> +3.3V
- TP51 pad 1: +1VA5 -> +1V5
- Te1 pad 1: Net-(D76-A) -> Net-(D77-A)
- Te1 pad 4: Net-(D75-A) -> Net-(D76-A)
- Te1 pad 7: Net-(D77-A) -> Net-(D78-A)
- Te1 pad 8: Net-(D77-A) -> Net-(D78-A)
- U10 pad 3: /pcb_potencia/Gate_Driver/GD_HS_2/ISO_GND -> /pcb_potencia/Gate_Driver/GDsupply1/ISO_GND
- U10 pad 9: GND -> GND1
- U11 pad 3: +12V -> +12VA
- U12 pad 1: /pcb_potencia/Gate_Driver/GD_LS_1/S_HV -> Net-(U12-AIN)
- U12 pad 16: /pcb_potencia/Gate_Driver/GD_LS_1/APWM -> Net-(U12-APWM)
- U12 pad 3: GNDPWR -> /pcb_potencia/Gate_Driver/GDsupply5/ISO_GND
- U12 pad 9: GND -> GND1
- U13 pad 3: +12V -> +12VA
- U14 pad 9: GND -> GND1
- U17 pad 1: /pcb_potencia/Gate_Driver/5V_ISO_3 -> /pcb_potencia/Gate_Driver/SensorTension/5V_ISO
- U17 pad 5: GND -> GND1
- U18 pad 1: /pcb_potencia/Gate_Driver/5V_ISO_1 -> /pcb_potencia/Gate_Driver/SensorTension/5V_ISO
- U18 pad 5: GND -> GND1
- U19 pad 1: /pcb_potencia/Gate_Driver/5V_ISO_1 -> /pcb_potencia/Gate_Driver/SensorTension/5V_ISO
- U19 pad 5: GND -> GND1
- U2 pad E1: /pcb_potencia/Gate_Driver/GD_HS_1/S_HV -> unconnected-(U2-PadE1)
- U2 pad E3: /pcb_potencia/Gate_Driver/GD_HS_2/ISO_GND -> unconnected-(U2-PadE3)
- U2 pad E5: /pcb_potencia/Gate_Driver/GD_HS_3/ISO_GND -> unconnected-(U2-PadE5)
- U2 pad T1: /pcb_potencia/Gate_Driver/GD_HS_1/S_HV -> /pcb_potencia/Gate_Driver/GDsupply/S_HV
- U2 pad T4: /pcb_potencia/Gate_Driver/GD_HS_2/ISO_GND -> /pcb_potencia/Gate_Driver/GDsupply1/ISO_GND
- U2 pad T6: /pcb_potencia/Gate_Driver/GD_HS_3/ISO_GND -> /pcb_potencia/Gate_Driver/GDsupply2/ISO_GND
- U20 pad 1: /pcb_potencia/Gate_Driver/5V_ISO_2 -> /pcb_potencia/Gate_Driver/SensorTension/5V_ISO
- U20 pad 5: GND -> GND1
- U21 pad 10: GND -> GND1
- U23 pad 1: Net-(D76-A) -> +12VF
- U23 pad 2: Net-(U23-FB) -> GND1
- U23 pad 3: Net-(D75-A) -> unconnected-(U23-NC-Pad3)
- U23 pad 5: Net-(U23-SS_BIAS) -> GNDPWR
- U23 pad 6: Net-(U23-TC) -> unconnected-(U23-NC-Pad6)
- U23 pad 7: Net-(U23-RSET) -> unconnected-(U23-NC-Pad7)
- U23 pad 8: GND -> /pcb_potencia/Gate_Driver/SensorTension/5V_ISO
- U24 pad 1: /pcb_logica/LogicSupply/5V_FB -> Net-(D77-A)
- U24 pad 2: GND -> Net-(U24-FB)
- U24 pad 3: /pcb_logica/LogicSupply/5V_FB -> Net-(D76-A)
- U24 pad 4: unconnected-(U24-NC-Pad4) -> Net-(U24-EN_UVLO)
- U24 pad 5: +3.3V_analog -> Net-(U24-SS_BIAS)
- U27 pad 1: +1V5 -> /pcb_logica/LogicSupply/5V_FB
- U27 pad 3: +5V -> /pcb_logica/LogicSupply/5V_FB
- U27 pad 4: +5V -> unconnected-(U27-N/C-Pad4)
- U27 pad 5: +3V0 -> +5V
- U3 pad 3: +12V -> +12VA
- U31 pad 4: GND -> GND1
- U31 pad 5: +5V -> +5VA
- U37 pad 10: GND -> GND1
- U4 pad 1: /pcb_potencia/Gate_Driver/GD_LS_2/S_HV -> Net-(U4-AIN)
- U4 pad 16: /pcb_potencia/Gate_Driver/GD_LS_2/APWM -> Net-(U4-APWM)
- U4 pad 3: GNDPWR -> /pcb_potencia/Gate_Driver/GDsupply4/ISO_GND
- U4 pad 9: GND -> GND1
- U5 pad 3: +12V -> +12VA
- U6 pad 1: /pcb_potencia/Gate_Driver/GD_LS_3/S_HV -> Net-(U6-AIN)
- U6 pad 16: /pcb_potencia/Gate_Driver/GD_LS_3/APWM -> Net-(U6-APWM)
- U6 pad 3: GNDPWR -> /pcb_potencia/Gate_Driver/GDsupply3/ISO_GND
- U6 pad 9: GND -> GND1
- U7 pad 3: +12V -> +12VA
- U8 pad 3: /pcb_potencia/Gate_Driver/GD_HS_3/ISO_GND -> /pcb_potencia/Gate_Driver/GDsupply2/ISO_GND
- U8 pad 9: GND -> GND1
- U9 pad 3: +12V -> +12VA
