File: PCB/Inverter/Primero_esquematico/_cowork_backup_20260628_231627/Primero_esquematico.kicad_sch (KiCad schematic)
At the start: 3 parts, among them J1 349128023

Commit message: Corregi cosas de la placa
Parts:
- renumbered C1 to C178, D1 to D75, J1 to J3
Other:
- sheet pcb_logica ports: added 1.5V_De_Logic, 12V_De_Logic, 3.3V_De_Logic, 5V_De_Logic; removed none
- sheet pcb_potencia ports: added 1.5V_De_Pote, 12V_De_Pote, 3.3V_De_Pote, 5V_De_Pote; removed none
- note removed: "Power Flag"
- moved on the sheet: C178, D75, J3
