File: PCB/Inverter/Primero_esquematico/_cowork_backup_20260628_231627/g_driver.kicad_sch (KiCad schematic)
At the start: 20 parts, among them U2 FS950R08A6P2BBPSA1

Commit message: Corregi cosas de la placa
Parts:
- removed C10: 220nF, Capacitor_SMD:C_0402_1005Metric, symbol Device:C
- removed C72: 100nF, Capacitor_SMD:C_0402_1005Metric, symbol Device:C
- removed R20: 360, Resistor_SMD:R_0402_1005Metric, symbol Device:R
Connections:
- net GND is gone; now on net GND1: D3.1 (K), D4.1 (K), D5.1 (K)
- net GDsupply/S_HV: no longer U2.E1
- net GDsupply1/ISO_GND: no longer U2.E3
- net GDsupply2/ISO_GND: no longer U2.E5
- net GNDPWR: no longer TH1.1
- net +3.3_digital renamed +3.3VA
- new net GDsupply4/ISO_GND: TH1.1
- no-connect marks 4 -> 9
Other:
- sheet GD_HS_1 renamed GDsupply
- sheet GD_HS_2 renamed GDsupply1
- sheet GD_HS_3 renamed GDsupply2
- sheet GD_LS_1 renamed GDsupply5
- sheet GD_LS_2 renamed GDsupply4
- sheet GD_LS_3 renamed GDsupply3
- added sheet gate_driver_LS (gate_driver_LS.kicad_sch)
- sheet GDsupply: file GD_HS.kicad_sch -> GDsupply.kicad_sch
- sheet GDsupply1: file GD_HS.kicad_sch -> GDsupply.kicad_sch
- sheet GDsupply2: file GD_HS.kicad_sch -> GDsupply.kicad_sch
- sheet GDsupply3: file GD_LS.kicad_sch -> GDsupply.kicad_sch
- sheet GDsupply3 ports: added 15V_ISO; removed 5V_ISO
- sheet GDsupply4: file GD_LS.kicad_sch -> GDsupply.kicad_sch
- sheet GDsupply4 ports: added 15V_ISO; removed 5V_ISO
- sheet GDsupply5: file GD_LS.kicad_sch -> GDsupply.kicad_sch
- sheet GDsupply5 ports: added 15V_ISO; removed 5V_ISO
- sheet SensorTension ports: added none; removed 5V_ISO_1, 5V_ISO_2, 5V_ISO_3
- moved on the sheet: TH1, TP10, TP11, TP3, TP4, TP5, TP6, TP7, TP8, TP9
