File: PCB/InverterV2.0/Primero_esquematico/Primero_esquematico.kicad_pcb (KiCad board)
At the start: 6 copper layers, 220 x 140 mm, 545 parts, among them J10 440670201, J3 347920040, J4 347928082, J5 348250125, J6 347928082, J7 1053091205, J8 1053091205, J9 1053091205, Q1 IRF4905STRLPBF, SW1 IT-1187-160GM-G, T1 750317595, T2 750317595, T3 750317595, T4 750317595, T5 750317595, T6 750317595, U1 FS950R08A6P2BBPSA1, U10 LM25180QNGURQ1, U11 UCC21750QDWRQ1, U12 UCC21750QDWRQ1, U13 LM25180QNGURQ1, U14 LP2951-5.0_VSSOP, U15 LM25180QNGURQ1, U16 UCC21750QDWRQ1, U17 F280049CPZS, U18 TPS3823-33DBVR, U19 AMC1311BQDWVRQ1, U2 UCC21750QDWRQ1, U20 AMC1311BQDWVRQ1, U21 AMC1311BQDWVRQ1, U22 AMC1311BQDWVRQ1, U23 TLV9004QDRQ1, U24 TPS7A2050PDBVR, U25 LM25180QNGURQ1, U26 LP5907QMFX-3.3Q1, U27 TPS7A2050PDBVR, U28 TLV76733QWDRBRQ1, U29 REF2030-Q1, U3 LM25180QNGURQ1, U30 TLV1702AQDGKRQ1, U31 TPD4E05U06DQA, U32 TPD4E05U06DQA, U33 ISO1042DWR, U34 ISO1042DWR, U35 SN65HVD82DR, U36 AM26LS32AIDR, U37 SN74LVC245ANSR, U38 TPD4E05U06DQA, U39 OPA2196xD, U4 LP2951-5.0_VSSOP, U40 TLV1701AQDCKRQ1, U41 OPA4991QPWRQ1, U5 UCC21750QDWRQ1, U6 LM25180QNGURQ1, U7 LP2951-5.0_VSSOP, U8 LM25180QNGURQ1, U9 UCC21750QDWRQ1, Y1 ABM8GAIG-20.000MHZ-8-7Z-T3

Commit message: aislacion encoder
Parts:
- added J11: 347920040, Snapeda:CONN04_34792_MOL, F.Cu at (-131.9, 90.0)
- added PS2: MEV1S1205SC, Snapeda:MEV1S1205SC, F.Cu at (-134.6, 65.0)
- added R146: 0, Resistor_SMD:R_0603_1608Metric, F.Cu at (-110.9, 78.3)
- added R147: 0, Resistor_SMD:R_0603_1608Metric, F.Cu at (-116.9, 82.8)
- added R148: 0, Resistor_SMD:R_0603_1608Metric, F.Cu at (-116.9, 73.8)
- added R149: 0, Resistor_SMD:R_0603_1608Metric, F.Cu at (-110.9, 73.8)
- added R150: 0, Resistor_SMD:R_0603_1608Metric, F.Cu at (-116.9, 87.3)
- added R151: 0, Resistor_SMD:R_0603_1608Metric, F.Cu at (-116.9, 78.3)
- added U42: ISO7710FDR, Snapeda:D0008B_HV, F.Cu at (-107.3, 47.6)
- U37: value SN74LVC245ANSR -> ISOW7843DWER; footprint Snapeda:NS20-L -> Snapeda:DWE0016A
- moved U37 168.2 mm to (-109.3, 64.7)
- moved J5 161.5 mm to (-130.5, 51.0), turned to 0 degrees
- moved J3 105.9 mm to (-131.9, 78.7)
- moved C161 84.7 mm to (-41.4, 101.8)
- moved C162 84.7 mm to (-41.2, 115.6)
- moved R180 84.7 mm to (-33.6, 99.7)
- moved R184 84.7 mm to (-38.7, 115.6)
- moved TP19 84.7 mm to (-18.9, 104.4)
- moved TP21 84.7 mm to (-18.9, 107.0)
- moved TP22 84.7 mm to (-18.0, 109.6)
- moved U32 84.7 mm to (-62.1, 109.1)
- moved C159 84.7 mm to (-44.9, 99.2)
- moved C160 84.7 mm to (-24.6, 98.0)
- moved C163 84.7 mm to (-45.5, 104.3)
- moved C164 84.7 mm to (-34.3, 104.3)
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Connections:
- net /pcb_logica/Temp_PCB renamed /pcb_logica/Temp_Motor
- C19 pad 2: +12V -> Net-(D21-A)
- C20 pad 1: +12V -> Net-(D21-A)
- C3 pad 2: +12V -> Net-(D10-A)
- C34 pad 2: +12V -> Net-(D32-A)
- C36 pad 1: +12V -> Net-(D32-A)
- C4 pad 1: +12V -> Net-(D10-A)
- C50 pad 2: +12V -> Net-(D43-A)
- C52 pad 1: +12V -> Net-(D43-A)
- C67 pad 2: +12V -> Net-(D54-A)
- C68 pad 1: +12V -> Net-(D54-A)
- C82 pad 2: +12V -> Net-(D65-A)
- C84 pad 1: +12V -> Net-(D65-A)
- D10 pad 2: +12V -> Net-(D10-A)
- D21 pad 2: +12V -> Net-(D21-A)
- D32 pad 2: +12V -> Net-(D32-A)
- D43 pad 2: +12V -> Net-(D43-A)
- D54 pad 2: +12V -> Net-(D54-A)
- D65 pad 2: +12V -> Net-(D65-A)
- J3 pad 1: Net-(D83-A2) -> GND_Can
- J3 pad 2: Net-(D83-A1) -> Net-(D83-A2)
- J3 pad 3: Net-(D82-A2) -> Net-(D83-A1)
- J3 pad 4: Net-(D82-A1) -> +5V_Can
- J5 pad 1: /pcb_logica/encoder/Clock+ -> /pcb_logica/A
- J5 pad 10: /pcb_logica/encoder/Data+ -> unconnected-(J5-Pad10)
- J5 pad 11: /pcb_logica/encoder/B- -> unconnected-(J5-Pad11)
- J5 pad 12: /pcb_logica/encoder/B+ -> unconnected-(J5-Pad12)
- J5 pad 2: /pcb_logica/encoder/Clock- -> /pcb_logica/B
- J5 pad 3: /pcb_logica/encoder/A- -> /pcb_logica/Z
- J5 pad 4: /pcb_logica/encoder/A+ -> /pcb_logica/Data
- J5 pad 5: +5V_digital -> unconnected-(J5-Pad5)
- J5 pad 6: GND -> unconnected-(J5-Pad6)
- J5 pad 7: /pcb_logica/encoder/Z+ -> unconnected-(J5-Pad7)
- J5 pad 8: /pcb_logica/encoder/Z- -> unconnected-(J5-Pad8)
- J5 pad 9: /pcb_logica/encoder/Data- -> unconnected-(J5-Pad9)
- R20 pad 1: +12V -> Net-(D21-A)
- R30 pad 1: +12V -> Net-(D32-A)
- R44 pad 1: +12V -> Net-(D43-A)
- R61 pad 1: +12V -> Net-(D54-A)
- R7 pad 1: +12V -> Net-(D10-A)
- R71 pad 1: +12V -> Net-(D65-A)
- T1 pad 4: +12V -> Net-(D10-A)
- T2 pad 4: +12V -> Net-(D21-A)
- T3 pad 4: +12V -> Net-(D32-A)
- T4 pad 4: +12V -> Net-(D43-A)
- T5 pad 4: +12V -> Net-(D54-A)
- T6 pad 4: +12V -> Net-(D65-A)
- U10 pad 3: +12V -> Net-(D43-A)
- U13 pad 3: +12V -> Net-(D54-A)
- U15 pad 3: +12V -> Net-(D65-A)
- U3 pad 3: +12V -> Net-(D10-A)
- U37 pad 1: +3.3_digital -> unconnected-(U37-VCC-Pad1)
- U37 pad 10: GND -> unconnected-(U37-SEL-Pad10)
- U37 pad 15: /pcb_logica/Data -> unconnected-(U37-GND2-Pad15)
- U37 pad 16: /pcb_logica/Z -> unconnected-(U37-VISO-Pad16)
- U37 pad 2: /pcb_logica/encoder/A_MCU_5V -> unconnected-(U37-GND1-Pad2)
- U37 pad 3: /pcb_logica/encoder/B_MCU_5V -> unconnected-(U37-INA-Pad3)
- U37 pad 4: /pcb_logica/encoder/Z_MCU_5V -> unconnected-(U37-OUTB-Pad4)
- U37 pad 5: /pcb_logica/encoder/DATA_MCU_5V -> unconnected-(U37-OUTC-Pad5)
- U37 pad 6: GND -> unconnected-(U37-OUTD-Pad6)
- U37 pad 7: GND -> unconnected-(U37-NC-Pad7)
- U37 pad 8: GND -> unconnected-(U37-GND1-Pad8)
- U37 pad 9: GND -> unconnected-(U37-GND2-Pad9)
- U6 pad 3: +12V -> Net-(D21-A)
- U8 pad 3: +12V -> Net-(D32-A)

Commit message: Mejoras en el rut
Parts:
- removed the C141 at (51.2, 73.6)
- removed the C142 at (38.7, 69.2)
- removed the C144 at (49.5, 69.2)
- removed the C159 at (-44.9, 99.2)
- removed the C160 at (-24.6, 98.0)
- removed the C161 at (-41.4, 101.8)
- removed the C162 at (-41.2, 115.6)
- removed the C163 at (-45.5, 104.3)
- removed the C164 at (-34.3, 104.3)
- removed the C165 at (-36.4, 115.6)
- removed the C166 at (-45.9, 115.9)
- removed the C22 at (89.5, 99.9)
- removed the C23 at (87.3, 99.9)
- removed the C40 at (113.0, 97.6)
- removed the C41 at (114.3, 97.6)
- removed the C56 at (163.1, 95.6)
- removed the C57 at (164.3, 95.6)
- removed the C6 at (138.1, 101.2)
- removed the C7 at (135.9, 101.2)
- removed the C70 at (184.1, 99.5)
- removed the C71 at (182.9, 99.5)
- removed the C88 at (210.8, 94.2)
- removed the C89 at (212.1, 94.2)
- removed the D2 at (74.8, 95.0)
- removed the D3 at (71.4, 95.0)
- removed the D4 at (82.8, 99.1)
- removed the F1 at (-14.4, 59.3)
- removed J11: 347920040, Snapeda:CONN04_34792_MOL
- removed the J3 at (-131.9, 78.7)
- removed the J5 at (-130.5, 51.0)
- removed JP2: solotest, Jumper:SolderJumper-2_P1.3mm_Open_RoundedPad1.0x1.5mm
- removed the R1 at (74.8, 91.7)
- removed the R146 at (-110.9, 78.3)
- removed the R147 at (-116.9, 82.8)
- removed the R148 at (-116.9, 73.8)
- removed the R149 at (-110.9, 73.8)
- removed the R150 at (-116.9, 87.3)
- removed the R151 at (-116.9, 78.3)
- removed the R180 at (-33.6, 99.7)
- removed the R181 at (-44.8, 97.3)
- removed the R182 at (-42.4, 104.3)
- removed the R183 at (-37.4, 104.3)
- removed the R184 at (-38.7, 115.6)
- removed the R2 at (71.4, 91.7)
- removed R27, R42: 5k, Resistor_SMD:R_0402_1005Metric
- removed R28, R57: 2k, Resistor_SMD:R_0402_1005Metric
- removed the R3 at (80.9, 99.2)
- removed the R43 at (115.3, 97.6)
- removed the R56 at (162.0, 95.6)
- removed the R68 at (185.3, 99.4)
- removed the R69 at (181.8, 99.4)
- removed the R83 at (209.7, 94.3)
- removed the R84 at (213.2, 94.3)
- removed the U27 at (51.2, 77.0)
- removed the U31 at (-62.1, 97.4)
- removed the U32 at (-62.1, 109.1)
- added C152: 10uF, Capacitor_SMD:C_0805_2012Metric, F.Cu at (41.1, 61.0)
- added C153: 1uF, Capacitor_SMD:C_0805_2012Metric, F.Cu at (48.7, 71.0)
- added C155: 1uF, Capacitor_SMD:C_0805_2012Metric, F.Cu at (45.7, 71.0)
- added C172: 10nF, Capacitor_SMD:C_0603_1608Metric, F.Cu at (44.1, 165.2)
- added C173: 10uF, Capacitor_SMD:C_0805_2012Metric, F.Cu at (47.1, 165.4)
- added C174: 1`00nF, Capacitor_SMD:C_0402_1005Metric, F.Cu at (-187.4, 79.7)
- added C175: 100nF, Capacitor_SMD:C_0603_1608Metric, F.Cu at (-195.5, 60.4)
- added C176: 100nF, Capacitor_SMD:C_0603_1608Metric, F.Cu at (-191.5, 70.4)
- added C177: 10nF, Capacitor_SMD:C_0603_1608Metric, F.Cu at (-195.5, 62.9)
- added C178: 100nF, Capacitor_SMD:C_0603_1608Metric, F.Cu at (-195.5, 65.4)
- added C179: 100nF, Capacitor_SMD:C_0603_1608Metric, F.Cu at (-195.5, 67.9)
- added C180: 1nF, Capacitor_SMD:C_0402_1005Metric, F.Cu at (-187.4, 77.7)
- added C181: 4,7uF, Capacitor_SMD:C_0805_2012Metric, F.Cu at (-154.4, 46.6)
- added C182: 100nF, Capacitor_SMD:C_0603_1608Metric, F.Cu at (-195.5, 73.0)
- added C183: 100nF, Capacitor_SMD:C_0603_1608Metric, F.Cu at (-195.5, 70.4)
- added C184: 10nF, Capacitor_SMD:C_0603_1608Metric, F.Cu at (-195.5, 75.5)
- added C185: 10uF, Capacitor_SMD:C_0805_2012Metric, F.Cu at (-154.4, 49.6)
- added C186: 10nF, Capacitor_SMD:C_0603_1608Metric, F.Cu at (-191.5, 60.4)
- added C187: 10nF, Capacitor_SMD:C_0603_1608Metric, F.Cu at (-191.5, 62.9)
- added C188: 10nF, Capacitor_SMD:C_0603_1608Metric, F.Cu at (-191.5, 65.4)
- added C189: 10nF, Capacitor_SMD:C_0603_1608Metric, F.Cu at (-191.5, 67.9)
- added C81: 100pF, Capacitor_SMD:C_0402_1005Metric, F.Cu at (190.8, 95.1)
- added C99: 100pF, Capacitor_SMD:C_0402_1005Metric, F.Cu at (188.2, 95.1)
- added D7: APT2012EC, LED_SMD:LED_0805_2012Metric, F.Cu at (193.0, 92.3)
- added He1: GND_chasis, MountingHole:MountingHole_2.2mm_M2_DIN965_Pad, F.Cu at (59.0, 32.5)
- added J10: 348250125, Snapeda:CONN_SD-34825-001_12_MOL, F.Cu at (36.5, 74.8)
- added J2: 347928082, Snapeda:CONN08_34792_MOL, F.Cu at (55.8, 158.8)
- added J8: Conector sobre PCB, FSAE_footprints:My-UTS012E14S, F.Cu at (-194.0, 37.5)
- added J9: 348250125, Snapeda:CONN_SD-34825-001_12_MOL, F.Cu at (-189.9, 51.6)
- added JP1: Jumper SMD, Jumper:SolderJumper-2_P1.3mm_Open_RoundedPad1.0x1.5mm, F.Cu at (-152.8, 36.7)
- added L2: MLZ2012N6R8LT000, Inductor_SMD:L_0805_2012Metric, F.Cu at (18.7, 60.2)
- added L3: MLZ2012N6R8LT000, Inductor_SMD:L_0805_2012Metric, F.Cu at (42.4, 165.5)
- added L4: MLZ2012N6R8LT000, Inductor_SMD:L_0805_2012Metric, F.Cu at (-160.6, 66.6)
- added R16: 5k, Resistor_SMD:R_0603_1608Metric, F.Cu at (190.8, 92.6)
- added R186: 3k, Resistor_SMD:R_0603_1608Metric, F.Cu at (-187.5, 75.5)
- added R187: 10k, Resistor_SMD:R_0603_1608Metric, F.Cu at (-191.5, 73.0)
- added R188: 3k, Resistor_SMD:R_0603_1608Metric, F.Cu at (-187.5, 70.4)
- added R189: 1k, Resistor_SMD:R_0402_1005Metric, F.Cu at (-156.5, 36.0)
- added R190: 1k, Resistor_SMD:R_0402_1005Metric, F.Cu at (-156.5, 38.0)
- added R191: 120, Resistor_SMD:R_0603_1608Metric, F.Cu at (-191.5, 75.5)
- added R192: 10k, Resistor_SMD:R_0402_1005Metric, F.Cu at (-156.5, 39.9)
- added R193: 10k, Resistor_SMD:R_0402_1005Metric, F.Cu at (-156.5, 41.9)
- added R194: 100, Resistor_SMD:R_0402_1005Metric, F.Cu at (-156.5, 43.9)
- added R195: 120, Resistor_SMD:R_0603_1608Metric, F.Cu at (-187.5, 60.4)
- added R196: 120, Resistor_SMD:R_0603_1608Metric, F.Cu at (-187.5, 62.9)
- added R197: 120, Resistor_SMD:R_0603_1608Metric, F.Cu at (-187.5, 65.4)
- added R198: 120, Resistor_SMD:R_0603_1608Metric, F.Cu at (-187.5, 67.9)
- added R203: 0, Resistor_SMD:R_0603_1608Metric, F.Cu at (43.0, 46.5)
- added R204: 0, Resistor_SMD:R_0603_1608Metric, F.Cu at (70.3, 144.7)
- added RV1: 500, Potentiometer_THT:Potentiometer_Bourns_3296W_Vertical, F.Cu at (-162.6, 55.7)
- added TP23: TestPoint, TestPoint:TestPoint_Pad_D1.0mm, F.Cu at (-158.3, 60.7)
- added TP24: TestPoint, TestPoint:TestPoint_Pad_D1.0mm, F.Cu at (-158.3, 63.7)
- added U29: TLV76733QWDRBRQ1, Package_SON:VSON-8-1EP_3x3mm_P0.65mm_EP1.65x2.4mm, F.Cu at (46.4, 76.3)
- added U39: OPA333xxDCK, Package_TO_SOT_SMD:SOT-353_SC-70-5, F.Cu at (-153.0, 40.4)
- added U40: ISO7710FDWR, Snapeda:SOIC16_DW_TEX-L, F.Cu at (-179.3, 74.2)
- added U41: TPD4E05U06DQA, Package_SON:USON-10_2.5x1.0mm_P0.5mm, F.Cu at (-196.1, 79.0)
- added U43: TPD4E05U06DQA, Package_SON:USON-10_2.5x1.0mm_P0.5mm, F.Cu at (-190.3, 79.0)
- J6: value 347928082 -> 1053091205; footprint Snapeda:CONN08_34792_MOL -> Snapeda:CONN_SD-105309-100_05_MOL
- R106: renamed from R88; footprint Resistor_SMD:R_0402_1005Metric -> Resistor_SMD:R_0603_1608Metric
- R108: renamed from R90; footprint Resistor_SMD:R_0402_1005Metric -> Resistor_SMD:R_0603_1608Metric
- R109: renamed from R91; footprint Resistor_SMD:R_0402_1005Metric -> Resistor_SMD:R_0603_1608Metric
- R14: footprint Resistor_SMD:R_0402_1005Metric -> Resistor_SMD:R_0603_1608Metric
- R15: value 2k -> 5k; footprint Resistor_SMD:R_0402_1005Metric -> Resistor_SMD:R_0603_1608Metric
- R185: value 120 -> 3k
- U28: value TLV76733QWDRBRQ1 -> TPS7A2050PDBVR; footprint Package_SON:VSON-8-1EP_3x3mm_P0.65mm_EP1.65x2.4mm -> Snapeda:DBV0005A-IPC_A
- U35: footprint NuevoGui:D8_TEX-L -> Snapeda:D8_TEX-L
- U38: value TPD4E05U06DQA -> AMC1200BDWV; footprint Package_SON:USON-10_2.5x1.0mm_P0.5mm -> Package_SO:SOIC-8_7.5x5.85mm_P1.27mm
- U42: value ISO7710FDR -> TPD4E05U06DQA; footprint Snapeda:D0008B_HV -> Package_SON:USON-10_2.5x1.0mm_P0.5mm
- moved R185 150.0 mm to (-187.5, 73.0), turned to 0 degrees
- moved TP19 149.1 mm to (-161.4, 60.7)
- moved TP21 148.9 mm to (-161.4, 63.7)
- moved TP20 145.9 mm to (-155.3, 60.7)
- moved TP22 144.8 mm to (-155.3, 63.7)
- moved PS1 130.3 mm to (46.8, 157.6), turned to 180 degrees
- moved U35 125.1 mm to (-155.7, 55.7), turned to 0 degrees
- moved U36 121.4 mm to (-156.6, 74.0), turned to 0 degrees
- moved U38 115.8 mm to (-163.7, 48.8), turned to 0 degrees
- moved R180 108.5 mm to (26.1, 157.3), turned to 180 degrees
- moved U42 91.4 mm to (-193.2, 79.0)
- moved U37 58.2 mm to (-166.7, 74.3)
- moved R14 55.4 mm to (192.9, 95.6), turned to -90 degrees
- moved R15 52.4 mm to (188.3, 92.6)
- moved PS2 47.4 mm to (-182.0, 65.6)
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- renumbered C185 to C1, C2 to C10, C90 to C101, C91 to C102, C92 to C103, C93 to C104, C94 to C105, C95 to C106, C96 to C107, C97 to C108, C98 to C109, C3 to C11, C99 to C110, C100 to C111, C101 to C112, C102 to C113, C103 to C114, C104 to C115, C105 to C116, C106 to C117, C107 to C118, C108 to C119, C4 to C12, C109 to C120, C110 to C121, C111 to C122, C112 to C123, C113 to C124, C114 to C125, C115 to C126, C116 to C127, C117 to C128, C118 to C129, C5 to C13, C119 to C130, C120 to C131, C121 to C132, C122 to C133, C123 to C134, C124 to C135, C125 to C136, C126 to C137, C127 to C138, C128 to C139, C129 to C140, C130 to C141, C131 to C142, C132 to C143, C133 to C144, C134 to C145, C135 to C146, C136 to C147, C137 to C148, C138 to C149, C139 to C150, C140 to C151, C143 to C154, C145 to C156, C146 to C157, C147 to C158, C195 to C159, C8 to C16, C189 to C160, C188 to C161, C186 to C162, C190 to C163, C194 to C164, C193 to C165, C192 to C166, C191 to C167, C155 to C168, C156 to C169, C9 to C17, C157 to C170, C158 to C171, C10 to C18, C11 to C19, C180 to C190, C184 to C2, C12 to C20, C13 to C21, C14 to C22, C15 to C23, C16 to C24, C17 to C25, C181 to C26, C18 to C27, C19 to C28, C20 to C29, C1 to C3, C21 to C30, C24 to C33, C25 to C34, C26 to C35, C27 to C36, C28 to C37, C29 to C38, C30 to C39, C176 to C4, C31 to C40, C32 to C41, C33 to C42, C182 to C43, C34 to C44, C35 to C45, C36 to C46, C37 to C47, C38 to C48, C39 to C49, C177 to C5, C42 to C52, C43 to C53, C44 to C54, C45 to C55, C46 to C56, C47 to C57, C48 to C58, C49 to C59, C179 to C6, C50 to C60, C51 to C61, C52 to C62, C53 to C63, C54 to C64, C55 to C65, C58 to C68, C59 to C69, C174 to C7, C60 to C70, C61 to C71, C62 to C72, C63 to C73, C64 to C74, C65 to C75, C66 to C76, C67 to C77, C68 to C78, C69 to C79, C175 to C8, C72 to C82, C73 to C83, C74 to C84, C75 to C85, C76 to C86, C77 to C87, C78 to C88, C79 to C89, C178 to C9, C80 to C90, C81 to C91, C183 to C92, C82 to C93, C83 to C94, C84 to C95, C85 to C96, C86 to C97, C87 to C98, D6 to D10, D7 to D11, D8 to D12, D9 to D13, D10 to D14, D11 to D15, D12 to D16, D13 to D17, D14 to D18, D15 to D19, D88 to D2, D16 to D20, D17 to D21, D18 to D22, D19 to D23, D20 to D24, D21 to D25, D22 to D26, D23 to D27, D24 to D28, D25 to D29, D81 to D3, D26 to D30, D27 to D31, D28 to D32, D29 to D33, D30 to D34, D31 to D35, D32 to D36, D33 to D37, D34 to D38, D35 to D39, D80 to D4, D36 to D40, D37 to D41, D38 to D42, D39 to D43, D40 to D44, D41 to D45, D42 to D46, D43 to D47, D44 to D48, D45 to D49, D86 to D5, D46 to D50, D47 to D51, D48 to D52, D49 to D53, D50 to D54, D51 to D55, D52 to D56, D53 to D57, D54 to D58, D55 to D59, D56 to D60, D57 to D61, D58 to D62, D59 to D63, D60 to D64, D61 to D65, D62 to D66, D63 to D67, D64 to D68, D65 to D69, D66 to D70, D67 to D71, D68 to D72, D69 to D73, D70 to D74, D71 to D75, D72 to D76, D73 to D77, D74 to D78, D75 to D79, D76 to D80, D77 to D81, D78 to D82, D79 to D83, D82 to D86, D83 to D87, D87 to D88, D5 to D9, F2 to F1, J10 to J1, J7 to J3, J8 to J4, J9 to J5, J4 to J7, R190 to R1, R200 to R10, R82 to R100, R85 to R103, R86 to R104, R87 to R105, R89 to R107, R195 to R11, R92 to R110, R93 to R111, R94 to R112, R95 to R113, R96 to R114, R97 to R115, R98 to R116, R99 to R117, R100 to R118, R101 to R119, R196 to R12, R102 to R120, R103 to R121, R104 to R122, R105 to R123, R106 to R124, R107 to R125, R108 to R126, R109 to R127, R110 to R128, R111 to R129, R112 to R130, R113 to R131, R114 to R132, R115 to R133, R116 to R134, R117 to R135, R118 to R136, R119 to R137, R120 to R138, R121 to R139, R122 to R140, R123 to R141, R124 to R142, R125 to R143, R126 to R144, R127 to R145, R128 to R146, R129 to R147, R130 to R148, R131 to R149, R132 to R150, R133 to R151, R134 to R152, R135 to R153, R136 to R154, R137 to R155, R138 to R156, R139 to R157, R140 to R158, R141 to R159, R142 to R160, R143 to R161, R144 to R162, R145 to R163, R220 to R164, R221 to R165, R219 to R166, R222 to R167, R223 to R168, R224 to R169, R4 to R17, R198 to R170, R197 to R171, R211 to R172, R210 to R173, R213 to R174, R212 to R175, R201 to R176, R214 to R177, R174 to R178, R175 to R179, R5 to R18, R186 to R180, R176 to R181, R177 to R182, R178 to R183, R179 to R184, R6 to R19, R206 to R199, R187 to R2, R7 to R20, R207 to R200, R208 to R201, R209 to R202, R8 to R21, R9 to R22, R10 to R23, R11 to R24, R12 to R25, R13 to R26, R16 to R29, R188 to R3, R17 to R31, R18 to R32, R19 to R33, R20 to R34, R21 to R35, R22 to R36, R23 to R37, R24 to R38, R25 to R39, R189 to R4, R26 to R40, R29 to R43, R30 to R45, R31 to R46, R32 to R47, R33 to R48, R34 to R49, R199 to R5, R35 to R50, R36 to R51, R37 to R52, R38 to R53, R39 to R54, R40 to R55, R41 to R56, R203 to R6, R44 to R60, R45 to R61, R46 to R62, R47 to R63, R48 to R64, R49 to R65, R50 to R66, R51 to R67, R52 to R68, R53 to R69, R202 to R7, R54 to R70, R55 to R71, R58 to R75, R59 to R76, R60 to R77, R61 to R78, R62 to R79, R204 to R8, R63 to R80, R64 to R81, R65 to R82, R66 to R83, R67 to R84, R70 to R87, R71 to R89, R205 to R9, R72 to R90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
Connections:
- C11 pad 2: Net-(D10-A) (its old number) -> +12V
- C12 pad 1: Net-(D10-A) (its old number) -> +12V
- C154 pad 2: /pcb_logica/LogicSupply/5V_FB -> Net-(D80-K)
- C156 pad 1: /pcb_logica/LogicSupply/5V_FB -> Net-(D80-K)
- C28 pad 2: Net-(D21-A) (its old number) -> +12V
- C29 pad 1: Net-(D21-A) (its old number) -> +12V
- C44 pad 2: Net-(D32-A) (its old number) -> +12V
- C46 pad 1: Net-(D32-A) (its old number) -> +12V
- C6 pad 2: Net-(D80-A1) -> Net-(D4-A1)
- C60 pad 2: Net-(D43-A) (its old number) -> +12V
- C62 pad 1: Net-(D43-A) (its old number) -> +12V
- C77 pad 2: Net-(D54-A) (its old number) -> +12V
- C78 pad 1: Net-(D54-A) (its old number) -> +12V
- C93 pad 2: Net-(D65-A) (its old number) -> +12V
- C95 pad 1: Net-(D65-A) (its old number) -> +12V
- D14 pad 2: Net-(D10-A) (its old number) -> +12V
- D25 pad 2: Net-(D21-A) (its old number) -> +12V
- D36 pad 2: Net-(D32-A) (its old number) -> +12V
- D4 pad 1: Net-(D80-A1) -> Net-(D4-A1)
- D47 pad 2: Net-(D43-A) (its old number) -> +12V
- D58 pad 2: Net-(D54-A) (its old number) -> +12V
- D69 pad 2: Net-(D65-A) (its old number) -> +12V
- D80 pad 1: /pcb_logica/LogicSupply/5V_FB -> Net-(D80-K)
- D81 pad 1: /pcb_logica/LogicSupply/5V_FB -> Net-(D80-K)
- D86 pad 1: Net-(D82-A1) -> /pcb_logica/comunicacionCAN/CAN_H_1
- D86 pad 2: Net-(D82-A2) -> /pcb_logica/comunicacionCAN/CAN_L_1
- D87 pad 1: Net-(D83-A1) -> /pcb_logica/comunicacionCAN/CAN_H_2
- D87 pad 2: Net-(D83-A2) -> /pcb_logica/comunicacionCAN/CAN_L_2
- J6 pad 1: +5V_analog -> /pcb_logica/comunicacionCAN/CAN_L_2
- J6 pad 2: +5V_analog -> /pcb_logica/comunicacionCAN/CAN_H_2
- J6 pad 3: /pcb_logica/apps/opamp_1 -> GND_Can
- J6 pad 4: /pcb_logica/apps/opamp_2 -> /pcb_logica/comunicacionCAN/CAN_L_1
- J6 pad 5: Net-(D80-A1) -> /pcb_logica/comunicacionCAN/CAN_H_1
- PS1 pad 1: +12V -> Net-(PS1-+VIN)
- PS1 pad 2: unconnected-(PS1--VIN-Pad2) -> GND
- PS1 pad 7: Net-(PS1-+VOUT) -> +5V_Can
- PS2 pad 1: unconnected-(PS2-+VIN-Pad1) -> Net-(PS2-+VIN)
- PS2 pad 2: unconnected-(PS2--VIN-Pad2) -> GND_EXT
- PS2 pad 5: unconnected-(PS2--VOUT-Pad5) -> GND_EXT_ISO
- PS2 pad 6: unconnected-(PS2-0V-Pad6) -> GND_EXT_ISO
- PS2 pad 7: unconnected-(PS2-+VOUT-Pad7) -> +5V_EXT_ISO
- R10 pad 1: Net-(D80-A1) -> Net-(D4-A1)
- R15 pad 1: /pcb_logica/GD_FLT -> /pcb_logica/Reset_Pote
- R163 pad 1: /pcb_logica/LogicSupply/5V_FB -> Net-(D80-K)
- R178 pad 1: Net-(D82-A1) -> /pcb_logica/comunicacionCAN/CAN_H_1
- R178 pad 2: Net-(D82-A2) -> /pcb_logica/comunicacionCAN/CAN_L_1
- R179 pad 1: Net-(D83-A1) -> /pcb_logica/comunicacionCAN/CAN_H_2
- R179 pad 2: Net-(D83-A2) -> /pcb_logica/comunicacionCAN/CAN_L_2
- R185 pad 1: /pcb_logica/encoder/A+ -> Net-(U38-VINN)
- R185 pad 2: Net-(C166-Pad2) -> +5V_EXT_ISO
- R20 pad 1: Net-(D10-A) (its old number) -> +12V
- R34 pad 1: Net-(D21-A) (its old number) -> +12V
- R45 pad 1: Net-(D32-A) (its old number) -> +12V
- R60 pad 1: Net-(D43-A) (its old number) -> +12V
- R78 pad 1: Net-(D54-A) (its old number) -> +12V
- R89 pad 1: Net-(D65-A) (its old number) -> +12V
- T1 pad 4: Net-(D10-A) (its old number) -> +12V
- T2 pad 4: Net-(D21-A) (its old number) -> +12V
- T3 pad 4: Net-(D32-A) (its old number) -> +12V
- T4 pad 4: Net-(D43-A) (its old number) -> +12V
- T5 pad 4: Net-(D54-A) (its old number) -> +12V
- T6 pad 4: Net-(D65-A) (its old number) -> +12V
- TP19 pad 1: /pcb_logica/A -> /pcb_logica/encoder/A_PCB_EXT
- TP20 pad 1: /pcb_logica/B -> /pcb_logica/encoder/CLK_ENC_EXT
- TP21 pad 1: /pcb_logica/Z -> /pcb_logica/encoder/B_PCB_EXT
- TP22 pad 1: /pcb_logica/Data -> /pcb_logica/encoder/TEMP_EXT
- U11 pad 3: Net-(D43-A) (its old number) -> +12V
- U14 pad 3: Net-(D54-A) (its old number) -> +12V
- U16 pad 3: Net-(D65-A) (its old number) -> +12V
- U28 pad 1: +3.3_digital -> /pcb_logica/LogicSupply/5V_FB
- U28 pad 2: unconnected-(U28-NC-Pad2) -> GND
- U28 pad 3: +3.3_digital -> /pcb_logica/LogicSupply/5V_FB
- U28 pad 4: GND -> unconnected-(U28-N/C-Pad4)
- U28 pad 5: /pcb_logica/LogicSupply/5V_FB -> +5V_digital
- U33 pad 12: Net-(D82-A2) -> /pcb_logica/comunicacionCAN/CAN_L_1
- U33 pad 13: Net-(D82-A1) -> /pcb_logica/comunicacionCAN/CAN_H_1
- U34 pad 12: Net-(D83-A2) -> /pcb_logica/comunicacionCAN/CAN_L_2
- U34 pad 13: Net-(D83-A1) -> /pcb_logica/comunicacionCAN/CAN_H_2
- U35 pad 4: /pcb_logica/Clk -> /pcb_logica/encoder/Clk_ISO
- U35 pad 5: GND -> GND_EXT_ISO
- U35 pad 8: +5V_digital -> +5V_EXT_ISO
- U36 pad 11: /pcb_logica/encoder/Z_MCU_5V -> /pcb_logica/encoder/Z_ISO
- U36 pad 12: GND -> GND_EXT_ISO
- U36 pad 13: /pcb_logica/encoder/DATA_MCU_5V -> /pcb_logica/encoder/DATA_ISO
- U36 pad 16: +5V_digital -> +5V_EXT_ISO
- U36 pad 3: /pcb_logica/encoder/A_MCU_5V -> /pcb_logica/encoder/A_ISO
- U36 pad 4: +5V_digital -> +5V_EXT_ISO
- U36 pad 5: /pcb_logica/encoder/B_MCU_5V -> /pcb_logica/encoder/B_ISO
- U36 pad 8: GND -> GND_EXT_ISO
- U37 pad 1: unconnected-(U37-VCC-Pad1) -> +3.3_EXT
- U37 pad 10: unconnected-(U37-SEL-Pad10) -> GND_EXT_ISO
- U37 pad 11: unconnected-(U37-IND-Pad11) -> /pcb_logica/encoder/B_ISO
- U37 pad 12: unconnected-(U37-INC-Pad12) -> /pcb_logica/encoder/A_ISO
- U37 pad 13: unconnected-(U37-INB-Pad13) -> /pcb_logica/encoder/DATA_ISO
- U37 pad 14: unconnected-(U37-OUTA-Pad14) -> /pcb_logica/encoder/Clk_ISO
- U37 pad 15: unconnected-(U37-GND2-Pad15) -> GND_EXT_ISO
- U37 pad 16: unconnected-(U37-VISO-Pad16) -> Net-(JP1-A)
- U37 pad 2: unconnected-(U37-GND1-Pad2) -> GND_EXT
- U37 pad 3: unconnected-(U37-INA-Pad3) -> /pcb_logica/encoder/CLK_ENC_EXT
- U37 pad 4: unconnected-(U37-OUTB-Pad4) -> /pcb_logica/encoder/DATA_PCB_EXT
- U37 pad 5: unconnected-(U37-OUTC-Pad5) -> /pcb_logica/encoder/A_PCB_EXT
- U37 pad 6: unconnected-(U37-OUTD-Pad6) -> /pcb_logica/encoder/B_PCB_EXT
- U37 pad 8: unconnected-(U37-GND1-Pad8) -> GND_EXT
- U37 pad 9: unconnected-(U37-GND2-Pad9) -> GND_EXT_ISO
- U38 pad 1: /pcb_logica/encoder/Data- -> +5V_EXT_ISO
- U38 pad 2: /pcb_logica/encoder/Data+ -> /pcb_logica/encoder/Temp+
- U38 pad 3: GND -> Net-(U38-VINN)
- U38 pad 4: /pcb_logica/encoder/Z+ -> GND_EXT_ISO
- U38 pad 5: /pcb_logica/encoder/Z- -> GND_EXT
- U38 pad 6: unconnected-(U38-NC-Pad6) -> Net-(U38-VOUTN)
- U38 pad 7: unconnected-(U38-NC-Pad7) -> Net-(U38-VOUTP)
- U38 pad 8: GND -> +3.3_EXT
- U4 pad 3: Net-(D10-A) (its old number) -> +12V
- U42 pad 1: unconnected-(U42-VCC1-Pad1) -> /pcb_logica/encoder/B-
- U42 pad 2: unconnected-(U42-IN-Pad2) -> /pcb_logica/encoder/B+
- U42 pad 3: unconnected-(U42-VCC1-Pad3) -> GND_EXT_ISO
- U42 pad 4: unconnected-(U42-GND1-Pad4) -> /pcb_logica/encoder/Temp+
- U42 pad 5: unconnected-(U42-GND2-Pad5) -> GND_EXT_ISO
- U42 pad 8: unconnected-(U42-VCC2-Pad8) -> GND_EXT_ISO
- U44 pad 4: /pcb_logica/Reset_Pote -> Net-(U44-OUT)
- U7 pad 3: Net-(D21-A) (its old number) -> +12V
- U9 pad 3: Net-(D32-A) (its old number) -> +12V
Routing:
- net +3.3V_analog: track 651.2 -> 60.8 mm, vias 18 -> 1
- net GND: track 553.7 -> 105.8 mm, vias 129 -> 20
- net +12V: track 646.7 -> 236.8 mm, vias 9 -> 12
- net /pcb_logica/LogicSupply/5V_FB: track 184.6 -> 7.88 mm, vias 6 -> 0
- net /pcb_logica/Temp_B: track 133.1 -> 1.09 mm, vias 3 -> 0
- net /pcb_logica/Reset_Pote: track 269.5 -> 163.2 mm, vias 13 -> 3
- net Net-(U18D-FLT1): track 105.2 -> 0.00 mm, vias 3 -> 0
- net /pcb_logica/Current_B: track 105.2 -> 1.11 mm, vias 2 -> 0
- net +3.3_digital: track 146.4 -> 50.5 mm, vias 19 -> 0
- net /pcb_logica/Temp_C: track 90.5 -> 0.00 mm, vias 2 -> 0
- net /pcb_logica/TMS: track 94.6 -> 12.0 mm, vias 1 -> 0
- net /pcb_logica/TCK: track 89.5 -> 14.2 mm, vias 1 -> 0
- net /pcb_logica/GD_FLT: track 217.2 -> 150.0 mm, vias 8 -> 3
- net /pcb_logica/GD_RDY: track 215.6 -> 148.5 mm, vias 8 -> 3
- net /pcb_logica/TDO: track 84.1 -> 17.5 mm, vias 1 -> 0
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- added copper zone on F.Cu, net +12V
- added copper zone on In4.Cu, net +12V
- added copper zone on F.Cu, net +12V_In
- added copper zone on In4.Cu, net +5V_Can
- added copper zone on B.Cu, net GND_Can
- added copper zone on In1.Cu, net GND_Can
- added copper zone on In3.Cu, net GND_Can
- added copper zone on F.Cu, net Net-(D1-A1)
- removed copper zone on B.Cu, net (none)
- removed copper zone on In1.Cu, net (none)
- removed copper zone on In3.Cu, net (none)
- removed copper zone on In4.Cu, net (none)
- removed copper zone on B.Cu, net +5V_digital
- removed copper zone on In4.Cu, net +5V_digital
- removed copper zone on B.Cu, net GND_Can_1
- removed copper zone on In1.Cu, net GND_Can_1
- removed copper zone on In3.Cu, net GND_Can_1
Other:
- board size 220 x 140 mm -> 220 x 145 mm
