File: PCB/InverterV2.0/Primero_esquematico/g_driver.kicad_sch (KiCad schematic)
At the start: 13 parts, among them U1 FS950R08A6P2BBPSA1

Commit message: Hice un par de cambios de pistas y dos boludeces mas
Changed lines of the file:
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@@
 		)
 	)
-	(hierarchical_label "C3_In_pos"
+	(hierarchical_label "C2_In_pos"
 		(shape input)
 		(at 25.4 95.25 180)

Commit message: Mejoras en el rut
Parts:
- removed D2, D3, D4: APT2012EC, LED_SMD:LED_0805_2012Metric, symbol Device:LED
- removed R1, R2, R3: 2k2, Resistor_SMD:R_0603_1608Metric, symbol Device:R
- added C81, C99: 100pF, Capacitor_SMD:C_0402_1005Metric, symbol Device:C
- added D7: APT2012EC, LED_SMD:LED_0805_2012Metric, symbol Device:LED
- added R14, R15, R16: 5k, Resistor_SMD:R_0603_1608Metric, symbol Device:R
- renumbered U1 to U2
Connections:
- net +3.3_digital: now also R14.2, R15.2, R16.2
- net GND: now also C81.1, C99.1, D7.1 (K)
- net RDY: now also D7.2 (A), R14.1
- net Reset/EN: now also C99.2, R15.1
- net ~FLT: now also C81.2, R16.1
