File: PCB/InverterV2.0/Primero_esquematico/g_driver.kicad_sch (KiCad schematic)
At the start: 13 parts, among them U2 FS950R08A6P2BBPSA1

Commit message: Correcciones de DRC del inverter: vias, serigrafia y reglas de diseno
Vias:
- 13 vias fuera de norma (0,30/0,15 y 0,45/0,30, anillo de 0,075 mm)
  llevadas a 0,45/0,25 (anillo 0,10 mm).
- Eliminados los dos presets de via invalidos que contradecian las
  propias reglas minimas de la placa. Agregado 0,8/0,3 que usan las
  netclasses de potencia.
- Minimos ajustados a capacidad de fabricacion estandar:
  diametro 0,45 / taladro 0,25 / anillo 0,10.

Serigrafia:
- 76 textos normalizados: espesor >= 0,15 mm y altura >= 0,8 mm.
- Espesor por defecto corregido de 0,1 a 0,15 mm (estaba por debajo
  del minimo exigido por la propia placa).
- Activado subtractmaskfromsilk para que los gerbers recorten la
  serigrafia sobre las aperturas de mascara.

Reglas:
- min_resolved_spokes de 2 a 1 (alivios termicos).
- Nuevo Primero_esquematico.kicad_dru: reglas de clearance para pads
  de encapsulados de paso 0,65 mm (U31, U5, U8, U15), donde la
  separacion la fija el fabricante del componente.

Ademas: ruteo, areas de reglas y g_driver actualizados.
Estado al momento del commit: 6 infracciones y 14 elementos sin conectar.

Co-Authored-By: Claude Opus 5 <noreply@anthropic.com>
Connections:
- removed net VCC_DC: U2.C1, U2.C3, U2.C5
- new net VCC_DC_1: U2.C1
- new net VCC_DC_2: U2.C3
- new net VCC_DC_3: U2.C5
Changed lines of the file:
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@@
 		)
 	)
-	(label "VCC_DC"
+	(label "VCC_DC_2"
 		(at 87.63 92.71 180)
 		(effects
@@
 		)
 	)
-	(label "VCC_DC"
-		(at 222.25 130.81 0)
-		(effects
-			(font
-				(size 1.27 1.27)
-			)
-			(justify left bottom)
-		)
-	)
 	(label "MP_3"
 		(at 127 139.7 0)
@@
 		)
 	)
-	(label "VCC_DC"
+	(label "VCC_DC_3"
 		(at 88.9 139.7 180)
 		(effects
@@
 	(label "ISO_GND_HS_1"
 		(at 76.2 55.88 0)
+		(effects
+			(font
+				(size 1.27 1.27)
+			)
+			(justify left bottom)
+		)
+	)
+	(label "VCC_DC_1"
+		(at 222.25 130.81 0)
 		(effects
 			(font
@@
 		)
 	)
-	(label "VCC_DC"
+	(label "VCC_DC_1"
 		(at 88.9 45.72 180)
 		(effects
