File: PCB/InverterV2.0/Primero_esquematico/pcb_logica.kicad_sch (KiCad schematic)
At the start: 0 parts

Commit message: aislacion encoder
Other:
- sheet F280049C ports: added C4_Temp_Motor; removed C4_Temp_PCB
Changed lines of the file:
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@@
-	(wire
-		(pts
-			(xy 39.37 96.52) (xy 40.64 96.52)
-		)
-		(stroke
-			(width 0)
-			(type default)
-		)
-	)
 	(wire
 		(pts
@@
 		(pts
 			(xy 218.44 130.81) (xy 232.41 130.81)
+		)
+		(stroke
+			(width 0)
+			(type default)
+		)
+	)
+	(wire
+		(pts
+			(xy 17.78 96.52) (xy 40.64 96.52)
 		)
 		(stroke
@@
 		)
 	)
+	(label "Temp_Motor"
+		(at 17.78 96.52 0)
+		(effects
+			(font
+				(size 1.27 1.27)
+				(thickness 0.254)
+				(bold yes)
+			)
+			(justify left bottom)
+		)
+	)
 	(label "Clk"
 		(at 149.86 105.41 0)
@@
 		(shape bidirectional)
 		(at 36.83 124.46 180)
-		(effects
-			(font
-				(size 1.27 1.27)
-			)
-			(justify right)
-		)
-	)
-	(hierarchical_label "Temp_PCB"
-		(shape bidirectional)
-		(at 39.37 96.52 180)
 		(effects
 			(font
@@
 			)
 		)
-		(pin "C4_Temp_PCB" bidirectional
-			(at 40.64 96.52 180)
-			(effects
-				(font
-					(size 1.27 1.27)
-				)
-				(justify left)
-			)
-		)
 		(pin "GP_0_PWM_MP_H_A" bidirectional
 			(at 119.38 63.5 0)
@@
 			(effects
 				(font
+					(size 1.27 1.27)
+				)
+				(justify left)
+			)
+		)
+		(pin "C4_Temp_Motor" bidirectional
+			(at 40.64 96.52 180)
+			(effects
+				(font

Commit message: Mejoras en el rut
Other:
- sheet encoder ports: added A_PCB_MCU, B_PCB_MCU, CLK_PCB_MCU, DATA_PCB_MCU, TEMP_MCU, Z_PCB_MCU; removed A_MCU, B_MCU, Clock_MCU, Data_MCU, Z_MCU
Changed lines of the file:
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@@
+	(wire
+		(pts
+			(xy 149.86 110.49) (xy 163.83 110.49)
+		)
+		(stroke
+			(width 0)
+			(type default)
+		)
+	)
 	(wire
 		(pts
@@
 	(label "CAN_TX_A"
 		(at 218.44 130.81 0)
+		(effects
+			(font
+				(size 1.27 1.27)
+				(thickness 0.254)
+				(bold yes)
+			)
+			(justify left bottom)
+		)
+	)
+	(label "Temp_Motor"
+		(at 149.86 110.49 0)
 		(effects
 			(font
@@
 			)
 		)
-		(pin "A_MCU" bidirectional
+		(pin "A_PCB_MCU" bidirectional
 			(at 163.83 88.9 180)
 			(effects
@@
 			)
 		)
-		(pin "B_MCU" bidirectional
+		(pin "B_PCB_MCU" bidirectional
 			(at 163.83 92.71 180)
 			(effects
@@
 			)
 		)
-		(pin "Clock_MCU" bidirectional
+		(pin "CLK_PCB_MCU" bidirectional
 			(at 163.83 105.41 180)
 			(effects
@@
 			)
 		)
-		(pin "Data_MCU" bidirectional
+		(pin "DATA_PCB_MCU" bidirectional
 			(at 163.83 102.87 180)
 			(effects
@@
 			)
 		)
-		(pin "Z_MCU" bidirectional
+		(pin "TEMP_MCU" bidirectional
+			(at 163.83 110.49 180)
+			(effects
+				(font
+					(size 1.27 1.27)
+				)
+				(justify left)
+			)
+		)
+		(pin "Z_PCB_MCU" bidirectional
 			(at 163.83 96.52 180)
 			(effects
