File: PCB/InverterV2.0/Primero_esquematico/F280049C.kicad_sch (KiCad schematic)
At the start: 39 parts, among them SW1 IT-1187-160GM-G, U17 F280049CPZS, U18 TPS3823-33DBVR, Y1 ABM8GAIG-20.000MHZ-8-7Z-T3

Commit message: aislacion encoder
Connections:
- net C4_Temp_PCB renamed C4_Temp_Motor
Changed lines of the file:
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@@
 		)
 	)
-	(hierarchical_label "C4_Temp_PCB"
+	(hierarchical_label "C4_Temp_Motor"
 		(shape bidirectional)
 		(at 30.48 81.28 180)

Commit message: Mejoras en el rut
Parts:
- R106: renamed from R88; footprint Resistor_SMD:R_0402_1005Metric -> Resistor_SMD:R_0603_1608Metric
- R108: renamed from R90; footprint Resistor_SMD:R_0402_1005Metric -> Resistor_SMD:R_0603_1608Metric
- R109: renamed from R91; footprint Resistor_SMD:R_0402_1005Metric -> Resistor_SMD:R_0603_1608Metric
- renumbered C98 to C109, C99 to C110, C100 to C111, C101 to C112, C102 to C113, C103 to C114, C104 to C115, C105 to C116, C106 to C117, C107 to C118, C108 to C119, C109 to C120, C110 to C121, C111 to C122, C112 to C123, C113 to C124, C114 to C125, C115 to C126, C116 to C127, C117 to C128, C118 to C129, C119 to C130, C120 to C131, D71 to D75, D72 to D76, D73 to D77, R85 to R103, R86 to R104, R87 to R105, R89 to R107, U17 to U18, U18 to U19
