File: PCB/InverterV2.0/Primero_esquematico/GD_HS.kicad_sch (KiCad schematic)
At the start: 46 parts, among them T3 750317595, U8 LM25180QNGURQ1, U9 UCC21750QDWRQ1

Commit message: aislacion encoder
Parts:
- added R146: 0, Resistor_SMD:R_0603_1608Metric, symbol Device:R
Connections:
- net +12V: now also R146.1; no longer C34.2, C36.1, D32.2 (A), R30.1, T3.4, U8.3 (VIN)
- new net: C34.2, C36.1, D32.2 (A), R146.2, R30.1, T3.4, U8.3 (VIN)
Changed lines of the file:
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@@
 	(wire
 		(pts
+			(xy 44.45 59.69) (xy 49.53 59.69)
+		)
+		(stroke
+			(width 0)
+			(type default)
+		)
+	)
+	(wire
+		(pts
 			(xy 87.63 144.78) (xy 87.63 147.32)
 		)
@@
 	(wire
 		(pts
-			(xy 36.83 59.69) (xy 49.53 59.69)
+			(xy 33.02 59.69) (xy 36.83 59.69)
 		)
 		(stroke
@@
 	(wire
 		(pts
-			(xy 36.83 58.42) (xy 36.83 59.69)
+			(xy 33.02 53.34) (xy 33.02 59.69)
 		)
 		(stroke
@@
 	)
 	(symbol
+		(lib_id "Device:R")
+		(at 40.64 59.69 90)
+		(unit 1)
+		(body_style 1)
+		(exclude_from_sim no)
+		(in_bom yes)
+		(on_board yes)
+		(in_pos_files yes)
+		(dnp no)
+		(fields_autoplaced yes)
+		(property "Reference" "R146"
+			(at 40.64 53.34 90)
+			(show_name no)
+			(do_not_autoplace no)
+			(effects
+				(font
+					(size 1.27 1.27)
+				)
+			)
+		)
+		(property "Value" "0"
+			(at 40.64 55.88 90)
+			(show_name no)
+			(do_not_autoplace no)
+			(effects
+				(font
+					(size 1.27 1.27)
+				)
+			)
+		)
+		(property "Footprint" "Resistor_SMD:R_0603_1608Metric"
+			(at 40.64 61.468 90)
+			(hide yes)
+			(show_name no)
+			(do_not_autoplace no)
+			(effects
+				(font
+					(size 1.27 1.27)
+				)
+			)
+		)
+		(property "Datasheet" ""
+			(at 40.64 59.69 0)
+			(hide yes)
+			(show_name no)
+			(do_not_autoplace no)
+			(effects
+				(font
+					(size 1.27 1.27)
+				)
+			)
+		)
+		(property "Description" "Resistor"
+			(at 40.64 59.69 0)
+			(hide yes)
+			(show_name no)
+			(do_not_autoplace no)
+			(effects
+				(font
+					(size 1.27 1.27)
+				)
+			)
+		)
+		(property "Compra" ""
+			(at 40.64 59.69 0)
+			(hide yes)
+			(show_name no)
+			(do_not_autoplace no)
+			(effects
+				(font
+					(size 1.27 1.27)
+				)
+			)
+		)
+		(property "Description_1" ""
+			(at 40.64 59.69 0)
+			(hide yes)
+			(show_name no)
+			(do_not_autoplace no)
+			(effects
+				(font
+					(size 1.27 1.27)
+				)
+			)
+		)
+		(property "Purchase-URL" ""
+			(at 40.64 59.69 0)
+			(hide yes)
+			(show_name no)
+			(do_not_autoplace no)
+			(effects
+				(font
+					(size 1.27 1.27)
+				)
+			)
+		)
+		(pin "1"
+		)
+		(pin "2"
+		)
+		(instances
+			(project "Primero_esquematico"
+				(path "/d930f486-f6ac-489c-907e-47f2cb34cf04/d101e913-ebd1-4e08-b728-82218f47123b/f5297dcd-d9e2-4174-98d4-ada2947e9df5/3742c66c-85ff-4287-9a19-7809bdcfdde9"
+					(reference "R148")
+					(unit 1)
+				)
+				(path "/d930f486-f6ac-489c-907e-47f2cb34cf04/d101e913-ebd1-4e08-b728-82218f47123b/f5297dcd-d9e2-4174-98d4-ada2947e9df5/a6c67f59-8868-40d8-9141-527ce9b5d508"
+					(reference "R146")
+					(unit 1)
+				)
+				(path "/d930f486-f6ac-489c-907e-47f2cb34cf04/d101e913-ebd1-4e08-b728-82218f47123b/f5297dcd-d9e2-4174-98d4-ada2947e9df5/d86b56e9-6f01-47d4-af65-f49184945e26"
+					(reference "R147")
+					(unit 1)
+				)
+			)
+		)
+	)
+	(symbol
 		(lib_id "Device:C")
 		(at 252.73 44.45 0)
@@
 	(symbol
 		(lib_id "power:+12V")
-		(at 36.83 58.42 0)
+		(at 33.02 53.34 0)
 		(unit 1)
 		(body_style 1)
@@
 		(fields_autoplaced yes)
 		(property "Reference" "#PWR042"
-			(at 36.83 62.23 0)
+			(at 33.02 57.15 0)
 			(hide yes)
 			(show_name no)
@@
 		)
 		(property "Value" "+12V"
-			(at 36.83 53.34 0)
+			(at 33.02 48.26 0)
 			(show_name no)
 			(do_not_autoplace no)
@@
 		)
 		(property "Footprint" ""
-			(at 36.83 58.42 0)
+			(at 33.02 53.34 0)
 			(hide yes)
 			(show_name no)
@@
 		)
 		(property "Datasheet" ""
-			(at 36.83 58.42 0)
+			(at 33.02 53.34 0)
 			(hide yes)
 			(show_name no)
@@
 		)
 		(property "Description" "Power symbol creates a global label with name \"+12V\""
-			(at 36.83 58.42 0)
+			(at 33.02 53.34 0)
 			(hide yes)
 			(show_name no)

Commit message: Mejoras en el rut
Parts:
- removed C40, C41: 100pF, Capacitor_SMD:C_0402_1005Metric, symbol Device:C
- removed R146: 0, Resistor_SMD:R_0603_1608Metric, symbol Device:R
- removed R42: 5k, Resistor_SMD:R_0402_1005Metric, symbol Device:R
- removed R43: 2k, Resistor_SMD:R_0402_1005Metric, symbol Device:R
- renumbered C34 to C44, C35 to C45, C36 to C46, C37 to C47, C38 to C48, C39 to C49, C42 to C52, C43 to C53, C44 to C54, C45 to C55, C46 to C56, C47 to C57, C48 to C58, C49 to C59, D27 to D31, D28 to D32, D29 to D33, D30 to D34, D31 to D35, D32 to D36, D33 to D37, D34 to D38, D35 to D39, D36 to D40, D37 to D41, R30 to R45, R31 to R46, R32 to R47, R33 to R48, R34 to R49, R35 to R50, R36 to R51, R37 to R52, R38 to R53, R39 to R54, R40 to R55, R41 to R56, U9 to U10, U8 to U9
Connections:
- net +12V: now also C44.2, C46.1, D36.2 (A), R45.1, T3.4, U9.3 (VIN)
Other:
- moved on the sheet: C45, C47, C49, C54, D31, D32, D33, D34, D35, R47, R49, R50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

Commit message: Todo Listo para mandar
Parts:
- added C198, C199: 100pF, Capacitor_SMD:C_0603_1608Metric, symbol Device:C_Small
- added TP25: TestPoint, TestPoint:TestPoint_Pad_D1.0mm, symbol Connector:TestPoint
Connections:
- net +IN: now also C198.1
- net -IN: now also C199.1
- net GND: now also C198.2, C199.2
- net ISO_GND: now also TP25.1
Other:
- moved on the sheet: C54

Commit message: Solo falta mandar a hacer
Parts:
- D31, D32: footprint Diode_SMD:D_SOD-323F -> Diode_SMD:D_SMA
