File: PCB/InverterV2.0/Primero_esquematico/GD_LS.kicad_sch (KiCad schematic)
At the start: 47 parts, among them T1 750317595, U2 UCC21750QDWRQ1, U3 LM25180QNGURQ1, U4 LP2951-5.0_VSSOP

Commit message: aislacion encoder
Parts:
- added R149: 0, Resistor_SMD:R_0603_1608Metric, symbol Device:R
Connections:
- net +12V: now also R149.1; no longer C3.2, C4.1, D10.2 (A), R7.1, T1.4, U3.3 (VIN)
- new net: C3.2, C4.1, D10.2 (A), R149.2, R7.1, T1.4, U3.3 (VIN)
Changed lines of the file:
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@@
+	(wire
+		(pts
+			(xy 46.99 59.69) (xy 49.53 59.69)
+		)
+		(stroke
+			(width 0)
+			(type default)
+		)
+	)
 	(wire
 		(pts
@@
 	(wire
 		(pts
-			(xy 36.83 59.69) (xy 49.53 59.69)
+			(xy 36.83 59.69) (xy 39.37 59.69)
 		)
 		(stroke
@@
 					(unit 1)
 				)
+			)
+		)
+	)
+	(symbol
+		(lib_id "Device:R")
+		(at 43.18 59.69 90)
+		(unit 1)
+		(body_style 1)
+		(exclude_from_sim no)
+		(in_bom yes)
+		(on_board yes)
+		(in_pos_files yes)
+		(dnp no)
+		(fields_autoplaced yes)
+		(property "Reference" "R149"
+			(at 43.18 53.34 90)
+			(show_name no)
+			(do_not_autoplace no)
+			(effects
+				(font
+					(size 1.27 1.27)
+				)
+			)
+		)
+		(property "Value" "0"
+			(at 43.18 55.88 90)
+			(show_name no)
+			(do_not_autoplace no)
+			(effects
+				(font
+					(size 1.27 1.27)
+				)
+			)
+		)
+		(property "Footprint" "Resistor_SMD:R_0603_1608Metric"
+			(at 43.18 61.468 90)
+			(hide yes)
+			(show_name no)
+			(do_not_autoplace no)
+			(effects
+				(font
+					(size 1.27 1.27)
+				)
+			)
+		)
+		(property "Datasheet" ""
+			(at 43.18 59.69 0)
+			(hide yes)
+			(show_name no)
+			(do_not_autoplace no)
+			(effects
+				(font
+					(size 1.27 1.27)
+				)
+			)
+		)
+		(property "Description" "Resistor"
+			(at 43.18 59.69 0)
+			(hide yes)
+			(show_name no)
+			(do_not_autoplace no)
+			(effects
+				(font
+					(size 1.27 1.27)
+				)
+			)
+		)
+		(property "Compra" ""
+			(at 43.18 59.69 0)
+			(hide yes)
+			(show_name no)
+			(do_not_autoplace no)
+			(effects
+				(font
+					(size 1.27 1.27)
+				)
+			)
+		)
+		(property "Description_1" ""
+			(at 43.18 59.69 0)
+			(hide yes)
+			(show_name no)
+			(do_not_autoplace no)
+			(effects
+				(font
+					(size 1.27 1.27)
+				)
+			)
+		)
+		(property "Purchase-URL" ""
+			(at 43.18 59.69 0)
+			(hide yes)
+			(show_name no)
+			(do_not_autoplace no)
+			(effects
+				(font
+					(size 1.27 1.27)
+				)
+			)
+		)
+		(pin "1"
+		)
+		(pin "2"
+		)
+		(instances
+			(project "Primero_esquematico"
+				(path "/d930f486-f6ac-489c-907e-47f2cb34cf04/d101e913-ebd1-4e08-b728-82218f47123b/f5297dcd-d9e2-4174-98d4-ada2947e9df5/5cdf39cf-afbe-4cc8-b2fc-5cff4a76438c"
+					(reference "R149")
+					(unit 1)
+				)
+				(path "/d930f486-f6ac-489c-907e-47f2cb34cf04/d101e913-ebd1-4e08-b728-82218f47123b/f5297dcd-d9e2-4174-98d4-ada2947e9df5/78ffa60a-7e25-44e8-bbd6-bfc8ed5e55d3"
+					(reference "R151")
+					(unit 1)
+				)
+				(path "/d930f486-f6ac-489c-907e-47f2cb34cf04/d101e913-ebd1-4e08-b728-82218f47123b/f5297dcd-d9e2-4174-98d4-ada2947e9df5/e0d894c7-fa45-4b97-bd7c-86f3d038d141"
+					(reference "R150")
+					(unit 1)
+				)

Commit message: Mejoras en el rut
Parts:
- removed C6, C7: 100pF, Capacitor_SMD:C_0402_1005Metric, symbol Device:C
- removed R14: 5k, Resistor_SMD:R_0402_1005Metric, symbol Device:R
- removed R149: 0, Resistor_SMD:R_0603_1608Metric, symbol Device:R
- removed R15: 2k, Resistor_SMD:R_0402_1005Metric, symbol Device:R
- renumbered C2 to C10, C3 to C11, C4 to C12, C5 to C13, C8 to C16, C9 to C17, C10 to C18, C11 to C19, C12 to C20, C13 to C21, C14 to C22, C15 to C23, C16 to C24, C17 to C25, C181 to C26, D6 to D10, D7 to D11, D8 to D12, D9 to D13, D10 to D14, D11 to D15, D12 to D16, D13 to D17, D14 to D18, D15 to D19, D5 to D9, R4 to R17, R5 to R18, R6 to R19, R7 to R20, R8 to R21, R9 to R22, R10 to R23, R11 to R24, R12 to R25, R13 to R26, R16 to R29, U2 to U3, U3 to U4, U4 to U5
Connections:
- net +12V: now also C11.2, C12.1, D14.2 (A), R20.1, T1.4, U4.3 (VIN)
Other:
- moved on the sheet: C10, C16, D10, D11, D12, D13, D9, R17, R18, R19, R24, R25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

Commit message: Todo Listo para mandar
Parts:
- added C192, C195: 100pF, Capacitor_SMD:C_0603_1608Metric, symbol Device:C_Small
- added TP28: TestPoint, TestPoint:TestPoint_Pad_D1.0mm, symbol Connector:TestPoint
Connections:
- net +IN: now also C192.1
- net -IN: now also C195.1
- net GND: now also C192.2, C195.2
- net ISO_GND: now also TP28.1
Other:
- moved on the sheet: C10, C16, C19, C25, C26, D10, D11, D12, D13, D9, R17, R18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

Commit message: Solo falta mandar a hacer
Parts:
- D10, D9: footprint Diode_SMD:D_SOD-323F -> Diode_SMD:D_SMA
