File: PCB/InverterV2.0/Primero_esquematico/Primero_esquematico.kicad_sch (KiCad schematic)
At the start: 5 parts, among them J1 349128022

Commit message: agus bancame un toque con esto
Parts:
- removed J1: 349128022, NuevoGui:CONN_SD-34912-001_02_MOL, symbol Snapeda:349128022
- added D88: APT2012EC, LED_SMD:LED_0805_2012Metric, symbol Device:LED
- added F2: 4A, Fuse:Fuse_0805_2012Metric, symbol Device:Fuse
- added J10: 440670201, Snapeda:CONN_SD-44067-001_02_MOL, symbol Snapeda:440670201
- added Q1: IRF4905STRLPBF, Snapeda:TRAN_IRF4905STRLPBF_INF-L, symbol Snapeda:IRF4905STRLPBF
- added R187, R188: 10k, Resistor_SMD:R_0603_1608Metric, symbol Device:R
- added R189: 1k 1/8W, Resistor_SMD:R_0603_1608Metric, symbol Device:R
- added R190: 100, Resistor_SMD:R_0603_1608Metric, symbol Device:R
Connections:
- net +12V: now also D88.2 (A), Q1.3, R187.2; no longer D1.1 (A1)
- net GND: now also J10.2, R188.1, R189.1
- new net: R187.1, R188.2, R190.1
- new net: Q1.1, R190.2
- new net: D1.1 (A1), F2.2, Q1.2
- new net: D88.1 (K), R189.2
- new net +12V_In: F2.1, J10.1
Other:
- note removed: "Chequear si este capa nos sirve o si tengo q poner una mas grande"
- moved on the sheet: C1, C184, C185, D1

Commit message: aislacion encoder
Connections:
- no-connect marks 1 -> 0
Other:
- sheet pcb_logica ports: added none; removed Temp_PCB
Changed lines of the file:
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@@
 		(color 0 0 0 0)
-	)
-	(no_connect
-		(at 115.57 62.23)
 	)
 	(wire
@@
 			(effects
 				(font
-					(size 1.27 1.27)
-				)
-				(justify left)
-			)
-		)
-		(pin "Temp_PCB" bidirectional
-			(at 115.57 62.23 180)
-			(effects
-				(font

Commit message: Mejoras en el rut
Parts:
- added He1: GND_chasis, MountingHole:MountingHole_2.2mm_M2_DIN965_Pad, symbol Mechanical:MountingHole_Pad
- renumbered C185 to C1, C184 to C2, C1 to C3, D88 to D2, F2 to F1, J10 to J1, R190 to R1, R187 to R2, R188 to R3, R189 to R4
Connections:
- net GND: now also He1.1
Other:
- moved on the sheet: C1, C2, C3, D1, D2, F1, J1, Q1, R1, R2, R3, R4

Commit message: Todo Listo para mandar
Parts:
- added He2, He3, He4: GND_chasis, MountingHole:MountingHole_2.2mm_M2_DIN965_Pad, symbol Mechanical:MountingHole_Pad
- added TP40, TP41, TP42, TP43, TP44, TP45, TP46, TP47: TestPoint, TestPoint:TestPoint_Pad_D1.0mm, symbol Connector:TestPoint
Connections:
- net GND: now also He2.1, He3.1, He4.1, TP40.1, TP41.1, TP42.1, TP43.1, TP44.1, TP45.1, TP46.1, TP47.1
Other:
- moved on the sheet: He1

Commit message: el drc esta tirando mucho error hay q solucionar eso
Changed lines of the file:
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@@
+	)
+	(symbol
+		(lib_id "power:+12V")
+		(at 264.16 72.39 0)
+		(mirror y)
+		(unit 1)
+		(body_style 1)
+		(exclude_from_sim no)
+		(in_bom yes)
+		(on_board yes)
+		(in_pos_files yes)
+		(dnp no)
+		(property "Reference" "#PWR0210"
+			(at 264.16 76.2 0)
+			(hide yes)
+			(show_name no)
+			(do_not_autoplace no)
+			(effects
+				(font
+					(size 1.27 1.27)
+				)
+			)
+		)
+		(property "Value" "+12V_In"
+			(at 267.716 67.818 0)
+			(show_name no)
+			(do_not_autoplace no)
+			(effects
+				(font
+					(size 1.27 1.27)
+				)
+				(justify left)
+			)
+		)
+		(property "Footprint" ""
+			(at 264.16 72.39 0)
+			(hide yes)
+			(show_name no)
+			(do_not_autoplace no)
+			(effects
+				(font
+					(size 1.27 1.27)
+				)
+			)
+		)
+		(property "Datasheet" ""
+			(at 264.16 72.39 0)
+			(hide yes)
+			(show_name no)
+			(do_not_autoplace no)
+			(effects
+				(font
+					(size 1.27 1.27)
+				)
+			)
+		)
+		(property "Description" "Power symbol creates a global label with name \"+12V\""
+			(at 264.16 72.39 0)
+			(hide yes)
+			(show_name no)
+			(do_not_autoplace no)
+			(effects
+				(font
+					(size 1.27 1.27)
+				)
+			)
+		)
+		(pin "1"
+		)
+		(instances
+			(project "Primero_esquematico"
+				(path "/d930f486-f6ac-489c-907e-47f2cb34cf04"
+					(reference "#PWR0210")
+					(unit 1)
+				)
+			)
+		)
 	)
 	(symbol
@@
 					(unit 1)
 				)
+			)
+		)
+	)
+	(symbol
+		(lib_id "power:PWR_FLAG")
+		(at 264.16 72.39 180)
+		(unit 1)
+		(body_style 1)
+		(exclude_from_sim no)
+		(in_bom yes)
+		(on_board yes)
+		(in_pos_files yes)
+		(dnp no)
+		(fields_autoplaced yes)
+		(property "Reference" "#FLG024"
+			(at 264.16 74.295 0)
+			(hide yes)
+			(show_name no)
+			(do_not_autoplace no)
+			(effects
+				(font
+					(size 1.27 1.27)
+				)
+			)
+		)
+		(property "Value" "PWR_FLAG"
+			(at 264.16 77.47 0)
+			(show_name no)
+			(do_not_autoplace no)
+			(effects
+				(font
+					(size 1.27 1.27)
+				)
+			)
+		)
+		(property "Footprint" ""
+			(at 264.16 72.39 0)
+			(hide yes)
+			(show_name no)
+			(do_not_autoplace no)
+			(effects
+				(font
+					(size 1.27 1.27)
+				)
+			)
+		)
+		(property "Datasheet" ""
+			(at 264.16 72.39 0)
+			(hide yes)
+			(show_name no)
+			(do_not_autoplace no)
+			(effects
+				(font
+					(size 1.27 1.27)
+				)
+			)
+		)
+		(property "Description" "Special symbol for telling ERC where power comes from"
+			(at 264.16 72.39 0)
+			(hide yes)
+			(show_name no)
+			(do_not_autoplace no)
+			(effects
+				(font
+					(size 1.27 1.27)
+				)
+			)
+		)
+		(pin "1"
+		)
+		(instances
+			(project "Primero_esquematico"
+				(path "/d930f486-f6ac-489c-907e-47f2cb34cf04"
+					(reference "#FLG024")
+					(unit 1)
+				)
