File: PCB/InverterV2.0/Primero_esquematico/SensorTension.kicad_sch (KiCad schematic)
At the start: 70 parts, among them U19 AMC1311BQDWVRQ1, U20 AMC1311BQDWVRQ1, U21 AMC1311BQDWVRQ1, U22 AMC1311BQDWVRQ1, U23 TLV9004QDRQ1

Commit message: Mejoras en el rut
Parts:
- renumbered C121 to C132, C122 to C133, C123 to C134, C124 to C135, C125 to C136, C126 to C137, C127 to C138, C128 to C139, C129 to C140, C130 to C141, C131 to C142, C132 to C143, C133 to C144, C134 to C145, C135 to C146, C136 to C147, C137 to C148, R92 to R110, R93 to R111, R94 to R112, R95 to R113, R96 to R114, R97 to R115, R98 to R116, R99 to R117, R100 to R118, R101 to R119, R102 to R120, R103 to R121, R104 to R122, R105 to R123, R106 to R124, R107 to R125, R108 to R126, R109 to R127, R110 to R128, R111 to R129, R112 to R130, R113 to R131, R114 to R132, R115 to R133, R116 to R134, R117 to R135, R118 to R136, R119 to R137, R120 to R138, R121 to R139, R122 to R140, R123 to R141, R124 to R142, R125 to R143, R126 to R144, R127 to R145, R128 to R146, R129 to R147, R130 to R148, R131 to R149, R132 to R150, R133 to R151, R134 to R152, R135 to R153, R136 to R154, R137 to R155, R138 to R156, R139 to R157, U19 to U20, U20 to U21, U21 to U22, U22 to U23, U23 to U24

Commit message: Casi listo
Connections:
- net +3.3V_analog renamed +3.3V_analog_2
