File: PCB/InverterV2.0/Primero_esquematico/SistemasProteccion.kicad_sch (KiCad schematic)
At the start: 8 parts, among them U30 TLV1702AQDGKRQ1

Commit message: agus bancame un toque con esto
Other:
- note added: "ESTE GRAFICO LO TENDRIA Q CAMBIAR PARA QUE SE ABRA CUANDO SE LOGRA PASAR LOS 60V ME SIRVE MAS ESE DATO"
Changed lines of the file:
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@@
+		)
+	)
+	(text "ESTE GRAFICO LO TENDRIA Q CAMBIAR PARA QUE SE ABRA CUANDO\nSE LOGRA PASAR LOS 60V ME SIRVE MAS ESE DATO"
+		(exclude_from_sim no)
+		(at 153.67 160.782 0)
+		(effects
+			(font
+				(size 2.54 2.54)
+			)
 		)
 	)

Commit message: Mejoras en el rut
Parts:
- renumbered C195 to C159, R220 to R164, R221 to R165, R219 to R166, R222 to R167, R223 to R168, R224 to R169, U30 to U31
Changed lines of the file:
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@@
 		(in_pos_files yes)
 		(dnp no)
-		(property "Reference" "U30"
+		(property "Reference" "U31"
 			(at 106.426 108.458 0)
 			(show_name no)
@@
 			(project "Primero_esquematico"
 				(path "/d930f486-f6ac-489c-907e-47f2cb34cf04/0bcc01e0-1903-49c9-8a02-17640b3194e7/80b781e6-4eb0-4935-8380-fde54fe82eff"
-					(reference "U30")
+					(reference "U31")
 					(unit 1)
 				)
@@
 		(dnp no)
 		(fields_autoplaced yes)
-		(property "Reference" "R223"
+		(property "Reference" "R168"
 			(at 64.77 161.2899 0)
 			(show_name no)
@@
 			(project "Primero_esquematico"
 				(path "/d930f486-f6ac-489c-907e-47f2cb34cf04/0bcc01e0-1903-49c9-8a02-17640b3194e7/80b781e6-4eb0-4935-8380-fde54fe82eff"
-					(reference "R223")
+					(reference "R168")
 					(unit 1)
 				)
@@
 		(dnp no)
 		(fields_autoplaced yes)
-		(property "Reference" "#PWR0179"
+		(property "Reference" "#PWR0205"
 			(at 62.23 97.79 0)
 			(hide yes)
@@
 			(project "Primero_esquematico"
 				(path "/d930f486-f6ac-489c-907e-47f2cb34cf04/0bcc01e0-1903-49c9-8a02-17640b3194e7/80b781e6-4eb0-4935-8380-fde54fe82eff"
-					(reference "#PWR0179")
+					(reference "#PWR0205")
 					(unit 1)
 				)
@@
 		(dnp no)
 		(fields_autoplaced yes)
-		(property "Reference" "R220"
+		(property "Reference" "R164"
 			(at 64.77 96.5199 0)
 			(show_name no)
@@
 			(project "Primero_esquematico"
 				(path "/d930f486-f6ac-489c-907e-47f2cb34cf04/0bcc01e0-1903-49c9-8a02-17640b3194e7/80b781e6-4eb0-4935-8380-fde54fe82eff"
-					(reference "R220")
+					(reference "R164")
 					(unit 1)
 				)
@@
 		(in_pos_files yes)
 		(dnp no)
-		(property "Reference" "#PWR0318"
+		(property "Reference" "#PWR0210"
 			(at 128.27 118.11 0)
 			(hide yes)
@@
 			(project "Primero_esquematico"
 				(path "/d930f486-f6ac-489c-907e-47f2cb34cf04/0bcc01e0-1903-49c9-8a02-17640b3194e7/80b781e6-4eb0-4935-8380-fde54fe82eff"
-					(reference "#PWR0318")
+					(reference "#PWR0210")
 					(unit 1)
 				)
@@
 		(dnp no)
 		(fields_autoplaced yes)
-		(property "Reference" "#PWR0180"
+		(property "Reference" "#PWR0207"
 			(at 62.23 152.4 0)
 			(hide yes)
@@
 			(project "Primero_esquematico"
 				(path "/d930f486-f6ac-489c-907e-47f2cb34cf04/0bcc01e0-1903-49c9-8a02-17640b3194e7/80b781e6-4eb0-4935-8380-fde54fe82eff"
-					(reference "#PWR0180")
+					(reference "#PWR0207")
 					(unit 1)
 				)
@@
 		(dnp no)
 		(fields_autoplaced yes)
-		(property "Reference" "#PWR0320"
+		(property "Reference" "#PWR0206"
 			(at 62.23 118.11 0)
 			(hide yes)
@@
 			(project "Primero_esquematico"
 				(path "/d930f486-f6ac-489c-907e-47f2cb34cf04/0bcc01e0-1903-49c9-8a02-17640b3194e7/80b781e6-4eb0-4935-8380-fde54fe82eff"
-					(reference "#PWR0320")
+					(reference "#PWR0206")
 					(unit 1)
 				)
@@
 		(dnp no)
 		(fields_autoplaced yes)
-		(property "Reference" "#PWR0321"
+		(property "Reference" "#PWR0208"
 			(at 62.23 172.72 0)
 			(hide yes)
@@
 			(project "Primero_esquematico"
 				(path "/d930f486-f6ac-489c-907e-47f2cb34cf04/0bcc01e0-1903-49c9-8a02-17640b3194e7/80b781e6-4eb0-4935-8380-fde54fe82eff"
-					(reference "#PWR0321")
+					(reference "#PWR0208")
 					(unit 1)
 				)
@@
 		(in_pos_files yes)
 		(dnp no)
-		(property "Reference" "#PWR0322"
+		(property "Reference" "#PWR0212"
 			(at 146.05 114.3 0)
 			(hide yes)
@@
 			(project "Primero_esquematico"
 				(path "/d930f486-f6ac-489c-907e-47f2cb34cf04/0bcc01e0-1903-49c9-8a02-17640b3194e7/80b781e6-4eb0-4935-8380-fde54fe82eff"
-					(reference "#PWR0322")
+					(reference "#PWR0212")
 					(unit 1)
 				)
@@
 		(dnp no)
 		(fields_autoplaced yes)
-		(property "Reference" "R219"
+		(property "Reference" "R166"
 			(at 62.23 119.38 90)
 			(show_name no)
@@
 			(project "Primero_esquematico"
 				(path "/d930f486-f6ac-489c-907e-47f2cb34cf04/0bcc01e0-1903-49c9-8a02-17640b3194e7/80b781e6-4eb0-4935-8380-fde54fe82eff"
-					(reference "R219")
+					(reference "R166")
 					(unit 1)
 				)
@@
 		(dnp no)
 		(fields_autoplaced yes)
-		(property "Reference" "R222"
+		(property "Reference" "R167"
 			(at 64.77 151.1299 0)
 			(show_name no)
@@
 			(project "Primero_esquematico"
 				(path "/d930f486-f6ac-489c-907e-47f2cb34cf04/0bcc01e0-1903-49c9-8a02-17640b3194e7/80b781e6-4eb0-4935-8380-fde54fe82eff"
-					(reference "R222")
+					(reference "R167")
 					(unit 1)
 				)
@@
 		(dnp no)
 		(fields_autoplaced yes)
-		(property "Reference" "#PWR0319"
+		(property "Reference" "#PWR0209"
 			(at 67.31 143.51 0)
 			(hide yes)
@@
 			(project "Primero_esquematico"
 				(path "/d930f486-f6ac-489c-907e-47f2cb34cf04/0bcc01e0-1903-49c9-8a02-17640b3194e7/80b781e6-4eb0-4935-8380-fde54fe82eff"
-					(reference "#PWR0319")
+					(reference "#PWR0209")
 					(unit 1)
 				)
@@
 		(dnp no)
 		(fields_autoplaced yes)
-		(property "Reference" "#PWR0323"
+		(property "Reference" "#PWR0211"
 			(at 124.46 143.51 0)
 			(hide yes)
@@
 			(project "Primero_esquematico"
 				(path "/d930f486-f6ac-489c-907e-47f2cb34cf04/0bcc01e0-1903-49c9-8a02-17640b3194e7/80b781e6-4eb0-4935-8380-fde54fe82eff"
-					(reference "#PWR0323")
+					(reference "#PWR0211")
 					(unit 1)
 				)
@@
 		(dnp no)
 		(fields_autoplaced yes)
-		(property "Reference" "R221"
+		(property "Reference" "R165"
 			(at 64.77 106.6799 0)
 			(show_name no)
@@
 			(project "Primero_esquematico"
 				(path "/d930f486-f6ac-489c-907e-47f2cb34cf04/0bcc01e0-1903-49c9-8a02-17640b3194e7/80b781e6-4eb0-4935-8380-fde54fe82eff"
-					(reference "R221")
+					(reference "R165")
 					(unit 1)
 				)
@@
 		(dnp no)
 		(fields_autoplaced yes)
-		(property "Reference" "R224"
+		(property "Reference" "R169"
 			(at 144.78 115.5699 0)
 			(show_name no)
@@
 			(project "Primero_esquematico"
 				(path "/d930f486-f6ac-489c-907e-47f2cb34cf04/0bcc01e0-1903-49c9-8a02-17640b3194e7/80b781e6-4eb0-4935-8380-fde54fe82eff"
-					(reference "R224")
+					(reference "R169")
 					(unit 1)
 				)
@@
 		(in_pos_files yes)
 		(dnp no)
-		(property "Reference" "C195"
+		(property "Reference" "C159"
 			(at 63.5 130.8099 0)
 			(show_name no)
@@
 			(project "Primero_esquematico"
 				(path "/d930f486-f6ac-489c-907e-47f2cb34cf04/0bcc01e0-1903-49c9-8a02-17640b3194e7/80b781e6-4eb0-4935-8380-fde54fe82eff"
-					(reference "C195")
-					(unit 1)
-				)
+					(reference "C159")
+					(unit 1)
+				)

Commit message: Casi listo
Connections:
- net +3.3V_analog renamed +3.3V_analog_2
Changed lines of the file:
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@@
-	)
-	(symbol
-		(lib_id "power:+3.3VP")
-		(at 124.46 116.84 0)
-		(unit 1)
-		(body_style 1)
-		(exclude_from_sim no)
-		(in_bom yes)
-		(on_board yes)
-		(in_pos_files yes)
-		(dnp no)
-		(property "Reference" "#PWR0210"
-			(at 128.27 118.11 0)
-			(hide yes)
-			(show_name no)
-			(do_not_autoplace no)
-			(effects
-				(font
-					(size 1.27 1.27)
-				)
-			)
-		)
-		(property "Value" "+3.3V_analog"
-			(at 121.92 112.776 0)
-			(show_name no)
-			(do_not_autoplace no)
-			(effects
-				(font
-					(size 1.27 1.27)
-				)
-				(justify left)
-			)
-		)
-		(property "Footprint" ""
-			(at 124.46 116.84 0)
-			(hide yes)
-			(show_name no)
-			(do_not_autoplace no)
-			(effects
-				(font
-					(size 1.27 1.27)
-				)
-			)
-		)
-		(property "Datasheet" ""
-			(at 124.46 116.84 0)
-			(hide yes)
-			(show_name no)
-			(do_not_autoplace no)
-			(effects
-				(font
-					(size 1.27 1.27)
-				)
-			)
-		)
-		(property "Description" "Power symbol creates a global label with name \"+3.3VP\""
-			(at 124.46 116.84 0)
-			(hide yes)
-			(show_name no)
-			(do_not_autoplace no)
-			(effects
-				(font
-					(size 1.27 1.27)
-				)
-			)
-		)
-		(pin "1"
-		)
-		(instances
-			(project "Primero_esquematico"
-				(path "/d930f486-f6ac-489c-907e-47f2cb34cf04/0bcc01e0-1903-49c9-8a02-17640b3194e7/80b781e6-4eb0-4935-8380-fde54fe82eff"
-					(reference "#PWR0210")
-					(unit 1)
-				)
-			)
-		)
 	)
 	(symbol
@@
 	)
 	(symbol
+		(lib_id "power:+3.3VP")
+		(at 124.46 116.84 0)
+		(unit 1)
+		(body_style 1)
+		(exclude_from_sim no)
+		(in_bom yes)
+		(on_board yes)
+		(in_pos_files yes)
+		(dnp no)
+		(property "Reference" "#PWR0358"
+			(at 128.27 118.11 0)
+			(hide yes)
+			(show_name no)
+			(do_not_autoplace no)
+			(effects
+				(font
+					(size 1.27 1.27)
+				)
+			)
+		)
+		(property "Value" "+3.3V_analog_2"
+			(at 120.142 111.252 0)
+			(show_name no)
+			(do_not_autoplace no)
+			(effects
+				(font
+					(size 1.27 1.27)
+				)
+				(justify left)
+			)
+		)
+		(property "Footprint" ""
+			(at 124.46 116.84 0)
+			(hide yes)
+			(show_name no)
+			(do_not_autoplace no)
+			(effects
+				(font
+					(size 1.27 1.27)
+				)
+			)
+		)
+		(property "Datasheet" ""
+			(at 124.46 116.84 0)
+			(hide yes)
+			(show_name no)
+			(do_not_autoplace no)
+			(effects
+				(font
+					(size 1.27 1.27)
+				)
+			)
+		)
+		(property "Description" "Power symbol creates a global label with name \"+3.3VP\""
+			(at 124.46 116.84 0)
+			(hide yes)
+			(show_name no)
+			(do_not_autoplace no)
+			(effects
+				(font
+					(size 1.27 1.27)
+				)
+			)
+		)
+		(pin "1"
+		)
+		(instances
+			(project "Primero_esquematico"
+				(path "/d930f486-f6ac-489c-907e-47f2cb34cf04/0bcc01e0-1903-49c9-8a02-17640b3194e7/80b781e6-4eb0-4935-8380-fde54fe82eff"
+					(reference "#PWR0358")
+					(unit 1)
+				)
+			)
+		)
+	)
+	(symbol
 		(lib_id "power:GND")
 		(at 62.23 111.76 0)
@@
 	)
 	(symbol
-		(lib_id "power:+3.3VP")
-		(at 142.24 113.03 0)
-		(unit 1)
-		(body_style 1)
-		(exclude_from_sim no)
-		(in_bom yes)
-		(on_board yes)
-		(in_pos_files yes)
-		(dnp no)
-		(property "Reference" "#PWR0212"
-			(at 146.05 114.3 0)
-			(hide yes)
-			(show_name no)
-			(do_not_autoplace no)
-			(effects
-				(font
-					(size 1.27 1.27)
-				)
-			)
-		)
-		(property "Value" "+3.3V_analog"
-			(at 139.7 108.966 0)
-			(show_name no)
-			(do_not_autoplace no)
-			(effects
-				(font
-					(size 1.27 1.27)
-				)
-				(justify left)
-			)
-		)
-		(property "Footprint" ""
-			(at 142.24 113.03 0)
-			(hide yes)
-			(show_name no)
-			(do_not_autoplace no)
-			(effects
-				(font
-					(size 1.27 1.27)
-				)
-			)
-		)
-		(property "Datasheet" ""
-			(at 142.24 113.03 0)
-			(hide yes)
-			(show_name no)
-			(do_not_autoplace no)
-			(effects
-				(font
-					(size 1.27 1.27)
-				)
-			)
-		)
-		(property "Description" "Power symbol creates a global label with name \"+3.3VP\""
-			(at 142.24 113.03 0)
-			(hide yes)
-			(show_name no)
-			(do_not_autoplace no)
-			(effects
-				(font
-					(size 1.27 1.27)
-				)
-			)
-		)
-		(pin "1"
-		)
-		(instances
-			(project "Primero_esquematico"
-				(path "/d930f486-f6ac-489c-907e-47f2cb34cf04/0bcc01e0-1903-49c9-8a02-17640b3194e7/80b781e6-4eb0-4935-8380-fde54fe82eff"
-					(reference "#PWR0212")
-					(unit 1)
-				)
-			)
-		)
-	)
-	(symbol
 		(lib_id "Device:R")
 		(at 62.23 125.73 90)
@@
 					(unit 1)
 				)
+			)
+		)
+	)
+	(symbol
+		(lib_id "power:+3.3VP")
+		(at 142.24 113.03 0)
+		(unit 1)
+		(body_style 1)
+		(exclude_from_sim no)
+		(in_bom yes)
+		(on_board yes)
+		(in_pos_files yes)
+		(dnp no)
+		(property "Reference" "#PWR0357"
+			(at 146.05 114.3 0)
+			(hide yes)
+			(show_name no)
+			(do_not_autoplace no)
+			(effects
+				(font
+					(size 1.27 1.27)
+				)
+			)
+		)
+		(property "Value" "+3.3V_analog_2"
+			(at 137.922 107.442 0)
+			(show_name no)
+			(do_not_autoplace no)
+			(effects
+				(font
+					(size 1.27 1.27)
+				)
+				(justify left)
+			)
+		)
+		(property "Footprint" ""
+			(at 142.24 113.03 0)
+			(hide yes)
+			(show_name no)
+			(do_not_autoplace no)
+			(effects
+				(font
+					(size 1.27 1.27)
+				)
+			)
+		)
+		(property "Datasheet" ""
+			(at 142.24 113.03 0)
+			(hide yes)
+			(show_name no)
+			(do_not_autoplace no)
+			(effects
+				(font
+					(size 1.27 1.27)
+				)
+			)
+		)
+		(property "Description" "Power symbol creates a global label with name \"+3.3VP\""
+			(at 142.24 113.03 0)
+			(hide yes)
+			(show_name no)
+			(do_not_autoplace no)
+			(effects
+				(font
+					(size 1.27 1.27)
+				)
+			)
+		)
+		(pin "1"
+		)
+		(instances
+			(project "Primero_esquematico"
+				(path "/d930f486-f6ac-489c-907e-47f2cb34cf04/0bcc01e0-1903-49c9-8a02-17640b3194e7/80b781e6-4eb0-4935-8380-fde54fe82eff"
+					(reference "#PWR0357")
+					(unit 1)
+				)
