File: PCB/InverterV2.0/Primero_esquematico/apps.kicad_sch (KiCad schematic)
At the start: 19 parts, among them J6 347928082, U39 OPA2196xD

Commit message: Mejoras en el rut
Parts:
- renumbered C176 to C4, C177 to C5, C179 to C6, C174 to C7, C175 to C8, C178 to C9, D81 to D3, D80 to D4, D86 to D5, J6 to J2, R200 to R10, R195 to R11, R196 to R12, R199 to R5, R203 to R6, R202 to R7, R204 to R8, R205 to R9, U39 to U1

Commit message: Casi listo
Connections:
- net opamp_1: now also D3.2 (A2); no longer D3.1 (A1)
- net opamp_2: now also D3.1 (A1); no longer D3.2 (A2)
- net +3.3V_analog renamed +3.3V_analog_2
