File: PCB/InverterV2.0/Primero_esquematico/comunicacionCAN.kicad_sch (KiCad schematic)
At the start: 12 parts, among them J2 347920040, J3 347920040, U33 ISO1042DWR, U34 ISO1042DWR

Commit message: agus bancame un toque con esto
Parts:
- removed J2: 347920040, Snapeda:CONN04_34792_MOL, symbol Snapeda:347920040
- added F1: 100mA, Fuse:Fuse_0603_1608Metric, symbol Device:Fuse
- added PS1: MEV1S1205SC, Snapeda:MEV1S1205SC, symbol Snapeda:MEV1S1205SC
- added R186: 220 1/4W, Resistor_SMD:R_0805_2012Metric, symbol Device:R_Small
Connections:
- net +5V_Can_1: no longer C158.1, U33.11 (VCC2), U33.16 (VCC2)
- net +5V_Can_2: no longer C157.1, J3.4, U34.11 (VCC2), U34.16 (VCC2)
- net GND_Can_1: no longer D82.3 (common), U33.10 (GND2), U33.15 (GND2), U33.9 (GND2)
- net GND_Can_2: no longer C157.2, D83.3 (common), J3.3, U34.10 (GND2), U34.15 (GND2), U34.9 (GND2)
- net at D82.1 (A1), R174.1, U33.13 (CANH): now also J3.4
- net at D82.2 (A2), R174.2, U33.12 (CANL): now also J3.3
- new net: F1.1, PS1.7 (+VOUT)
- new net +12V: PS1.1 (+VIN)
- new net +5V_Can: C157.1, C158.1, F1.2, R186.1, U33.11 (VCC2), U33.16 (VCC2), U34.11 (VCC2), U34.16 (VCC2)
- new net GND_Can: C157.2, D82.3 (common), D83.3 (common), PS1.5 (-VOUT), R186.2, U33.10 (GND2), U33.15 (GND2), U33.9 (GND2), U34.10 (GND2), U34.15 (GND2), U34.9 (GND2)
- no-connect marks 8 -> 9
Other:
- note added: "Esta resistencia cumple la funcion de estabilizar la salida con una carga minima"

Commit message: aislacion encoder
Parts:
- added J11: 347920040, Snapeda:CONN04_34792_MOL, symbol Snapeda:347920040
Connections:
- net +5V_Can: now also J3.4, J11.4
- net GND_Can: now also J3.1, J11.1
- net at D82.1 (A1), R174.1, U33.13 (CANH): now also J11.3; no longer J3.4
- net at D82.2 (A2), R174.2, U33.12 (CANL): now also J11.2; no longer J3.3
- net at D83.2 (A2), R175.2, U34.12 (CANL): now also J3.2; no longer J3.1
- net at D83.1 (A1), R175.1, U34.13 (CANH): now also J3.3; no longer J3.2
Other:
- moved on the sheet: F1, R186, Reference: PS1

Commit message: Mejoras en el rut
Parts:
- removed F1: 100mA, Fuse:Fuse_0603_1608Metric, symbol Device:Fuse
- removed J11, J3: 347920040, Snapeda:CONN04_34792_MOL, symbol Snapeda:347920040
- added C172: 10nF, Capacitor_SMD:C_0603_1608Metric, symbol Device:C
- added C173: 10uF, Capacitor_SMD:C_0805_2012Metric, symbol Device:C
- added J6: 1053091205, Snapeda:CONN_SD-105309-100_05_MOL, symbol Snapeda:1053091205
- added L3: MLZ2012N6R8LT000, Inductor_SMD:L_0805_2012Metric, symbol Device:L
- PS1: MANUFACTURER_PART_NUMBER (none) -> MEV1S1205SC; Manufacturer_Part_Number MEV1S1205SC -> (none)
- renumbered C155 to C168, C156 to C169, C157 to C170, C158 to C171, D82 to D86, D83 to D87, R174 to R178, R175 to R179, R186 to R180
Connections:
- net +12V: now also L3.2; no longer PS1.1 (+VIN)
- net +5V_Can: now also PS1.7 (+VOUT)
- net GND: now also PS1.2 (-VIN), C172.2, C173.2
- net GND_Can: now also J6.3
- net CAN_H_1: now reaches D86.1 (A1), R178.1, U33.13 (CANH)
- net CAN_H_1: now also J6.5
- net CAN_L_1: now reaches D86.2 (A2), R178.2, U33.12 (CANL)
- net CAN_L_1: now also J6.4
- net CAN_H_2: now reaches D87.1 (A1), R179.1, U34.13 (CANH)
- net CAN_H_2: now also J6.2
- net CAN_L_2: now reaches D87.2 (A2), R179.2, U34.12 (CANL)
- net CAN_L_2: now also J6.1
- new net: C172.1, C173.1, L3.1, PS1.1 (+VIN)
Other:
- moved on the sheet: R180, Reference: PS1

Commit message: el drc esta tirando mucho error hay q solucionar eso
Connections:
- net GND_Can_1 is gone; now on net GND_Can: C171.2
