File: PCB/InverterV2.0/Primero_esquematico/conectores_externos.kicad_sch (KiCad schematic)
At the start: 7 parts, among them J4 347928082

Commit message: Mejoras en el rut
Parts:
- renumbered D87 to D88, J4 to J7, R176 to R181, R177 to R182, R178 to R183, R179 to R184
Changed lines of the file:
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@@
 		(in_pos_files yes)
 		(dnp no)
-		(property "Reference" "J4"
+		(property "Reference" "J7"
 			(at 247.65 107.696 0)
 			(show_name no)
@@
 			(project "Primero_esquematico"
 				(path "/d930f486-f6ac-489c-907e-47f2cb34cf04/0bcc01e0-1903-49c9-8a02-17640b3194e7/49867297-e849-416a-bae2-6d0463384f96"
-					(reference "J4")
+					(reference "J7")
 					(unit 1)
 				)
@@
 		(in_pos_files yes)
 		(dnp no)
-		(property "Reference" "#PWR0236"
+		(property "Reference" "#PWR0275"
 			(at 227.33 104.14 0)
 			(hide yes)
@@
 			(project "Primero_esquematico"
 				(path "/d930f486-f6ac-489c-907e-47f2cb34cf04/0bcc01e0-1903-49c9-8a02-17640b3194e7/49867297-e849-416a-bae2-6d0463384f96"
-					(reference "#PWR0236")
+					(reference "#PWR0275")
 					(unit 1)
 				)
@@
 		(in_pos_files yes)
 		(dnp no)
-		(property "Reference" "#PWR0326"
+		(property "Reference" "#PWR0274"
 			(at 227.33 69.85 0)
 			(hide yes)
@@
 			(project "Primero_esquematico"
 				(path "/d930f486-f6ac-489c-907e-47f2cb34cf04/0bcc01e0-1903-49c9-8a02-17640b3194e7/49867297-e849-416a-bae2-6d0463384f96"
-					(reference "#PWR0326")
+					(reference "#PWR0274")
 					(unit 1)
 				)
@@
 		(dnp no)
 		(fields_autoplaced yes)
-		(property "Reference" "#PWR0237"
+		(property "Reference" "#PWR0276"
 			(at 231.14 125.73 0)
 			(hide yes)
@@
 			(project "Primero_esquematico"
 				(path "/d930f486-f6ac-489c-907e-47f2cb34cf04/0bcc01e0-1903-49c9-8a02-17640b3194e7/49867297-e849-416a-bae2-6d0463384f96"
-					(reference "#PWR0237")
+					(reference "#PWR0276")
 					(unit 1)
 				)
@@
 		(in_pos_files yes)
 		(dnp no)
-		(property "Reference" "D87"
+		(property "Reference" "D88"
 			(at 246.38 57.912 0)
 			(show_name no)
@@
 			(project "Primero_esquematico"
 				(path "/d930f486-f6ac-489c-907e-47f2cb34cf04/0bcc01e0-1903-49c9-8a02-17640b3194e7/49867297-e849-416a-bae2-6d0463384f96"
-					(reference "D87")
+					(reference "D88")
 					(unit 1)
 				)
@@
 		(in_pos_files yes)
 		(dnp no)
-		(property "Reference" "R177"
+		(property "Reference" "R182"
 			(at 167.64 106.6799 0)
 			(show_name no)
@@
 			(project "Primero_esquematico"
 				(path "/d930f486-f6ac-489c-907e-47f2cb34cf04/0bcc01e0-1903-49c9-8a02-17640b3194e7/49867297-e849-416a-bae2-6d0463384f96"
-					(reference "R177")
+					(reference "R182")
 					(unit 1)
 				)
@@
 		(dnp no)
 		(fields_autoplaced yes)
-		(property "Reference" "#PWR0327"
+		(property "Reference" "#PWR0277"
 			(at 236.22 92.71 0)
 			(hide yes)
@@
 			(project "Primero_esquematico"
 				(path "/d930f486-f6ac-489c-907e-47f2cb34cf04/0bcc01e0-1903-49c9-8a02-17640b3194e7/49867297-e849-416a-bae2-6d0463384f96"
-					(reference "#PWR0327")
+					(reference "#PWR0277")
 					(unit 1)
 				)
@@
 		(dnp no)
 		(fields_autoplaced yes)
-		(property "Reference" "R178"
+		(property "Reference" "R183"
 			(at 177.8 81.2799 0)
 			(show_name no)
@@
 			(project "Primero_esquematico"
 				(path "/d930f486-f6ac-489c-907e-47f2cb34cf04/0bcc01e0-1903-49c9-8a02-17640b3194e7/49867297-e849-416a-bae2-6d0463384f96"
-					(reference "R178")
+					(reference "R183")
 					(unit 1)
 				)
@@
 		(in_pos_files yes)
 		(dnp no)
-		(property "Reference" "#PWR0234"
+		(property "Reference" "#PWR0272"
 			(at 172.72 80.01 0)
 			(hide yes)
@@
 			(project "Primero_esquematico"
 				(path "/d930f486-f6ac-489c-907e-47f2cb34cf04/0bcc01e0-1903-49c9-8a02-17640b3194e7/49867297-e849-416a-bae2-6d0463384f96"
-					(reference "#PWR0234")
+					(reference "#PWR0272")
 					(unit 1)
 				)
@@
 		(dnp no)
 		(fields_autoplaced yes)
-		(property "Reference" "#PWR0235"
+		(property "Reference" "#PWR0273"
 			(at 175.26 118.11 0)
 			(hide yes)
@@
 			(project "Primero_esquematico"
 				(path "/d930f486-f6ac-489c-907e-47f2cb34cf04/0bcc01e0-1903-49c9-8a02-17640b3194e7/49867297-e849-416a-bae2-6d0463384f96"
-					(reference "#PWR0235")
+					(reference "#PWR0273")
 					(unit 1)
 				)
@@
 		(in_pos_files yes)
 		(dnp no)
-		(property "Reference" "R179"
+		(property "Reference" "R184"
 			(at 177.8 106.6799 0)
 			(show_name no)
@@
 			(project "Primero_esquematico"
 				(path "/d930f486-f6ac-489c-907e-47f2cb34cf04/0bcc01e0-1903-49c9-8a02-17640b3194e7/49867297-e849-416a-bae2-6d0463384f96"
-					(reference "R179")
+					(reference "R184")
 					(unit 1)
 				)
@@
 		(dnp no)
 		(fields_autoplaced yes)
-		(property "Reference" "#PWR0233"
+		(property "Reference" "#PWR0271"
 			(at 170.18 118.11 0)
 			(hide yes)
@@
 			(project "Primero_esquematico"
 				(path "/d930f486-f6ac-489c-907e-47f2cb34cf04/0bcc01e0-1903-49c9-8a02-17640b3194e7/49867297-e849-416a-bae2-6d0463384f96"
-					(reference "#PWR0233")
+					(reference "#PWR0271")
 					(unit 1)
 				)
@@
 		(in_pos_files yes)
 		(dnp no)
-		(property "Reference" "R176"
+		(property "Reference" "R181"
 			(at 167.64 81.2799 0)
 			(show_name no)
@@
 			(project "Primero_esquematico"
 				(path "/d930f486-f6ac-489c-907e-47f2cb34cf04/0bcc01e0-1903-49c9-8a02-17640b3194e7/49867297-e849-416a-bae2-6d0463384f96"
-					(reference "R176")
+					(reference "R181")
 					(unit 1)
 				)

Commit message: Casi listo
Connections:
- net TCK: now also J7.3; no longer J7.5
- net TDI: now also J7.6; no longer J7.3
- net TMS: now also J7.5; no longer J7.6
Changed lines of the file:
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@@
+	(hierarchical_label "TDI"
+		(shape bidirectional)
+		(at 232.41 113.03 180)
+		(effects
+			(font
+				(size 1.27 1.27)
+			)
+			(justify right)
+		)
+	)
+	(hierarchical_label "TMS"
+		(shape bidirectional)
+		(at 232.41 110.49 180)
+		(effects
+			(font
+				(size 1.27 1.27)
+			)
+			(justify right)
+		)
+	)
 	(hierarchical_label "TDI"
 		(shape bidirectional)
@@
 		)
 	)
-	(hierarchical_label "TDO"
-		(shape bidirectional)
-		(at 232.41 107.95 180)
-		(effects
-			(font
-				(size 1.27 1.27)
-			)
-			(justify right)
-		)
-	)
-	(hierarchical_label "TDI"
-		(shape bidirectional)
-		(at 232.41 105.41 180)
-		(effects
-			(font
-				(size 1.27 1.27)
-			)
-			(justify right)
-		)
-	)
-	(hierarchical_label "TMS"
-		(shape bidirectional)
-		(at 232.41 113.03 180)
-		(effects
-			(font
-				(size 1.27 1.27)
-			)
-			(justify right)
-		)
-	)
 	(hierarchical_label "Mcu_Reset"
 		(shape bidirectional)
@@
 		(shape bidirectional)
 		(at 168.91 87.63 180)
+		(effects
+			(font
+				(size 1.27 1.27)
+			)
+			(justify right)
+		)
+	)
+	(hierarchical_label "TCK"
+		(shape bidirectional)
+		(at 232.41 105.41 180)
 		(effects
 			(font
@@
 		)
 	)
-	(hierarchical_label "TCK"
+	(hierarchical_label "TDO"
 		(shape bidirectional)
-		(at 232.41 110.49 180)
+		(at 232.41 107.95 180)
 		(effects
 			(font

Commit message: Rooteao de todo solo falta los gate drivers de arriba
Connections:
- net TCK: now also D88.12 (D2P); no longer D88.9 (D3P)
- net TDI: now also D88.8 (D3N); no longer D88.12 (D2P)
- net TMS: now also D88.9 (D3P); no longer D88.8 (D3N)
Changed lines of the file:
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@@
-		)
-	)
-	(hierarchical_label "TCK"
-		(shape bidirectional)
-		(at 232.41 76.2 180)
-		(effects
-			(font
-				(size 1.27 1.27)
-			)
-			(justify right)
 		)
 	)
@@
 		)
 	)
-	(hierarchical_label "TDI"
+	(hierarchical_label "TMS"
 		(shape bidirectional)
-		(at 232.41 71.12 180)
+		(at 232.41 76.2 180)
+		(effects
+			(font
+				(size 1.27 1.27)
+			)
+			(justify right)
+		)
+	)
+	(hierarchical_label "TDO"
+		(shape bidirectional)
+		(at 232.41 73.66 180)
 		(effects
 			(font
@@
 		)
 	)
-	(hierarchical_label "Mcu_Reset"
+	(hierarchical_label "TCK"
 		(shape bidirectional)
-		(at 232.41 68.58 180)
+		(at 232.41 71.12 180)
+		(effects
+			(font
+				(size 1.27 1.27)
+			)
+			(justify right)
+		)
+	)
+	(hierarchical_label "TDI"
+		(shape bidirectional)
+		(at 232.41 78.74 180)
 		(effects
 			(font
@@
 	(hierarchical_label "TDO"
 		(shape bidirectional)
-		(at 232.41 73.66 180)
-		(effects
-			(font
-				(size 1.27 1.27)
-			)
-			(justify right)
-		)
-	)
-	(hierarchical_label "TDO"
-		(shape bidirectional)
 		(at 232.41 107.95 180)
 		(effects
@@
 		)
 	)
-	(hierarchical_label "TMS"
+	(hierarchical_label "Mcu_Reset"
 		(shape bidirectional)
-		(at 232.41 78.74 180)
+		(at 232.41 68.58 180)
 		(effects
 			(font
