File: PCB/InverterV2.0/Primero_esquematico/currentS.kicad_sch (KiCad schematic)
At the start: 23 parts, among them J7 1053091205, J8 1053091205, J9 1053091205, U41 OPA4991QPWRQ1

Commit message: Mejoras en el rut
Parts:
- renumbered C189 to C160, C188 to C161, C186 to C162, C190 to C163, C194 to C164, C193 to C165, C192 to C166, C191 to C167, D79 to D83, J7 to J3, J8 to J4, J9 to J5, R198 to R170, R197 to R171, R211 to R172, R210 to R173, R213 to R174, R212 to R175, R201 to R176, R214 to R177, U41 to U32

Commit message: Casi listo
Connections:
- net +3.3V_analog renamed +3.3V_analog_1
- net +3.3V_analog_1: no longer D84.1 (K1)

Commit message: el drc esta tirando mucho error hay q solucionar eso
Connections:
- net +3.3V_analog_1: now also D84.1 (K1)
Changed lines of the file:
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@@
+	(symbol
+		(lib_id "power:+3.3VP")
+		(at 194.31 121.92 0)
+		(unit 1)
+		(body_style 1)
+		(exclude_from_sim no)
+		(in_bom yes)
+		(on_board yes)
+		(in_pos_files yes)
+		(dnp no)
+		(property "Reference" "#PWR0242"
+			(at 198.12 123.19 0)
+			(hide yes)
+			(show_name no)
+			(do_not_autoplace no)
+			(effects
+				(font
+					(size 1.27 1.27)
+				)
+			)
+		)
+		(property "Value" "+3.3V_analog_1"
+			(at 190.246 116.332 0)
+			(show_name no)
+			(do_not_autoplace no)
+			(effects
+				(font
+					(size 1.27 1.27)
+				)
+				(justify left)
+			)
+		)
+		(property "Footprint" ""
+			(at 194.31 121.92 0)
+			(hide yes)
+			(show_name no)
+			(do_not_autoplace no)
+			(effects
+				(font
+					(size 1.27 1.27)
+				)
+			)
+		)
+		(property "Datasheet" ""
+			(at 194.31 121.92 0)
+			(hide yes)
+			(show_name no)
+			(do_not_autoplace no)
+			(effects
+				(font
+					(size 1.27 1.27)
+				)
+			)
+		)
+		(property "Description" "Power symbol creates a global label with name \"+3.3VP\""
+			(at 194.31 121.92 0)
+			(hide yes)
+			(show_name no)
+			(do_not_autoplace no)
+			(effects
+				(font
+					(size 1.27 1.27)
+				)
+			)
+		)
+		(pin "1"
+		)
+		(instances
+			(project "Primero_esquematico"
+				(path "/d930f486-f6ac-489c-907e-47f2cb34cf04/d101e913-ebd1-4e08-b728-82218f47123b/ea501642-1303-4ac1-bfff-b969418bd5d5"
+					(reference "#PWR0242")
+					(unit 1)
+				)
+			)
+		)
+	)
 	(symbol
 		(lib_id "power:+3.3VP")
