File: PCB/InverterV2.0/Primero_esquematico/encoder.kicad_sch (KiCad schematic)
At the start: 25 parts, among them J5 348250125, U31 TPD4E05U06DQA, U32 TPD4E05U06DQA, U35 SN65HVD82DR, U36 AM26LS32AIDR, U37 SN74LVC245ANSR, U38 TPD4E05U06DQA

Commit message: aislacion encoder
Parts:
- removed U37: SN74LVC245ANSR, Snapeda:NS20-L, symbol Snapeda:SN74LVC245ANSR
- added C167, C168: 100nF, Capacitor_SMD:C_0603_1608Metric, symbol Device:C
- added C169, C170: 1nF, Capacitor_SMD:C_0603_1608Metric, symbol Device:C
- added C171, C172: 10nF, Capacitor_SMD:C_0603_1608Metric, symbol Device:C
- added C173: 10uF, Capacitor_SMD:C_0805_2012Metric, symbol Device:C
- added C187: 4,7uF, Capacitor_SMD:C_0805_2012Metric, symbol Device:C
- added J2: Conn_01x14_Socket, symbol Connector:Conn_01x14_Socket
- added JP1: Jumper SMD, symbol Jumper:Jumper_2_Open
- added L3: MLZ2012N6R8LT000, Inductor_SMD:L_0805_2012Metric, symbol Device:L
- added PS2: MEV1S1205SC, Snapeda:MEV1S1205SC, symbol Snapeda:MEV1S1205SC
- added R191, R192: 10, Resistor_SMD:R_0603_1608Metric, symbol Device:R
- added R193: 300, Resistor_SMD:R_0603_1608Metric, symbol Device:R
- added U37: ISOW7843DWER, Snapeda:DWE0016A, symbol Snapeda:ISOW7843DWER
- added U42: ISO7710FDWR, Snapeda:D0008B_HV, symbol Snapeda:ISO7710FDWR
- added U43: AMC1303E2520DWV, Snapeda:DWV0008A_TEX-L, symbol Snapeda:AMC1303E2520DWV
- added U44: REF3012, Package_TO_SOT_SMD:SOT-23, symbol Reference_Voltage:REF3012
Connections:
- net +3.3_digital: now also J5.1, C168.1, U37.1 (VCC), U42.14 (VCC2), U43.8 (DVDD)
- net A+: now also J2.4 (Pin_4); no longer J5.4
- net A-: now also J2.3 (Pin_3); no longer J5.3
- net A_MCU: now also J5.3, U37.5 (OUTC)
- net B+: now also J2.12 (Pin_12); no longer J5.12
- net B-: now also J2.11 (Pin_11); no longer J5.11
- net B_MCU: now also J5.4, U37.6 (OUTD)
- net Clock+: now also J2.1 (Pin_1); no longer J5.1
- net Clock-: now also J2.2 (Pin_2); no longer J5.2
- net Clock_MCU: now also U37.3 (INA); no longer U35.4 (D)
- net Data+: now also J2.10 (Pin_10); no longer J5.10
- net Data-: now also J2.9 (Pin_9); no longer J5.9
- net Data_MCU: now also J5.6, U37.4 (OUTB)
- net GND: now also J5.10, J5.11, J5.12, J5.9, C168.2, C172.2, C173.2, PS2.2 (-VIN), U37.2 (GND1), U37.8 (GND1), U42.16 (GND2), U42.9 (GND2), U43.5 (DGND); no longer C161.2, C162.2, J5.6, U31.3 (GND), U31.8 (GND), U32.3 (GND), U32.8 (GND), U35.5 (GND), U36.12 (*G), U36.8 (GND), U38.3 (GND), U38.8 (GND)
- net Z+: now also J2.7 (Pin_7); no longer J5.7
- net Z-: now also J2.8 (Pin_8); no longer J5.8
- net Z_MCU: now also J5.5, U42.13 (OUT)
- net +5V_digital renamed 5V_ISO
- net 5V_ISO: now also C167.1, C187.1, J2.5 (Pin_5), JP1.2 (B), PS2.7 (+VOUT), U42.3 (VCC1), U43.1 (AVDD), U44.1 (IN); no longer J5.5, U32.4 (D2+), U32.5 (D2-)
- net A_MCU_5V renamed A_ISO
- net A_ISO: now also U37.12 (INC)
- net B_MCU_5V renamed B_ISO
- net B_ISO: now also U37.11 (IND)
- net DATA_MCU_5V renamed DATA_ISO
- net DATA_ISO: now also U37.13 (INB)
- net Z_MCU_5V renamed Z_ISO
- net Z_ISO: now also U42.4 (IN)
- new net: JP1.1 (A), U37.16 (VISO)
- new net: C172.1, C173.1, L3.1, PS2.1 (+VIN)
- new net: C169.1, C171.1, R191.1, U43.2 (AINP)
- new net: C170.1, C171.2, R192.2, U43.3 (AINN)
- new net +12V: J5.2
- new net +12V_In: L3.2
- new net Clk_ISO: U35.4 (D), U37.14 (OUTA)
- new net Clk_Temp_MCU: J5.7, U43.7 (CLKOUT)
- new net D_Temp_MCU: J5.8, U43.6 (DOUT)
- new net GND_ISO: C161.2, C162.2, C167.2, C169.2, C170.2, C187.2, J2.6 (Pin_6), PS2.5 (-VOUT), PS2.6 (0V), R192.1, R193.2, U31.3 (GND), U31.8 (GND), U32.3 (GND), U32.8 (GND), U35.5 (GND), U36.12 (*G), U36.8 (GND), U37.10 (SEL), U37.15 (GND2), U37.9 (GND2), U38.3 (GND), U38.8 (GND), U42.1 (GND1), U42.7 (GND1), U43.4 (AGND), U44.3 (GND)
- new net Temp+: J2.13 (Pin_13), U32.4 (D2+), U44.2 (OUT)
- new net Temp-: J2.14 (Pin_14), R191.2, R193.1, U32.5 (D2-)
- no-connect marks 5 -> 10
Other:
- note added: "Conector exterior UTS012E14S"
- note added: "RM44SI"
- note removed: "Conector"
- note removed: "Level shifter"
- moved on the sheet: C159, C160, C161, C162, C163, C164, C165, C166, R180, R181, R182, R183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

Commit message: Mejoras en el rut
Parts:
- removed C167: 100nF, Capacitor_SMD:C_0603_1608Metric, symbol Device:C
- removed C169, C170: 1nF, Capacitor_SMD:C_0603_1608Metric, symbol Device:C
- removed C171: 10nF, Capacitor_SMD:C_0603_1608Metric, symbol Device:C
- removed C187: 4,7uF, Capacitor_SMD:C_0805_2012Metric, symbol Device:C
- removed R191: 10, Resistor_SMD:R_0603_1608Metric, symbol Device:R
- removed U43: AMC1303E2520DWV, Snapeda:DWV0008A_TEX-L, symbol Snapeda:AMC1303E2520DWV
- removed U44: REF3012, Package_TO_SOT_SMD:SOT-23, symbol Reference_Voltage:REF3012
- added C174: 1`00nF, Capacitor_SMD:C_0402_1005Metric, symbol Device:C_Small
- added C175: 100nF, Capacitor_SMD:C_0603_1608Metric, symbol Device:C_Small
- added C176: 100nF, Capacitor_SMD:C_0603_1608Metric, symbol Device:C
- added C180: 1nF, Capacitor_SMD:C_0402_1005Metric, symbol Device:C_Small
- added C181: 4,7uF, Capacitor_SMD:C_0805_2012Metric, symbol Device:C
- added J10: 348250125, Snapeda:CONN_SD-34825-001_12_MOL, symbol Snapeda:348250125
- added R185, R186, R188: 3k, Resistor_SMD:R_0603_1608Metric, symbol Device:R
- added R189, R190: 1k, Resistor_SMD:R_0402_1005Metric, symbol Device:R
- added R194: 100, Resistor_SMD:R_0402_1005Metric, symbol Device:R
- added RV1: 500, Potentiometer_THT:Potentiometer_Bourns_3296W_Vertical, symbol Device:R_Potentiometer_Trim
- added TP20, TP22: TestPoint, TestPoint:TestPoint_Pad_D1.0mm, symbol Connector:TestPoint
- added U38: AMC1200BDWV, Package_SO:SOIC-8_7.5x5.85mm_P1.27mm, symbol Isolator_Analog:AMC1200BDWV
- added U39: OPA333xxDCK, Package_TO_SOT_SMD:SOT-353_SC-70-5, symbol Amplifier_Operational:OPA333xxDCK
- J8: renamed from J2; value Conn_01x14_Socket -> Conector sobre PCB; footprint (none) -> FSAE_footprints:My-UTS012E14S
- JP1: footprint (none) -> Jumper:SolderJumper-2_P1.3mm_Open_RoundedPad1.0x1.5mm
- PS2: MANUFACTURER_PART_NUMBER (none) -> MEV1S1205SC; Manufacturer_Part_Number MEV1S1205SC -> (none)
- R192: value 10 -> 10k; footprint Resistor_SMD:R_0603_1608Metric -> Resistor_SMD:R_0402_1005Metric
- R193: value 300 -> 10k; footprint Resistor_SMD:R_0603_1608Metric -> Resistor_SMD:R_0402_1005Metric
- U35: footprint NuevoGui:D8_TEX-L -> Snapeda:D8_TEX-L
- U40: renamed from U42; footprint Snapeda:D0008B_HV -> Snapeda:SOIC16_DW_TEX-L
- renumbered C159 to C177, C162 to C178, C161 to C179, C160 to C182, C168 to C183, C172 to C184, C173 to C185, C163 to C186, C164 to C187, C165 to C188, C166 to C189, J5 to J9, L3 to L4, R180 to R187, R181 to R191, R182 to R195, R183 to R196, R184 to R197, R185 to R198, TP20 to TP21, TP21 to TP23, TP22 to TP24, U31 to U41, U32 to U42, U38 to U43
Connections:
- net Clock_MCU is gone; now on net CLK_ENC_EXT: U37.3 (INA)
- net +12V: now also J10.2; no longer J9.2
- net +3.3_digital: now also J10.1; no longer C182.1, C183.1, J9.1, U37.1 (VCC), U40.14 (VCC2)
- net GND: now also J10.10, J10.11, J10.12, J10.9; no longer C182.2, C183.2, C184.2, C185.2, J9.10, J9.11, J9.12, J9.9, PS2.2 (-VIN), U37.2 (GND1), U37.8 (GND1), U40.16 (GND2), U40.9 (GND2)
- net Temp+: now also R188.1, U38.2 (VINP)
- net at R192.2: now also R190.2, U39.3 (-)
- net +12V_In renamed +12V_EXT
- net +12V_EXT: now also J9.2
- net 5V_ISO renamed +5V_EXT_ISO
- net +5V_EXT_ISO: now also C174.1, C181.1, R185.2, R188.2, U38.1 (VDD1)
- net A_MCU renamed A_PCB_EXT
- net B_MCU renamed B_PCB_EXT
- net Clk_Temp_MCU renamed CLK_ENC_EXT
- net CLK_ENC_EXT: now also TP20.1
- net D_Temp_MCU renamed TEMP_EXT
- net TEMP_EXT: now also C180.1, R194.2, TP22.1
- net Data_MCU renamed DATA_PCB_EXT
- net GND_ISO renamed GND_EXT_ISO
- net GND_EXT_ISO: now also J8.14 (Pin_14), U42.5 (D2-), C174.2, C181.2, RV1.1, RV1.2, U38.4 (GND1); no longer R192.1, R193.2
- removed net Temp-: J8.14 (Pin_14), R193.1, U42.5 (D2-)
- net Z_MCU renamed Z_PCB_EXT
- new net: C175.1, R189.1, U38.7 (VOUTP)
- new net: R189.2, R193.1, U39.1 (+)
- new net: R193.2, R194.1, U39.4
- new net: C175.2, R190.1, U38.6 (VOUTN)
- new net: R185.1, R186.2, U38.3 (VINN)
- new net: R186.1, RV1.3
- new net +3.3_EXT: C176.1, C182.1, C183.1, J9.1, U37.1 (VCC), U38.8 (VDD2), U39.5 (V+), U40.14 (VCC2)
- new net A_PCB_MCU: J10.3
- new net B_PCB_MCU: J10.4
- new net CLK_PCB_MCU: J10.7
- new net DATA_PCB_MCU: J10.6
- new net GND_EXT: C176.2, C180.2, C182.2, C183.2, C184.2, C185.2, J9.10, J9.11, J9.12, J9.9, PS2.2 (-VIN), R192.1, U37.2 (GND1), U37.8 (GND1), U38.5 (GND2), U39.2 (V-), U40.16 (GND2), U40.9 (GND2)
- new net TEMP_MCU: J10.8
- new net Z_PCB_MCU: J10.5
Other:
- note added: "Bloques Aislados:"
- note removed: "Compatible para encoder absolutos e incrametanles. Protocolo unidireccional SSI Compatible para modelos de RM44SI y RM44SC entre otros"
- note removed: "RM44SIA+/A−, B+/B−, Z+/Z− + Clock±, Data± (BiSS c/SSI)"
- note removed: "SE DESCARTO ESTO POR SER MUCHO HARDWARE QUE NO SE VA A USAR Vamos a dimencionar el encoder para el caso del RM44SI dado a que es el sistema mas completo (Prefieron que sobre hardware a que falte)"
- moved on the sheet: C178, C179, C182, C183, C184, C185, C186, C187, C188, C189, JP1, L4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

Commit message: Casi listo
Connections:
- net +12V: now also J10.3, J10.4; no longer J10.2
- net +3.3_digital: now also J10.6; no longer J10.1
- net A_PCB_MCU: now also J10.2; no longer J10.3
- net B_PCB_MCU: now also J10.1; no longer J10.4
- net DATA_PCB_MCU: now also J10.8; no longer J10.6
- net GND: no longer J10.10
- net TEMP_MCU: now also J10.10; no longer J10.8

Commit message: el drc esta tirando mucho error hay q solucionar eso
Parts:
- removed C174: 1`00nF, Capacitor_SMD:C_0402_1005Metric, symbol Device:C_Small
- removed C175: 100nF, Capacitor_SMD:C_0603_1608Metric, symbol Device:C_Small
- removed C176, C178, C179, C182, C183: 100nF, Capacitor_SMD:C_0603_1608Metric, symbol Device:C
- removed C177, C184, C186, C187, C188, C189: 10nF, Capacitor_SMD:C_0603_1608Metric, symbol Device:C
- removed C180: 1nF, Capacitor_SMD:C_0402_1005Metric, symbol Device:C_Small
- removed C181: 4,7uF, Capacitor_SMD:C_0805_2012Metric, symbol Device:C
- removed C185: 10uF, Capacitor_SMD:C_0805_2012Metric, symbol Device:C
- removed J8: Conector sobre PCB, FSAE_footprints:My-UTS012E14S, symbol Connector:Conn_01x14_Socket
- removed J9: 348250125, Snapeda:CONN_SD-34825-001_12_MOL, symbol Snapeda:348250125
- removed JP1: Jumper SMD, Jumper:SolderJumper-2_P1.3mm_Open_RoundedPad1.0x1.5mm, symbol Jumper:Jumper_2_Open
- removed L4: MLZ2012N6R8LT000, Inductor_SMD:L_0805_2012Metric, symbol Device:L
- removed PS2: MEV1S1205SC, Snapeda:MEV1S1205SC, symbol Snapeda:MEV1S1205SC
- removed R185, R186, R188: 3k, Resistor_SMD:R_0603_1608Metric, symbol Device:R
- removed R187: 10k, Resistor_SMD:R_0603_1608Metric, symbol Device:R
- removed R189, R190: 1k, Resistor_SMD:R_0402_1005Metric, symbol Device:R
- removed R191, R195, R196, R197, R198: 120, Resistor_SMD:R_0603_1608Metric, symbol Device:R
- removed R192, R193: 10k, Resistor_SMD:R_0402_1005Metric, symbol Device:R
- removed R194: 100, Resistor_SMD:R_0402_1005Metric, symbol Device:R
- removed RV1: 500, Potentiometer_THT:Potentiometer_Bourns_3296W_Vertical, symbol Device:R_Potentiometer_Trim
- removed TP19, TP20, TP21, TP22, TP23, TP24: TestPoint, TestPoint:TestPoint_Pad_D1.0mm, symbol Connector:TestPoint
- removed U35: SN65HVD82DR, Snapeda:D8_TEX-L, symbol Snapeda:SN65HVD82DR
- removed U36: AM26LS32AIDR, Snapeda:D16-L, symbol Snapeda:AM26LS32AIDR
- removed U37: ISOW7843DWER, Snapeda:DWE0016A, symbol Snapeda:ISOW7843DWER
- removed U38: AMC1200BDWV, Package_SO:SOIC-8_7.5x5.85mm_P1.27mm, symbol Isolator_Analog:AMC1200BDWV
- removed U39: OPA333xxDCK, Package_TO_SOT_SMD:SOT-353_SC-70-5, symbol Amplifier_Operational:OPA333xxDCK
- removed U40: ISO7710FDWR, Snapeda:SOIC16_DW_TEX-L, symbol Snapeda:ISO7710FDWR
- removed U41, U42, U43: TPD4E05U06DQA, Package_SON:USON-10_2.5x1.0mm_P0.5mm, symbol Power_Protection:TPD4E05U06DQA
Connections:
- no-connect marks 10 -> 0
Other:
- note added: "El resto de los conectores y circuitos integrados estan en una pcb externa"
- note removed: "Bloques Aislados:"
- note removed: "El fabricante recomienda"
- note removed: "Receiver RS-422"
- note removed: "Transceiver RS-422"
- moved on the sheet: J10
