File: PCB/InverterV2.0/Primero_esquematico/pcb_potencia.kicad_sch (KiCad schematic)
At the start: 0 parts

Commit message: Todo Listo para mandar
Parts:
- added R44, R57, R58, R59, R72, R73: 22, Capacitor_SMD:C_0402_1005Metric_Pad0.74x0.62mm_HandSolder, symbol Device:R
Connections:
- net PWM_H_A: now also R44.2
- net PWM_H_B: now also R59.2
- net PWM_H_C: now also R73.2
- net PWM_L_A: now also R57.1
- net PWM_L_B: now also R58.1
- net PWM_L_C: now also R72.1
- new net Gate_Driver/C1_In_neg: R57.2
- new net Gate_Driver/C1_In_pos: R44.1
- new net Gate_Driver/C2_In_neg: R58.2
- new net Gate_Driver/C2_In_pos: R59.1
- new net Gate_Driver/C3_In_neg: R72.2
- new net Gate_Driver/C3_In_pos: R73.1
