File: PCB/InverterV2.0/EncoderBoard/EncoderBoard.kicad_sch (KiCad schematic)
At the start: 52 parts, among them J10 348250125, J8 Conector sobre PCB, J9 348250125, U35 SN65HVD82DR, U36 AM26LS32AIDR, U37 ISOW7843DWER, U38 AMC1200BDWV, U39 OPA333xxDCK, U40 ISO7710FDWR, U41 TPD4E05U06DQA, U42 TPD4E05U06DQA, U43 TPD4E05U06DQA

Commit message: pcb encoder
Parts:
- removed J10: 348250125, Snapeda:CONN_SD-34825-001_12_MOL, symbol Snapeda:348250125
- added H2: 3mm, MountingHole:MountingHole_3.2mm_M3_ISO14580_Pad_TopBottom, symbol Mechanical:MountingHole_Pad
- added H3, H4: 3mm, MountingHole:MountingHole_3.2mm_M3, symbol Mechanical:MountingHole
- C174: value 1`00nF -> 100nF; footprint Capacitor_SMD:C_0402_1005Metric -> Capacitor_SMD:C_0603_1608Metric
- C180: footprint Capacitor_SMD:C_0402_1005Metric -> Capacitor_SMD:C_0603_1608Metric
Connections:
- net A+: now also U41.5 (D2-); no longer U41.4 (D2+)
- net A-: now also U41.4 (D2+); no longer U41.5 (D2-)
- net A_PCB_EXT: now also J9.10; no longer J9.3
- net B+: now also J8.11 (Pin_11); no longer J8.12 (Pin_12)
- net B-: now also J8.10 (Pin_10); no longer J8.11 (Pin_11)
- net B_PCB_EXT: now also J9.9; no longer J9.4
- net CLK_ENC_EXT: now also J9.12; no longer J9.7
- net DATA_PCB_EXT: now also J9.11; no longer J9.6
- net Data+: now also J8.9 (Pin_9), U43.5 (D2-); no longer J8.10 (Pin_10), U43.2 (D1-)
- net Data-: now also J8.8 (Pin_8), U43.4 (D2+); no longer J8.9 (Pin_9), U43.1 (D1+)
- net GND_EXT: now also J9.3, J9.4, J9.7, J9.8, H2.1; no longer J9.10, J9.11, J9.12, J9.9
- net GND_EXT_ISO: now also J8.13 (Pin_13); no longer J8.6 (Pin_6)
- net TEMP_EXT: now also J9.6; no longer J9.8
- net Temp+: now also J8.12 (Pin_12); no longer J8.13 (Pin_13)
- net Z+: now also J8.6 (Pin_6), U43.1 (D1+); no longer J8.7 (Pin_7), U43.4 (D2+)
- net Z-: now also J8.7 (Pin_7), U43.2 (D1-); no longer J8.8 (Pin_8), U43.5 (D2-)
Other:
- note added: "Temp Motor"
- moved on the sheet: C181, C183, C184, C185, J9, L4, PS2, TP19, TP20, TP21, TP22, TP23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
