File: PCB/FSAE-Precarga/Medicion.kicad_sch (KiCad schematic)
At the start: 47 parts, among them U10 6N137, U2 LM331N, U3 6N137, U4 LM2904, U5 LM331N

Commit message: Agrego correcciones/agregados placa precarga
Parts:
- added J6: Conn_01x02_Pin, symbol Connector:Conn_01x02_Pin
- added Q2: AO3407A, Package_TO_SOT_SMD:SOT-23, symbol Transistor_FET:AO3401A
- added R39: 54.9k, Resistor_SMD:R_0805_2012Metric, symbol Device:R
- added R40: 3.3k, Resistor_SMD:R_0805_2012Metric, symbol Device:R
- added R41: 47k, Resistor_SMD:R_0805_2012Metric, symbol Device:R
- added R42: 1M, Resistor_SMD:R_0805_2012Metric, symbol Device:R
- added R43: 3.3K, Resistor_SMD:R_0805_2012Metric, symbol Device:R
- added R44: 22K, Resistor_SMD:R_0805_2012Metric, symbol Device:R
- added U12: PC817, Package_DIP:DIP-4_W7.62mm, symbol Isolator:PC817
- added U7: TLV1701AIDBVR, Mis_Huellas:DBV0005A_N, symbol 2026-09-18_04-07-55:TLV1701AIDBVR
Connections:
- net 12VMed: now also R39.1, R41.1, R43.1, U7.5 (V+)
- net GndLogic: now also J6.2 (Pin_2), R44.2
- net GndMed: now also R40.2, U7.2 (V-)
- net IN_Cmp: now reaches R6.1, U4.6 (-), U4.7
- net IN_Cmp: now also U7.3 (IN-)
- new net: J6.1 (Pin_1), Q2.3 (D)
- new net: R41.2, R42.2, U12.2, U7.4 (OUT)
- new net: R43.2, U12.1
- new net: Q2.1 (G), R44.1, U12.3
- new net 12VLogic: Q2.2 (S), U12.4
- new net Vref: R39.2, R40.1, R42.1, U7.1 (IN+)
Other:
- moved on the sheet: C1, C2, CL1, CL2, CL3, CL4, CL5, CL6, Ct1, Ct2, R1, R14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

Commit message: Agrego circuito de control/verificacion de los AIR en placa de precarga
Parts:
- added Q4: 2N7002, Package_TO_SOT_SMD:SOT-23, symbol Transistor_FET:2N7002
- R43: value 3.3K -> 3.3k
Connections:
- net 12VLogic: now also R44.1; no longer U12.4
- net GndLogic: now also U12.3; no longer R44.2
- net GndMed: now also Q4.2 (S)
- net at R41.2, R42.2, U7.4 (OUT): now also Q4.1 (G); no longer U12.2
- new net: Q4.3 (D), U12.2
- new net: Q2.1 (G), R44.2, U12.4
Other:
- moved on the sheet: J6, Q2, R44
