File: PCB/FSAE-PosicionVolante/FSAE-PosicionVolante.kicad_sch (KiCad schematic)
At the start: 17 parts, among them IC1 LM1085IT-5.0_NOPB, J1 Conn_ Molex, U1 TJA1042T-3, U2 ESP

Commit message: Correciones placa sensor de posicion del Volante
Parts:
- removed C1: 10uF, Capacitor_SMD:C_0805_2012Metric_Pad1.18x1.45mm_HandSolder, symbol Device:C_Polarized
- C4: footprint Capacitor_Tantalum_SMD:CP_EIA-2012-12_Kemet-R_HandSolder -> Capacitor_Tantalum_SMD:CP_EIA-3216-18_Kemet-A_HandSolder
- C5: footprint Capacitor_SMD:C_0805_2012Metric_Pad1.18x1.45mm_HandSolder -> Capacitor_SMD:C_1206_3216Metric_Pad1.33x1.80mm_HandSolder
Connections:
- net GND: now also CR2.2; no longer CR2.1
- net VBAT_PROT: now also CR2.1; no longer CR2.2
