File: PCB/FSAE-PosicionVolante/FSAE-PosicionVolante.kicad_pcb (KiCad board)
At the start: 2 copper layers, 45 x 50.1 mm, 19 parts, among them IC1 LM1085IT-5.0_NOPB, J1 Conn_ Molex, U1 TJA1042T-3, U2 ESP

Commit message: Correciones placa sensor de posicion del Volante
Parts:
- removed C1: 10uF, Capacitor_SMD:C_0805_2012Metric_Pad1.18x1.45mm_HandSolder
- added G: LOGO, FSAE_Kicad_Footprints:logo, F.Cu at (109.3, 109.4)
- C4: footprint Capacitor_Tantalum_SMD:CP_EIA-2012-12_Kemet-R_HandSolder -> Capacitor_Tantalum_SMD:CP_EIA-3216-18_Kemet-A_HandSolder
- C5: footprint Capacitor_SMD:C_0805_2012Metric_Pad1.18x1.45mm_HandSolder -> Capacitor_SMD:C_1206_3216Metric_Pad1.33x1.80mm_HandSolder
- moved C5 0.82 mm to (116.4, 92.9)
- moved CR2 0.69 mm to (109.0, 90.9), turned to 180 degrees
Connections:
- CR2 pad 1: GND -> /VBAT_PROT
- CR2 pad 2: /VBAT_PROT -> GND
Routing:
- net /VBAT_PROT: track 15.3 -> 16.8 mm
- net GND: track 24.5 -> 25.8 mm, vias 0 -> 1
- net +5V: track 60.3 -> 59.0 mm
- added copper zone on B.Cu, net GND
Other:
- board text added: "By AnaLE"
- board text added: "Sensor Pos. Volante"
- board text added: "V1.0"

Commit message: Actualizacion pcb placa pos. volante
Other:
- board text added: "By Ana LE"
- board text removed: "By AnaLE"
Changed lines of the file:
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@@
 		)
 	)
-	(gr_text "By AnaLE\n"
+	(gr_text "By Ana LE"
 		(at 140.1 125.641223 0)
 		(layer "B.SilkS")

Commit message: Actulizacion Placa sensor posicion volante
Parts:
- moved IC1 9.87 mm to (107.3, 98.1), turned to 90 degrees
- moved CR2 7.63 mm to (114.7, 96.0), turned to 0 degrees
- moved F1 4.48 mm to (112.7, 88.4)
- moved C5 1.81 mm to (115.7, 91.2), turned to 0 degrees
- moved C4 0.50 mm to (121.0, 95.8)
Routing:
- net +5V: track 59.0 -> 72.0 mm, vias 0 -> 1
- net GND: track 25.8 -> 16.2 mm
- net /VBAT: track 3.74 -> 8.09 mm
- net /VBAT_PROT: track 16.8 -> 15.6 mm
- net /ENC_B: track 11.1 -> 10.0 mm
- net +3V3: track 45.2 -> 46.3 mm, vias 0 -> 1
- net /CANH: track 9.95 -> 9.41 mm
- net /ENC_A: track 20.9 -> 20.8 mm, vias 0 -> 1
